Commit message: update 4WD ros2_control.xacro

File: romea_odo_description/ros2_control/4WD.ros2_control.xacro (robot description, xacro)
@@ -6,6 +6,6 @@
           <plugin>gazebo_ros2_control/GazeboSystem</plugin>
         </hardware>
-         <joint name="${front_left_wheel_spining_joint}">
-           <command_interface name="position">
+         <joint name="${prefix}${front_left_wheel_spinning_joint}">
+           <command_interface name="velocity">
              <param name="min">-1</param>
              <param name="max">1</param>
@@ -13,6 +13,6 @@
            <state_interface name="velocity"/>
          </joint>
-        <joint name="${front_right_wheel_spining_joint}">
-          <command_interface name="position">
+        <joint name="${prefix}${front_right_wheel_spinning_joint}">
+          <command_interface name="velocity">
             <param name="min">-1</param>
             <param name="max">1</param>
@@ -20,6 +20,6 @@
           <state_interface name="velocity"/>
         </joint>
-        <joint name="${rear_right_wheel_spining_joint}">
-          <command_interface name="position">
+        <joint name="${prefix}${rear_left_wheel_spinning_joint}">
+          <command_interface name="velocity">
             <param name="min">-1</param>
             <param name="max">1</param>
@@ -27,6 +27,6 @@
           <state_interface name="velocity"/>
         </joint>
-        <joint name="${rear_right_wheel_spining_joint}">
-          <command_interface name="position">
+        <joint name="${prefix}${rear_right_wheel_spinning_joint}">
+          <command_interface name="velocity">
             <param name="min">-1</param>
             <param name="max">1</param>
