Commit message: robot_odo_description : add option to select hardware plugin

File: romea_odo_description/ros2_control/2FWS_4WD.ros2_control.xacro (robot description, xacro)
@@ -1,9 +1,11 @@
 <?xml version="1.0"?>
 <robot xmlns:xacro="http://www.ros.org/wiki/xacro">
-  <xacro:macro name="base_control">
+  <xacro:macro name="base_control" params="use_sim">
     <ros2_control name="${prefix}base" type="system">
-        <hardware>
-          <plugin>gazebo_ros2_control/GazeboSystem</plugin>
-        </hardware>
+        <xacro:if value="$(arg use_sim)">
+             <hardware>
+               <plugin>gazebo_ros2_control/GazeboSystem</plugin>
+             </hardware>
+        </xacro:if>
         <joint name="${prefix}${front_left_wheel_steering_joint}">
           <command_interface name="position">

File: romea_odo_description/ros2_control/2RWS_4WD.ros2_control.xacro (robot description, xacro)
@@ -1,9 +1,11 @@
 <?xml version="1.0"?>
 <robot xmlns:xacro="http://www.ros.org/wiki/xacro">
-  <xacro:macro name="base_control">
+  <xacro:macro name="base_control" params="use_sim">
     <ros2_control name="${prefix}base" type="system">
-        <hardware>
-          <plugin>gazebo_ros2_control/GazeboSystem</plugin>
-        </hardware>
+        <xacro:if value="$(arg use_sim)">
+            <hardware>
+              <plugin>gazebo_ros2_control/GazeboSystem</plugin>
+            </hardware>
+        </xacro:if>
         <joint name="${prefix}${rear_left_wheel_steering_joint}">
           <command_interface name="position">

File: romea_odo_description/ros2_control/4WD.ros2_control.xacro (robot description, xacro)
@@ -1,9 +1,11 @@
 <?xml version="1.0"?>
 <robot xmlns:xacro="http://www.ros.org/wiki/xacro">
-  <xacro:macro name="base_control">
+  <xacro:macro name="base_control" params="use_sim">
     <ros2_control name="${prefix}base" type="system">
-        <hardware>
-          <plugin>gazebo_ros2_control/GazeboSystem</plugin>
-        </hardware>
+        <xacro:if value="$(arg use_sim)">
+            <hardware>
+              <plugin>gazebo_ros2_control/GazeboSystem</plugin>
+            </hardware>
+         </xacro:if>
          <joint name="${prefix}${front_left_wheel_spinning_joint}">
            <command_interface name="velocity">

File: romea_odo_description/ros2_control/4WS_4WD.ros2_control.xacro (robot description, xacro)
@@ -1,9 +1,11 @@
 <?xml version="1.0"?>
 <robot xmlns:xacro="http://www.ros.org/wiki/xacro">
-  <xacro:macro name="base_control">
+  <xacro:macro name="base_control" params="use_sim">
     <ros2_control name="${prefix}base" type="system">
-        <hardware>
-          <plugin>gazebo_ros2_control/GazeboSystem</plugin>
-        </hardware>
+        <xacro:if value="$(arg use_sim)">
+            <hardware>
+              <plugin>gazebo_ros2_control/GazeboSystem</plugin>
+            </hardware>
+        </xacro:if>
         <joint name="${prefix}${front_left_wheel_steering_joint}">
           <command_interface name="position">
