Commit message: mobile base description : add axcro files for track vehicules

File: romea_mobile_base_description/ros2_control/2THD.ros2_control.xacro (robot description, xacro)
@@ -8,33 +8,23 @@
             </hardware>
         </xacro:if>
-        <joint name="${prefix}${front_left_wheel_steering_joint}">
-          <command_interface name="position">
+        <joint name="${prefix}${high_left_sprocket_wheel_spinning_joint}">
+          <command_interface name="velocity">
             <param name="min">-1</param>
             <param name="max">1</param>
           </command_interface>
           <state_interface name="position"/>
+          <state_interface name="velocity"/>
+          <state_interface name="effort"/>
         </joint>
-        <joint name="${prefix}${front_right_wheel_steering_joint}">
-          <command_interface name="position">
+        <joint name="${prefix}${high_right_sprocket_wheel_spinning_joint}">
+          <command_interface name="velocity">
             <param name="min">-1</param>
             <param name="max">1</param>
           </command_interface>
           <state_interface name="position"/>
+          <state_interface name="velocity"/>
+          <state_interface name="effort"/>
         </joint>
-        <joint name="${prefix}${rear_left_wheel_steering_joint}">
-          <command_interface name="position">
-            <param name="min">-1</param>
-            <param name="max">1</param>
-          </command_interface>
-          <state_interface name="position"/>
-        </joint>
-        <joint name="${prefix}${rear_right_wheel_steering_joint}">
-          <command_interface name="position">
-            <param name="min">-1</param>
-            <param name="max">1</param>
-          </command_interface>
-          <state_interface name="position"/>
-        </joint>
-         <joint name="${prefix}${front_left_wheel_spinning_joint}">
+         <joint name="${prefix}${front_left_idler_wheel_spinning_joint}">
            <command_interface name="velocity">
              <param name="min">-1</param>
@@ -45,5 +35,5 @@
            <state_interface name="effort"/>
          </joint>
-        <joint name="${prefix}${front_right_wheel_spinning_joint}">
+        <joint name="${prefix}${front_right_idler_wheel_spinning_joint}">
           <command_interface name="velocity">
             <param name="min">-1</param>
@@ -54,5 +44,5 @@
           <state_interface name="effort"/>
         </joint>
-        <joint name="${prefix}${rear_right_wheel_spinning_joint}">
+        <joint name="${prefix}${rear_left_idler_wheel_spinning_joint}">
           <command_interface name="velocity">
             <param name="min">-1</param>
@@ -63,13 +53,13 @@
           <state_interface name="effort"/>
         </joint>
-        <joint name="${prefix}${rear_right_wheel_spinning_joint}">
-          <command_interface name="velocity">
-            <param name="min">-1</param>
-            <param name="max">1</param>
-          </command_interface>
-          <state_interface name="position"/>
-          <state_interface name="velocity"/>
-          <state_interface name="effort"/>
-        </joint>
+       <joint name="${prefix}${rear_right_idler_wheel_spinning_joint}">
+         <command_interface name="velocity">
+           <param name="min">-1</param>
+           <param name="max">1</param>
+         </command_interface>
+         <state_interface name="position"/>
+         <state_interface name="velocity"/>
+         <state_interface name="effort"/>
+       </joint>
     </ros2_control>
   </xacro:macro>
