Commit message: mobile base description :  add xacro for 2TTD vechiles  fix pbs in 4WS4WD xacro files

File: romea_mobile_base_description/ros2_control/2TTD.ros2_control.xacro (robot description, xacro)
@@ -1,40 +1,48 @@
 <?xml version="1.0"?>
 <robot xmlns:xacro="http://www.ros.org/wiki/xacro">
-  <xacro:macro name="base_control" params="use_sim:=true">
+  <xacro:macro name="base_control" params="use_sim">
     <ros2_control name="${prefix}base" type="system">
-        <xacro:if value="${use_sim}">
+        <xacro:if value="$(arg use_sim)">
             <hardware>
               <plugin>gazebo_ros2_control/GazeboSystem</plugin>
             </hardware>
         </xacro:if>
-        <joint name="${prefix}${front_left_wheel_steering_joint}">
-          <command_interface name="position">
+        <joint name="${prefix}${high_left_sprocket_wheel_spinning_joint}">
+          <command_interface name="velocity">
             <param name="min">-1</param>
             <param name="max">1</param>
           </command_interface>
           <state_interface name="position"/>
+          <state_interface name="velocity"/>
+          <state_interface name="effort"/>
         </joint>
-        <joint name="${prefix}${front_right_wheel_steering_joint}">
-          <command_interface name="position">
+        <joint name="${prefix}${high_right_sprocket_wheel_spinning_joint}">
+          <command_interface name="velocity">
             <param name="min">-1</param>
             <param name="max">1</param>
           </command_interface>
           <state_interface name="position"/>
+          <state_interface name="velocity"/>
+          <state_interface name="effort"/>
         </joint>
-        <joint name="${prefix}${rear_left_wheel_steering_joint}">
-          <command_interface name="position">
+        <joint name="${prefix}${left_idler_wheel_spinning_joint}">
+          <command_interface name="velocity">
             <param name="min">-1</param>
             <param name="max">1</param>
           </command_interface>
           <state_interface name="position"/>
+          <state_interface name="velocity"/>
+          <state_interface name="effort"/>
         </joint>
-        <joint name="${prefix}${rear_right_wheel_steering_joint}">
-          <command_interface name="position">
-            <param name="min">-1</param>
-            <param name="max">1</param>
-          </command_interface>
-          <state_interface name="position"/>
+        <joint name="${prefix}${right_idler_wheel_spinning_joint}">
+         <command_interface name="velocity">
+           <param name="min">-1</param>
+           <param name="max">1</param>
+         </command_interface>
+         <state_interface name="position"/>
+         <state_interface name="velocity"/>
+         <state_interface name="effort"/>
         </joint>
-         <joint name="${prefix}${front_left_wheel_spinning_joint}">
+         <joint name="${prefix}${front_left_roller_wheel_spinning_joint}">
            <command_interface name="velocity">
              <param name="min">-1</param>
@@ -45,5 +53,5 @@
            <state_interface name="effort"/>
          </joint>
-        <joint name="${prefix}${front_right_wheel_spinning_joint}">
+        <joint name="${prefix}${front_right_roller_wheel_spinning_joint}">
           <command_interface name="velocity">
             <param name="min">-1</param>
@@ -54,5 +62,5 @@
           <state_interface name="effort"/>
         </joint>
-        <joint name="${prefix}${rear_left_wheel_spinning_joint}">
+        <joint name="${prefix}${rear_left_roller_wheel_spinning_joint}">
           <command_interface name="velocity">
             <param name="min">-1</param>
@@ -63,13 +71,13 @@
           <state_interface name="effort"/>
         </joint>
-        <joint name="${prefix}${rear_right_wheel_spinning_joint}">
-          <command_interface name="velocity">
-            <param name="min">-1</param>
-            <param name="max">1</param>
-          </command_interface>
-          <state_interface name="position"/>
-          <state_interface name="velocity"/>
-          <state_interface name="effort"/>
-        </joint>
+       <joint name="${prefix}${rear_right_roller_wheel_spinning_joint}">
+         <command_interface name="velocity">
+           <param name="min">-1</param>
+           <param name="max">1</param>
+         </command_interface>
+         <state_interface name="position"/>
+         <state_interface name="velocity"/>
+         <state_interface name="effort"/>
+       </joint>
     </ros2_control>
   </xacro:macro>

File: romea_mobile_base_description/ros2_control/4WD.ros2_control.xacro (robot description, xacro)
@@ -1,9 +1,10 @@
 <?xml version="1.0"?>
 <robot xmlns:xacro="http://www.ros.org/wiki/xacro">
-  <xacro:macro name="base_control" params="use_sim">
+  <xacro:macro name="base_control" params="use_sim:=true">
     <ros2_control name="${prefix}base" type="system">
-        <xacro:if value="$(arg use_sim)">
+        <xacro:if value="${use_sim}">
             <hardware>
-              <plugin>gazebo_ros2_control/GazeboSystem</plugin>
+<!--              <plugin>gazebo_ros2_control/GazeboSystem</plugin>-->
+              <plugin>romea_mobile_base_gazebo/GazeboSystemInterface4WD</plugin>
             </hardware>
          </xacro:if>

File: romea_mobile_base_description/urdf/2TTD.xacro (robot description, xacro)
@@ -28,7 +28,7 @@
     </xacro:wheel>
     <xacro:wheel parent_link="${base_link}"
-                 wheel_spinning_link="${front_left_idler_spinning_link}"
-                 wheel_spinning_joint="${front_left_idler_spinning_joint}"
-                 wheel_mass="${front_idler_wheel_mass}"
+                 wheel_spinning_link="${left_idler_wheel_spinning_link}"
+                 wheel_spinning_joint="${left_idler_wheel_spinning_joint}"
+                 wheel_mass="${idler_wheel_mass}"
                  wheel_width="${track_width}"
                  wheel_radius="${idler_wheel_radius}"
@@ -47,4 +47,44 @@
       <xacro:insert_block name="visual_wheel"/>
     </xacro:wheel>
+    <xacro:wheel parent_link="${base_link}"
+                 wheel_spinning_link="${front_left_roller_wheel_spinning_link}"
+                 wheel_spinning_joint="${front_left_roller_wheel_spinning_joint}"
+                 wheel_mass="${roller_wheel_mass}"
+                 wheel_width="${track_width}"
+                 wheel_radius="${roller_wheel_radius}"
+                 left_right="-1">
+      <origin xyz="${front_roller_wheel_x} ${track/2} ${roller_wheel_radius - chassis_height}" rpy="${-M_PI/2} 0 0" />
+      <xacro:insert_block name="visual_wheel"/>
+    </xacro:wheel>
+    <xacro:wheel parent_link="${base_link}"
+                 wheel_spinning_link="${front_right_roller_wheel_spinning_link}"
+                 wheel_spinning_joint="${front_right_roller_wheel_spinning_joint}"
+                 wheel_mass="${idler_wheel_mass}"
+                 wheel_width="${track_width}"
+                 wheel_radius="${idler_wheel_radius}"
+                 left_right="1">
+      <origin xyz="${front_roller_wheel_x} ${-track/2} ${roller_wheel_radius - chassis_height}" rpy="${-M_PI/2} 0 0" />
+      <xacro:insert_block name="visual_wheel"/>
+    </xacro:wheel>
+   <xacro:wheel parent_link="${base_link}"
+                wheel_spinning_link="${rear_left_roller_wheel_spinning_link}"
+                wheel_spinning_joint="${rear_left_roller_wheel_spinning_joint}"
+                wheel_mass="${roller_wheel_mass}"
+                wheel_width="${track_width}"
+                wheel_radius="${roller_wheel_radius}"
+                left_right="-1">
+     <origin xyz="${rear_roller_wheel_x} ${track/2} ${roller_wheel_radius - chassis_height}" rpy="${-M_PI/2} 0 0" />
+     <xacro:insert_block name="visual_wheel"/>
+   </xacro:wheel>
+   <xacro:wheel parent_link="${base_link}"
+                wheel_spinning_link="${rear_right_roller_wheel_spinning_link}"
+                wheel_spinning_joint="${rear_right_roller_wheel_spinning_joint}"
+                wheel_mass="${idler_wheel_mass}"
+                wheel_width="${track_width}"
+                wheel_radius="${idler_wheel_radius}"
+                left_right="1">
+     <origin xyz="${rear_roller_wheel_x} ${-track/2} ${roller_wheel_radius - chassis_height}" rpy="${-M_PI/2} 0 0" />
+     <xacro:insert_block name="visual_wheel"/>
+   </xacro:wheel>
   </xacro:macro>
 </robot>
