Commit message: mobile bas description : add some urdf model

File: romea_mobile_base_description/ros2_control/1FAS_4WD.ros2_control.xacro (robot description, xacro)
@@ -4,8 +4,15 @@
     <ros2_control name="${prefix}base" type="system">
         <xacro:if value="$(arg use_sim)">
-            <hardware>
-              <plugin>gazebo_ros2_control/GazeboSystem</plugin>
-            </hardware>
+             <hardware>
+               <plugin>gazebo_ros2_control/GazeboSystem</plugin>
+             </hardware>
         </xacro:if>
+       <joint name="${prefix}${front_axle_steering_joint}">
+         <command_interface name="position">
+           <param name="min">-1</param>
+           <param name="max">1</param>
+         </command_interface>
+         <state_interface name="position"/>
+       </joint>
         <joint name="${prefix}${front_left_wheel_steering_joint}">
           <command_interface name="position">
@@ -22,20 +29,6 @@
           <state_interface name="position"/>
         </joint>
-        <joint name="${prefix}${rear_left_wheel_steering_joint}">
-          <command_interface name="position">
-            <param name="min">-1</param>
-            <param name="max">1</param>
-          </command_interface>
-          <state_interface name="position"/>
-        </joint>
-        <joint name="${prefix}${rear_right_wheel_steering_joint}">
-          <command_interface name="position">
-            <param name="min">-1</param>
-            <param name="max">1</param>
-          </command_interface>
-          <state_interface name="position"/>
-        </joint>
-         <joint name="${prefix}${front_left_wheel_spinning_joint}">
-           <command_interface name="position">
+         <joint name="${prefix}${front_left_wheel_spining_joint}">
+           <command_interface name="velocity">
              <param name="min">-1</param>
              <param name="max">1</param>
@@ -45,6 +38,6 @@
            <state_interface name="effort"/>
          </joint>
-        <joint name="${prefix}${front_right_wheel_spinning_joint}">
-          <command_interface name="position">
+        <joint name="${prefix}${front_right_wheel_spining_joint}">
+          <command_interface name="velocity">
             <param name="min">-1</param>
             <param name="max">1</param>
@@ -54,6 +47,6 @@
           <state_interface name="effort"/>
         </joint>
-        <joint name="${prefix}${rear_right_wheel_spinning_joint}">
-          <command_interface name="position">
+        <joint name="${prefix}${rear_right_wheel_spining_joint}">
+          <command_interface name="velocity">
             <param name="min">-1</param>
             <param name="max">1</param>
@@ -63,5 +56,5 @@
           <state_interface name="effort"/>
         </joint>
-        <joint name="${prefix}${rear_right_wheel_spinning_joint}">
+        <joint name="${rear_right_wheel_spining_joint}">
           <command_interface name="position">
             <param name="min">-1</param>

File: romea_mobile_base_description/ros2_control/2AS_4WD.ros2_control.xacro (robot description, xacro)
@@ -8,4 +8,18 @@
             </hardware>
         </xacro:if>
+        <joint name="${prefix}${front_axle_steering_joint}">
+          <command_interface name="position">
+            <param name="min">-1</param>
+            <param name="max">1</param>
+          </command_interface>
+          <state_interface name="position"/>
+        </joint>
+       <joint name="${prefix}${rear_axle_steering_joint}">
+         <command_interface name="position">
+           <param name="min">-1</param>
+           <param name="max">1</param>
+         </command_interface>
+         <state_interface name="position"/>
+       </joint>
         <joint name="${prefix}${front_left_wheel_steering_joint}">
           <command_interface name="position">

File: romea_mobile_base_description/ros2_control/2FWS_4WD.ros2_control.xacro (robot description, xacro)
@@ -15,5 +15,5 @@
           <state_interface name="position"/>
         </joint>
-        <joint name="${front_right_wheel_steering_joint}">
+        <joint name="${prefix}${front_right_wheel_steering_joint}">
           <command_interface name="position">
             <param name="min">-1</param>
@@ -22,17 +22,30 @@
           <state_interface name="position"/>
         </joint>
-         <joint name="${front_left_wheel_spining_joint}">
-           <command_interface name="position">
+         <joint name="${prefix}${front_left_wheel_spining_joint}">
+           <command_interface name="velocity">
              <param name="min">-1</param>
              <param name="max">1</param>
            </command_interface>
            <state_interface name="position"/>
+           <state_interface name="velocity"/>
+           <state_interface name="effort"/>
          </joint>
-        <joint name="${front_right_wheel_spining_joint}">
-          <command_interface name="position">
+        <joint name="${prefix}${front_right_wheel_spining_joint}">
+          <command_interface name="velocity">
             <param name="min">-1</param>
             <param name="max">1</param>
           </command_interface>
           <state_interface name="position"/>
+          <state_interface name="velocity"/>
+          <state_interface name="effort"/>
+        </joint>
+        <joint name="${prefix}${rear_right_wheel_spining_joint}">
+          <command_interface name="velocity">
+            <param name="min">-1</param>
+            <param name="max">1</param>
+          </command_interface>
+          <state_interface name="position"/>
+          <state_interface name="velocity"/>
+          <state_interface name="effort"/>
         </joint>
         <joint name="${rear_right_wheel_spining_joint}">
@@ -42,11 +55,6 @@
           </command_interface>
           <state_interface name="position"/>
-        </joint>
-        <joint name="${rear_right_wheel_spining_joint}">
-          <command_interface name="position">
-            <param name="min">-1</param>
-            <param name="max">1</param>
-          </command_interface>
-          <state_interface name="position"/>
+          <state_interface name="velocity"/>
+          <state_interface name="effort"/>
         </joint>
     </ros2_control>

File: romea_mobile_base_description/ros2_control/2RWS_4WD.ros2_control.xacro (robot description, xacro)
@@ -15,5 +15,5 @@
           <state_interface name="position"/>
         </joint>
-        <joint name="${rear_right_wheel_steering_joint}">
+        <joint name="${prefix}${rear_right_wheel_steering_joint}">
           <command_interface name="position">
             <param name="min">-1</param>
@@ -22,5 +22,5 @@
           <state_interface name="position"/>
         </joint>
-         <joint name="${front_left_wheel_spining_joint}">
+         <joint name="${prefix}${front_left_wheel_spining_joint}">
            <command_interface name="position">
              <param name="min">-1</param>
@@ -28,6 +28,8 @@
            </command_interface>
            <state_interface name="position"/>
+           <state_interface name="velocity"/>
+           <state_interface name="effort"/>
          </joint>
-        <joint name="${front_right_wheel_spining_joint}">
+        <joint name="${prefix}${front_right_wheel_spining_joint}">
           <command_interface name="position">
             <param name="min">-1</param>
@@ -35,6 +37,8 @@
           </command_interface>
           <state_interface name="position"/>
+          <state_interface name="velocity"/>
+          <state_interface name="effort"/>
         </joint>
-        <joint name="${rear_right_wheel_spining_joint}">
+        <joint name="${prefix}${rear_right_wheel_spining_joint}">
           <command_interface name="position">
             <param name="min">-1</param>
@@ -42,6 +46,8 @@
           </command_interface>
           <state_interface name="position"/>
+          <state_interface name="velocity"/>
+          <state_interface name="effort"/>
         </joint>
-        <joint name="${rear_right_wheel_spining_joint}">
+        <joint name="${prefix}${rear_right_wheel_spining_joint}">
           <command_interface name="position">
             <param name="min">-1</param>
@@ -49,4 +55,6 @@
           </command_interface>
           <state_interface name="position"/>
+          <state_interface name="velocity"/>
+          <state_interface name="effort"/>
         </joint>
     </ros2_control>

File: romea_mobile_base_description/ros2_control/4WD.ros2_control.xacro (robot description, xacro)
@@ -13,5 +13,7 @@
              <param name="max">1</param>
            </command_interface>
+           <state_interface name="position"/>
            <state_interface name="velocity"/>
+           <state_interface name="effort"/>
          </joint>
         <joint name="${prefix}${front_right_wheel_spinning_joint}">
@@ -20,5 +22,7 @@
             <param name="max">1</param>
           </command_interface>
+          <state_interface name="position"/>
           <state_interface name="velocity"/>
+          <state_interface name="effort"/>
         </joint>
         <joint name="${prefix}${rear_left_wheel_spinning_joint}">
@@ -27,5 +31,7 @@
             <param name="max">1</param>
           </command_interface>
+          <state_interface name="position"/>
           <state_interface name="velocity"/>
+          <state_interface name="effort"/>
         </joint>
         <joint name="${prefix}${rear_right_wheel_spinning_joint}">
@@ -34,5 +40,7 @@
             <param name="max">1</param>
           </command_interface>
+          <state_interface name="position"/>
           <state_interface name="velocity"/>
+          <state_interface name="effort"/>
         </joint>
     </ros2_control>

Commit message: mobile base description : fix joint names in ros2_control.xacro files

File: romea_mobile_base_description/ros2_control/1FAS_4WD.ros2_control.xacro (robot description, xacro)
@@ -1,7 +1,7 @@
 <?xml version="1.0"?>
 <robot xmlns:xacro="http://www.ros.org/wiki/xacro">
-  <xacro:macro name="base_control" params="use_sim">
+  <xacro:macro name="base_control" params="use_sim:=true">
     <ros2_control name="${prefix}base" type="system">
-        <xacro:if value="$(arg use_sim)">
+        <xacro:if value="${use_sim}">
              <hardware>
                <plugin>gazebo_ros2_control/GazeboSystem</plugin>
@@ -47,5 +47,5 @@
           <state_interface name="effort"/>
         </joint>
-        <joint name="${prefix}${rear_right_wheel_spining_joint}">
+        <joint name="${prefix}${rear_left_wheel_spinning_joint}">
           <command_interface name="velocity">
             <param name="min">-1</param>
@@ -56,5 +56,5 @@
           <state_interface name="effort"/>
         </joint>
-        <joint name="${rear_right_wheel_spining_joint}">
+        <joint name="${rear_right_wheel_spinning_joint}">
           <command_interface name="position">
             <param name="min">-1</param>

File: romea_mobile_base_description/ros2_control/2FWS_4WD.ros2_control.xacro (robot description, xacro)
@@ -22,5 +22,5 @@
           <state_interface name="position"/>
         </joint>
-         <joint name="${prefix}${front_left_wheel_spining_joint}">
+         <joint name="${prefix}${front_left_wheel_spinning_joint}">
            <command_interface name="velocity">
              <param name="min">-1</param>
@@ -31,5 +31,5 @@
            <state_interface name="effort"/>
          </joint>
-        <joint name="${prefix}${front_right_wheel_spining_joint}">
+        <joint name="${prefix}${front_right_wheel_spinning_joint}">
           <command_interface name="velocity">
             <param name="min">-1</param>
@@ -40,5 +40,5 @@
           <state_interface name="effort"/>
         </joint>
-        <joint name="${prefix}${rear_right_wheel_spining_joint}">
+        <joint name="${prefix}${rear_right_wheel_spinning_joint}">
           <command_interface name="velocity">
             <param name="min">-1</param>
@@ -49,5 +49,5 @@
           <state_interface name="effort"/>
         </joint>
-        <joint name="${rear_right_wheel_spining_joint}">
+        <joint name="${prefix}${rear_right_wheel_spinning_joint}">
           <command_interface name="position">
             <param name="min">-1</param>

File: romea_mobile_base_description/ros2_control/2RWS_4WD.ros2_control.xacro (robot description, xacro)
@@ -1,9 +1,10 @@
 <?xml version="1.0"?>
 <robot xmlns:xacro="http://www.ros.org/wiki/xacro">
-  <xacro:macro name="base_control" params="use_sim">
+  <xacro:macro name="base_control" params="use_sim:=true">
     <ros2_control name="${prefix}base" type="system">
-        <xacro:if value="$(arg use_sim)">
+        <xacro:if value="${use_sim}">
             <hardware>
-              <plugin>gazebo_ros2_control/GazeboSystem</plugin>
+                <plugin>gazebo_ros2_control/GazeboSystem</plugin>
+<!--              <plugin>romea_mobile_base_gazebo/GazeboSystemInterfac2FWS4WD</plugin>-->
             </hardware>
         </xacro:if>

Commit message: update ros2_control vxacro to take account two different hardware plugin in simulation and in live

File: romea_mobile_base_description/ros2_control/1FAS_4WD.ros2_control.xacro (robot description, xacro)
@@ -1,11 +1,16 @@
 <?xml version="1.0"?>
 <robot xmlns:xacro="http://www.ros.org/wiki/xacro">
-  <xacro:macro name="base_control" params="use_sim:=true">
+   <xacro:macro name="base_control" params="mode">
     <ros2_control name="${prefix}base" type="system">
-        <xacro:if value="${use_sim}">
-             <hardware>
-               <plugin>gazebo_ros2_control/GazeboSystem</plugin>
-             </hardware>
-        </xacro:if>
+      <xacro:if value="${mode == 'live'}">
+          <hardware>
+            <plugin>${live_hardware_plugin}</plugin>
+          </hardware>
+      </xacro:if>
+       <xacro:if value="${mode == 'simulation'}">
+           <hardware>
+             <plugin>${simulation_hardware_plugin}</plugin>
+           </hardware>
+       </xacro:if>
        <joint name="${prefix}${front_axle_steering_joint}">
          <command_interface name="position">

File: romea_mobile_base_description/ros2_control/2AS_4WD.ros2_control.xacro (robot description, xacro)
@@ -1,11 +1,16 @@
 <?xml version="1.0"?>
 <robot xmlns:xacro="http://www.ros.org/wiki/xacro">
-  <xacro:macro name="base_control" params="use_sim">
+  <xacro:macro name="base_control" params="mode">
     <ros2_control name="${prefix}base" type="system">
-        <xacro:if value="$(arg use_sim)">
+        <xacro:if value="${mode == 'live'}">
             <hardware>
-              <plugin>gazebo_ros2_control/GazeboSystem</plugin>
+              <plugin>${live_hardware_plugin}</plugin>
             </hardware>
         </xacro:if>
+         <xacro:if value="${mode == 'simulation'}">
+             <hardware>
+               <plugin>${simulation_hardware_plugin}</plugin>
+             </hardware>
+         </xacro:if>
         <joint name="${prefix}${front_axle_steering_joint}">
           <command_interface name="position">

File: romea_mobile_base_description/ros2_control/2FWS_4WD.ros2_control.xacro (robot description, xacro)
@@ -1,10 +1,15 @@
 <?xml version="1.0"?>
 <robot xmlns:xacro="http://www.ros.org/wiki/xacro">
-  <xacro:macro name="base_control" params="use_sim">
+  <xacro:macro name="base_control" params="mode">
     <ros2_control name="${prefix}base" type="system">
-        <xacro:if value="$(arg use_sim)">
-             <hardware>
-               <plugin>gazebo_ros2_control/GazeboSystem</plugin>
-             </hardware>
+       <xacro:if value="${mode == 'live'}">
+           <hardware>
+             <plugin>${live_hardware_plugin}</plugin>
+           </hardware>
+       </xacro:if>
+        <xacro:if value="${mode == 'simulation'}">
+            <hardware>
+              <plugin>${simulation_hardware_plugin}</plugin>
+            </hardware>
         </xacro:if>
         <joint name="${prefix}${front_left_wheel_steering_joint}">

File: romea_mobile_base_description/ros2_control/2RWS_4WD.ros2_control.xacro (robot description, xacro)
@@ -1,10 +1,14 @@
 <?xml version="1.0"?>
 <robot xmlns:xacro="http://www.ros.org/wiki/xacro">
-  <xacro:macro name="base_control" params="use_sim:=true">
+  <xacro:macro name="base_control" params="mode">
     <ros2_control name="${prefix}base" type="system">
-        <xacro:if value="${use_sim}">
+       <xacro:if value="${mode == 'live'}">
+           <hardware>
+             <plugin>${live_hardware_plugin}</plugin>
+           </hardware>
+       </xacro:if>
+        <xacro:if value="${mode == 'simulation'}">
             <hardware>
-                <plugin>gazebo_ros2_control/GazeboSystem</plugin>
-<!--              <plugin>romea_mobile_base_gazebo/GazeboSystemInterfac2FWS4WD</plugin>-->
+              <plugin>${simulation_hardware_plugin}</plugin>
             </hardware>
         </xacro:if>

File: romea_mobile_base_description/ros2_control/2TD.ros2_control.xacro (robot description, xacro)
@@ -1,9 +1,14 @@
 <?xml version="1.0"?>
 <robot xmlns:xacro="http://www.ros.org/wiki/xacro">
-  <xacro:macro name="base_control" params="use_sim">
+  <xacro:macro name="base_control" params="mode">
     <ros2_control name="${prefix}base" type="system">
-        <xacro:if value="$(arg use_sim)">
+       <xacro:if value="${mode == 'live'}">
+           <hardware>
+             <plugin>${live_hardware_plugin}</plugin>
+           </hardware>
+       </xacro:if>
+        <xacro:if value="${mode == 'simulation'}">
             <hardware>
-              <plugin>gazebo_ros2_control/GazeboSystem</plugin>
+              <plugin>${simulation_hardware_plugin}</plugin>
             </hardware>
         </xacro:if>

File: romea_mobile_base_description/ros2_control/2THD.ros2_control.xacro (robot description, xacro)
@@ -1,9 +1,14 @@
 <?xml version="1.0"?>
 <robot xmlns:xacro="http://www.ros.org/wiki/xacro">
-  <xacro:macro name="base_control" params="use_sim">
+   <xacro:macro name="base_control" params="mode">
     <ros2_control name="${prefix}base" type="system">
-        <xacro:if value="$(arg use_sim)">
+       <xacro:if value="${mode == 'live'}">
+           <hardware>
+             <plugin>${live_hardware_plugin}</plugin>
+           </hardware>
+       </xacro:if>
+        <xacro:if value="${mode == 'simulation'}">
             <hardware>
-              <plugin>gazebo_ros2_control/GazeboSystem</plugin>
+              <plugin>${simulation_hardware_plugin}</plugin>
             </hardware>
         </xacro:if>

File: romea_mobile_base_description/ros2_control/2TTD.ros2_control.xacro (robot description, xacro)
@@ -1,11 +1,16 @@
 <?xml version="1.0"?>
 <robot xmlns:xacro="http://www.ros.org/wiki/xacro">
-  <xacro:macro name="base_control" params="use_sim">
+  <xacro:macro name="base_control" params="mode">
     <ros2_control name="${prefix}base" type="system">
-        <xacro:if value="$(arg use_sim)">
-            <hardware>
-              <plugin>gazebo_ros2_control/GazeboSystem</plugin>
-            </hardware>
-        </xacro:if>
+      <xacro:if value="${mode == 'live'}">
+          <hardware>
+            <plugin>${live_hardware_plugin}</plugin>
+          </hardware>
+      </xacro:if>
+       <xacro:if value="${mode == 'simulation'}">
+           <hardware>
+             <plugin>${simulation_hardware_plugin}</plugin>
+           </hardware>
+       </xacro:if>
         <joint name="${prefix}${high_left_sprocket_wheel_spinning_joint}">
           <command_interface name="velocity">

File: romea_mobile_base_description/ros2_control/4WD.ros2_control.xacro (robot description, xacro)
@@ -1,11 +1,15 @@
 <?xml version="1.0"?>
 <robot xmlns:xacro="http://www.ros.org/wiki/xacro">
-  <xacro:macro name="base_control" params="use_sim:=true">
+  <xacro:macro name="base_control" params="mode">
     <ros2_control name="${prefix}base" type="system">
-        <xacro:if value="${use_sim}">
+        <xacro:if value="${mode == 'live'}">
             <hardware>
-<!--              <plugin>gazebo_ros2_control/GazeboSystem</plugin>-->
-              <plugin>romea_mobile_base_gazebo/GazeboSystemInterface4WD</plugin>
+              <plugin>${live_hardware_plugin}</plugin>
             </hardware>
+        </xacro:if>
+         <xacro:if value="${mode == 'simulation'}">
+             <hardware>
+               <plugin>${simulation_hardware_plugin}</plugin>
+             </hardware>
          </xacro:if>
          <joint name="${prefix}${front_left_wheel_spinning_joint}">

File: romea_mobile_base_description/ros2_control/4WS_4WD.ros2_control.xacro (robot description, xacro)
@@ -1,10 +1,14 @@
 <?xml version="1.0"?>
 <robot xmlns:xacro="http://www.ros.org/wiki/xacro">
-  <xacro:macro name="base_control" params="use_sim:=true">
+  <xacro:macro name="base_control" params="mode">
     <ros2_control name="${prefix}base" type="system">
-        <xacro:if value="${use_sim}">
+       <xacro:if value="${mode == 'live'}">
+           <hardware>
+             <plugin>${live_hardware_plugin}</plugin>
+           </hardware>
+       </xacro:if>
+        <xacro:if value="${mode == 'simulation'}">
             <hardware>
-<!--              <plugin>gazebo_ros2_control/GazeboSystem</plugin>-->
-              <plugin>romea_mobile_base_gazebo/GazeboSystemInterface4WS4WD</plugin>
+              <plugin>${simulation_hardware_plugin}</plugin>
             </hardware>
         </xacro:if>
