Commit message: mobile base description : fix some errors in ros2 control xacro files

File: romea_mobile_base_description/ros2_control/1FAS_4WD.ros2_control.xacro (robot description, xacro)
@@ -21,15 +21,7 @@
        </joint>
         <joint name="${prefix}${front_left_wheel_steering_joint}">
-          <command_interface name="position">
-            <param name="min">-1</param>
-            <param name="max">1</param>
-          </command_interface>
           <state_interface name="position"/>
         </joint>
         <joint name="${prefix}${front_right_wheel_steering_joint}">
-          <command_interface name="position">
-            <param name="min">-1</param>
-            <param name="max">1</param>
-          </command_interface>
           <state_interface name="position"/>
         </joint>

File: romea_mobile_base_description/ros2_control/2AS_4WD.ros2_control.xacro (robot description, xacro)
@@ -11,4 +11,7 @@
              <hardware>
                <plugin>${simulation_hardware_plugin}</plugin>
+               <param name="wheelbase">${wheelbase}</param>
+               <param name="front_track">${front_track}</param>
+               <param name="rear_track">${rear_track}</param>
              </hardware>
          </xacro:if>
@@ -28,33 +31,17 @@
        </joint>
         <joint name="${prefix}${front_left_wheel_steering_joint}">
-          <command_interface name="position">
-            <param name="min">-1</param>
-            <param name="max">1</param>
-          </command_interface>
           <state_interface name="position"/>
         </joint>
         <joint name="${prefix}${front_right_wheel_steering_joint}">
-          <command_interface name="position">
-            <param name="min">-1</param>
-            <param name="max">1</param>
-          </command_interface>
           <state_interface name="position"/>
         </joint>
         <joint name="${prefix}${rear_left_wheel_steering_joint}">
-          <command_interface name="position">
-            <param name="min">-1</param>
-            <param name="max">1</param>
-          </command_interface>
           <state_interface name="position"/>
         </joint>
         <joint name="${prefix}${rear_right_wheel_steering_joint}">
-          <command_interface name="position">
-            <param name="min">-1</param>
-            <param name="max">1</param>
-          </command_interface>
           <state_interface name="position"/>
         </joint>
          <joint name="${prefix}${front_left_wheel_spinning_joint}">
-           <command_interface name="position">
+           <command_interface name="velocity">
              <param name="min">-1</param>
              <param name="max">1</param>
@@ -65,5 +52,14 @@
          </joint>
         <joint name="${prefix}${front_right_wheel_spinning_joint}">
-          <command_interface name="position">
+          <command_interface name="velocity">
+            <param name="min">-1</param>
+            <param name="max">1</param>
+          </command_interface>
+          <state_interface name="position"/>
+          <state_interface name="velocity"/>
+          <state_interface name="effort"/>
+        </joint>
+        <joint name="${prefix}${rear_left_wheel_spinning_joint}">
+          <command_interface name="velocity">
             <param name="min">-1</param>
             <param name="max">1</param>
@@ -74,14 +70,5 @@
         </joint>
         <joint name="${prefix}${rear_right_wheel_spinning_joint}">
-          <command_interface name="position">
-            <param name="min">-1</param>
-            <param name="max">1</param>
-          </command_interface>
-          <state_interface name="position"/>
-          <state_interface name="velocity"/>
-          <state_interface name="effort"/>
-        </joint>
-        <joint name="${prefix}${rear_right_wheel_spinning_joint}">
-          <command_interface name="position">
+          <command_interface name="velocity">
             <param name="min">-1</param>
             <param name="max">1</param>

File: romea_mobile_base_description/ros2_control/2FWS_4WD.ros2_control.xacro (robot description, xacro)
@@ -1,3 +1,3 @@
-<?xml version="1.0"?>
+ <?xml version="1.0"?>
 <robot xmlns:xacro="http://www.ros.org/wiki/xacro">
   <xacro:macro name="base_control" params="mode">

File: romea_mobile_base_description/ros2_control/2THD.ros2_control.xacro (robot description, xacro)
@@ -13,5 +13,5 @@
             </hardware>
         </xacro:if>
-        <joint name="${prefix}${high_left_sprocket_wheel_spinning_joint}">
+        <joint name="${prefix}${left_sprocket_wheel_spinning_joint}">
           <command_interface name="velocity">
             <param name="min">-1</param>
@@ -22,5 +22,5 @@
           <state_interface name="effort"/>
         </joint>
-        <joint name="${prefix}${high_right_sprocket_wheel_spinning_joint}">
+        <joint name="${prefix}${right_sprocket_wheel_spinning_joint}">
           <command_interface name="velocity">
             <param name="min">-1</param>

File: romea_mobile_base_description/ros2_control/2TTD.ros2_control.xacro (robot description, xacro)
@@ -13,5 +13,5 @@
            </hardware>
        </xacro:if>
-        <joint name="${prefix}${high_left_sprocket_wheel_spinning_joint}">
+        <joint name="${prefix}${left_sprocket_wheel_spinning_joint}">
           <command_interface name="velocity">
             <param name="min">-1</param>
@@ -22,5 +22,5 @@
           <state_interface name="effort"/>
         </joint>
-        <joint name="${prefix}${high_right_sprocket_wheel_spinning_joint}">
+        <joint name="${prefix}${right_sprocket_wheel_spinning_joint}">
           <command_interface name="velocity">
             <param name="min">-1</param>

File: romea_mobile_base_description/urdf/axle_steering.xacro (robot description, xacro)
@@ -2,5 +2,13 @@
 <robot xmlns:xacro="http://www.ros.org/wiki/xacro" name="axle_steering">
   <xacro:macro name="axle_steering" params="parent_link axle_steering_link axle_steering_joint *joint_origin">
-    <link name="${prefix}${axle_steering_link}"/>
+    <link name="${prefix}${axle_steering_link}">
+      <inertial>
+        <mass value="${steering_link_mass}" />
+        <origin xyz="0 0 0" />
+        <inertia  ixx="${steering_link_mass/12.0 * (steering_link_y*steering_link_y + steering_link_xz*steering_link_xz)}" ixy="0" ixz="0"
+                  iyy="${steering_link_mass/12.0 * (steering_link_xz*steering_link_xz + steering_link_xz*steering_link_xz)}" iyz="0"
+                  izz="${steering_link_mass/12.0 * (steering_link_y*steering_link_y + steering_link_xz*steering_link_xz)}" />
+      </inertial>
+   </link>
     <joint name="${prefix}${axle_steering_joint}" type="revolute">
       <limit lower="${minimal_axle_steering_angle}" upper="${maximal_axle_steering_angle}" effort="10000000" velocity="1000000"/>
@@ -10,4 +18,13 @@
       <axis xyz="0 0 1" rpy="0 0 0" />
     </joint>
+   <transmission name="${prefix}${axle_steering_joint}_trans" type="SimpleTransmission">
+     <type>transmission_interface/SimpleTransmission</type>
+     <actuator name="${prefix}${axle_steering_joint}_motor">
+       <mechanicalReduction>1</mechanicalReduction>
+     </actuator>
+     <joint name="${prefix}${axle_steering_joint}">
+       <hardwareInterface>hardware_interface/PositionJointInterface</hardwareInterface>
+     </joint>
+   </transmission>
   </xacro:macro>
 </robot>
