Commit message: mobile_base_description : add ros2_control xacro file for 1FAS_2FWD, 1FAS_2RWD, 1FWS_2FWD, 2FWS_2FWD and 2FWS_2RWD vehicles

File: romea_mobile_base_description/ros2_control/1FAS_2FWD.ros2_control.xacro (robot description, xacro)
@@ -1,32 +1,31 @@
 <?xml version="1.0"?>
 <robot xmlns:xacro="http://www.ros.org/wiki/xacro">
-  <xacro:macro name="base_control" params="mode">
+   <xacro:macro name="base_control" params="mode">
     <ros2_control name="${prefix}base" type="system">
-       <xacro:if value="${mode == 'live'}">
+      <xacro:if value="${mode == 'live'}">
+          <hardware>
+            <plugin>${live_hardware_plugin}</plugin>
+          </hardware>
+      </xacro:if>
+       <xacro:if value="${mode == 'simulation'}">
            <hardware>
-             <plugin>${live_hardware_plugin}</plugin>
+             <plugin>${simulation_hardware_plugin}</plugin>
            </hardware>
        </xacro:if>
-        <xacro:if value="${mode == 'simulation'}">
-            <hardware>
-              <plugin>${simulation_hardware_plugin}</plugin>
-            </hardware>
-        </xacro:if>
-        <joint name="${prefix}${rear_left_wheel_steering_joint}">
-          <command_interface name="position">
-            <param name="min">-1</param>
-            <param name="max">1</param>
-          </command_interface>
+       <joint name="${prefix}${front_axle_steering_joint}">
+         <command_interface name="position">
+           <param name="min">-1</param>
+           <param name="max">1</param>
+         </command_interface>
+         <state_interface name="position"/>
+       </joint>
+        <joint name="${prefix}${front_left_wheel_steering_joint}">
           <state_interface name="position"/>
         </joint>
-        <joint name="${prefix}${rear_right_wheel_steering_joint}">
-          <command_interface name="position">
-            <param name="min">-1</param>
-            <param name="max">1</param>
-          </command_interface>
+        <joint name="${prefix}${front_right_wheel_steering_joint}">
           <state_interface name="position"/>
         </joint>
          <joint name="${prefix}${front_left_wheel_spinning_joint}">
-           <command_interface name="position">
+           <command_interface name="velocity">
              <param name="min">-1</param>
              <param name="max">1</param>
@@ -37,5 +36,5 @@
          </joint>
         <joint name="${prefix}${front_right_wheel_spinning_joint}">
-          <command_interface name="position">
+          <command_interface name="velocity">
             <param name="min">-1</param>
             <param name="max">1</param>
@@ -45,9 +44,5 @@
           <state_interface name="effort"/>
         </joint>
-        <joint name="${prefix}${rear_right_wheel_spinning_joint}">
-          <command_interface name="position">
-            <param name="min">-1</param>
-            <param name="max">1</param>
-          </command_interface>
+        <joint name="${prefix}${rear_left_wheel_spinning_joint}">
           <state_interface name="position"/>
           <state_interface name="velocity"/>
@@ -55,8 +50,4 @@
         </joint>
         <joint name="${prefix}${rear_right_wheel_spinning_joint}">
-          <command_interface name="position">
-            <param name="min">-1</param>
-            <param name="max">1</param>
-          </command_interface>
           <state_interface name="position"/>
           <state_interface name="velocity"/>

File: romea_mobile_base_description/ros2_control/1FAS_2RWD.ros2_control.xacro (robot description, xacro)
@@ -1,35 +1,30 @@
 <?xml version="1.0"?>
 <robot xmlns:xacro="http://www.ros.org/wiki/xacro">
-  <xacro:macro name="base_control" params="mode">
+   <xacro:macro name="base_control" params="mode">
     <ros2_control name="${prefix}base" type="system">
-       <xacro:if value="${mode == 'live'}">
+      <xacro:if value="${mode == 'live'}">
+          <hardware>
+            <plugin>${live_hardware_plugin}</plugin>
+          </hardware>
+      </xacro:if>
+       <xacro:if value="${mode == 'simulation'}">
            <hardware>
-             <plugin>${live_hardware_plugin}</plugin>
+             <plugin>${simulation_hardware_plugin}</plugin>
            </hardware>
        </xacro:if>
-        <xacro:if value="${mode == 'simulation'}">
-            <hardware>
-              <plugin>${simulation_hardware_plugin}</plugin>
-            </hardware>
-        </xacro:if>
-        <joint name="${prefix}${rear_left_wheel_steering_joint}">
-          <command_interface name="position">
-            <param name="min">-1</param>
-            <param name="max">1</param>
-          </command_interface>
+       <joint name="${prefix}${front_axle_steering_joint}">
+         <command_interface name="position">
+           <param name="min">-1</param>
+           <param name="max">1</param>
+         </command_interface>
+         <state_interface name="position"/>
+       </joint>
+        <joint name="${prefix}${front_left_wheel_steering_joint}">
           <state_interface name="position"/>
         </joint>
-        <joint name="${prefix}${rear_right_wheel_steering_joint}">
-          <command_interface name="position">
-            <param name="min">-1</param>
-            <param name="max">1</param>
-          </command_interface>
+        <joint name="${prefix}${front_right_wheel_steering_joint}">
           <state_interface name="position"/>
         </joint>
          <joint name="${prefix}${front_left_wheel_spinning_joint}">
-           <command_interface name="position">
-             <param name="min">-1</param>
-             <param name="max">1</param>
-           </command_interface>
            <state_interface name="position"/>
            <state_interface name="velocity"/>
@@ -37,5 +32,10 @@
          </joint>
         <joint name="${prefix}${front_right_wheel_spinning_joint}">
-          <command_interface name="position">
+          <state_interface name="position"/>
+          <state_interface name="velocity"/>
+          <state_interface name="effort"/>
+        </joint>
+        <joint name="${prefix}${rear_left_wheel_spinning_joint}">
+          <command_interface name="velocity">
             <param name="min">-1</param>
             <param name="max">1</param>
@@ -46,14 +46,5 @@
         </joint>
         <joint name="${prefix}${rear_right_wheel_spinning_joint}">
-          <command_interface name="position">
-            <param name="min">-1</param>
-            <param name="max">1</param>
-          </command_interface>
-          <state_interface name="position"/>
-          <state_interface name="velocity"/>
-          <state_interface name="effort"/>
-        </joint>
-        <joint name="${prefix}${rear_right_wheel_spinning_joint}">
-          <command_interface name="position">
+          <command_interface name="velocity">
             <param name="min">-1</param>
             <param name="max">1</param>

File: romea_mobile_base_description/ros2_control/1FWS_2RWD.ros2_control.xacro (robot description, xacro)
@@ -13,5 +13,5 @@
            </hardware>
        </xacro:if>
-       <joint name="${prefix}${front_axle_steering_joint}">
+       <joint name="${prefix}${front_wheel_steering_joint}">
          <command_interface name="position">
            <param name="min">-1</param>
@@ -20,28 +20,9 @@
          <state_interface name="position"/>
        </joint>
-        <joint name="${prefix}${front_left_wheel_steering_joint}">
-          <state_interface name="position"/>
-        </joint>
-        <joint name="${prefix}${front_right_wheel_steering_joint}">
-          <state_interface name="position"/>
-        </joint>
-         <joint name="${prefix}${front_left_wheel_spinning_joint}">
-           <command_interface name="velocity">
-             <param name="min">-1</param>
-             <param name="max">1</param>
-           </command_interface>
-           <state_interface name="position"/>
-           <state_interface name="velocity"/>
-           <state_interface name="effort"/>
-         </joint>
-        <joint name="${prefix}${front_right_wheel_spinning_joint}">
-          <command_interface name="velocity">
-            <param name="min">-1</param>
-            <param name="max">1</param>
-          </command_interface>
-          <state_interface name="position"/>
-          <state_interface name="velocity"/>
-          <state_interface name="effort"/>
-        </joint>
+      <joint name="${prefix}${front_wheel_spinning_joint}">
+         <state_interface name="position"/>
+         <state_interface name="velocity"/>
+         <state_interface name="effort"/>
+      </joint>
         <joint name="${prefix}${rear_left_wheel_spinning_joint}">
           <command_interface name="velocity">

File: romea_mobile_base_description/ros2_control/2FWS_2FWD.ros2_control.xacro (robot description, xacro)
@@ -13,5 +13,5 @@
             </hardware>
         </xacro:if>
-        <joint name="${prefix}${rear_left_wheel_steering_joint}">
+        <joint name="${prefix}${front_left_wheel_steering_joint}">
           <command_interface name="position">
             <param name="min">-1</param>
@@ -20,5 +20,5 @@
           <state_interface name="position"/>
         </joint>
-        <joint name="${prefix}${rear_right_wheel_steering_joint}">
+        <joint name="${prefix}${front_right_wheel_steering_joint}">
           <command_interface name="position">
             <param name="min">-1</param>
@@ -28,5 +28,5 @@
         </joint>
          <joint name="${prefix}${front_left_wheel_spinning_joint}">
-           <command_interface name="position">
+           <command_interface name="velocity">
              <param name="min">-1</param>
              <param name="max">1</param>
@@ -37,5 +37,5 @@
          </joint>
         <joint name="${prefix}${front_right_wheel_spinning_joint}">
-          <command_interface name="position">
+          <command_interface name="velocity">
             <param name="min">-1</param>
             <param name="max">1</param>
@@ -45,9 +45,5 @@
           <state_interface name="effort"/>
         </joint>
-        <joint name="${prefix}${rear_right_wheel_spinning_joint}">
-          <command_interface name="position">
-            <param name="min">-1</param>
-            <param name="max">1</param>
-          </command_interface>
+        <joint name="${prefix}${rear_left_wheel_spinning_joint}">
           <state_interface name="position"/>
           <state_interface name="velocity"/>
@@ -55,8 +51,4 @@
         </joint>
         <joint name="${prefix}${rear_right_wheel_spinning_joint}">
-          <command_interface name="position">
-            <param name="min">-1</param>
-            <param name="max">1</param>
-          </command_interface>
           <state_interface name="position"/>
           <state_interface name="velocity"/>

File: romea_mobile_base_description/ros2_control/2FWS_2RWD.ros2_control.xacro (robot description, xacro)
@@ -13,5 +13,5 @@
             </hardware>
         </xacro:if>
-        <joint name="${prefix}${rear_left_wheel_steering_joint}">
+        <joint name="${prefix}${front_left_wheel_steering_joint}">
           <command_interface name="position">
             <param name="min">-1</param>
@@ -20,5 +20,5 @@
           <state_interface name="position"/>
         </joint>
-        <joint name="${prefix}${rear_right_wheel_steering_joint}">
+        <joint name="${prefix}${front_right_wheel_steering_joint}">
           <command_interface name="position">
             <param name="min">-1</param>
@@ -28,8 +28,4 @@
         </joint>
          <joint name="${prefix}${front_left_wheel_spinning_joint}">
-           <command_interface name="position">
-             <param name="min">-1</param>
-             <param name="max">1</param>
-           </command_interface>
            <state_interface name="position"/>
            <state_interface name="velocity"/>
@@ -37,5 +33,10 @@
          </joint>
         <joint name="${prefix}${front_right_wheel_spinning_joint}">
-          <command_interface name="position">
+          <state_interface name="position"/>
+          <state_interface name="velocity"/>
+          <state_interface name="effort"/>
+        </joint>
+        <joint name="${prefix}${rear_left_wheel_spinning_joint}">
+          <command_interface name="velocity">
             <param name="min">-1</param>
             <param name="max">1</param>
@@ -46,14 +47,5 @@
         </joint>
         <joint name="${prefix}${rear_right_wheel_spinning_joint}">
-          <command_interface name="position">
-            <param name="min">-1</param>
-            <param name="max">1</param>
-          </command_interface>
-          <state_interface name="position"/>
-          <state_interface name="velocity"/>
-          <state_interface name="effort"/>
-        </joint>
-        <joint name="${prefix}${rear_right_wheel_spinning_joint}">
-          <command_interface name="position">
+          <command_interface name="velocity">
             <param name="min">-1</param>
             <param name="max">1</param>

File: romea_mobile_base_description/ros2_control/2FWS_4WD.ros2_control.xacro (robot description, xacro)
@@ -1,3 +1,3 @@
- <?xml version="1.0"?>
+<?xml version="1.0"?>
 <robot xmlns:xacro="http://www.ros.org/wiki/xacro">
   <xacro:macro name="base_control" params="mode">
@@ -45,5 +45,5 @@
           <state_interface name="effort"/>
         </joint>
-        <joint name="${prefix}${rear_right_wheel_spinning_joint}">
+        <joint name="${prefix}${rear_left_wheel_spinning_joint}">
           <command_interface name="velocity">
             <param name="min">-1</param>
@@ -55,5 +55,5 @@
         </joint>
         <joint name="${prefix}${rear_right_wheel_spinning_joint}">
-          <command_interface name="position">
+          <command_interface name="velocity">
             <param name="min">-1</param>
             <param name="max">1</param>

File: romea_mobile_base_description/ros2_control/2TD.ros2_control.xacro (robot description, xacro)
@@ -32,8 +32,4 @@
         </joint>
          <joint name="${prefix}${left_idler_wheel_spinning_joint}">
-           <command_interface name="velocity">
-             <param name="min">-1</param>
-             <param name="max">1</param>
-           </command_interface>
            <state_interface name="position"/>
            <state_interface name="velocity"/>
@@ -41,8 +37,4 @@
          </joint>
         <joint name="${prefix}${right_idler_wheel_spinning_joint}">
-          <command_interface name="velocity">
-            <param name="min">-1</param>
-            <param name="max">1</param>
-          </command_interface>
           <state_interface name="position"/>
           <state_interface name="velocity"/>

File: romea_mobile_base_description/urdf/1RAS_4WD_chassis.xacro (robot description, xacro)
@@ -14,5 +14,5 @@
     <xacro:wheel parent_link="base_link"
                  wheel_spinning_link="${front_left_wheel_spinning_link}"
-                 wheel_spinning_joint="${front_left_wheel_spining_joint}"
+                 wheel_spinning_joint="${front_left_wheel_spinning_joint}"
                  wheel_origin_y="${front_wheel_y_offset}"
                  wheel_mass="${front_wheel_mass}"
@@ -26,5 +26,5 @@
      <xacro:wheel parent_link="base_link"
                   wheel_spinning_link="${front_right_wheel_spinning_link}"
-                  wheel_spinning_joint="${front_right_wheel_spining_joint}"
+                  wheel_spinning_joint="${front_right_wheel_spinning_joint}"
                   wheel_origin_y="${-front_wheel_y_offset}"
                   wheel_mass="${front_wheel_mass}"
@@ -40,5 +40,5 @@
                           wheel_steering_joint="${rear_left_wheel_steering_joint}"
                           wheel_spinning_link="${rear_left_wheel_spinning_link}"
-                          wheel_spinning_joint="${rear_left_wheel_spining_joint}"
+                          wheel_spinning_joint="${rear_left_wheel_spinning_joint}"
                           wheel_origin_y="${rear_wheel_y_offset}"
                           wheel_mass="${rear_wheel_mass}"
@@ -54,5 +54,5 @@
                          wheel_steering_joint="${rear_right_wheel_steering_joint}"
                          wheel_spinning_link="${rear_right_wheel_spinning_link}"
-                         wheel_spinning_joint="${rear_right_wheel_spining_joint}"
+                         wheel_spinning_joint="${rear_right_wheel_spinning_joint}"
                          wheel_origin_y="${-rear_wheel_y_offset}"
                          wheel_mass="${rear_wheel_mass}"

File: romea_mobile_base_description/urdf/2RWS_4WD_chassis.xacro (robot description, xacro)
@@ -9,5 +9,5 @@
     <xacro:wheel parent_link="base_link"
                  wheel_spinning_link="${front_left_wheel_spinning_link}"
-                 wheel_spinning_joint="${front_left_wheel_spining_joint}"
+                 wheel_spinning_joint="${front_left_wheel_spinning_joint}"
                  wheel_origin_y="${front_wheel_y_offset}"
                  wheel_mass="${front_wheel_mass}"
@@ -21,5 +21,5 @@
      <xacro:wheel parent_link="base_link"
                   wheel_spinning_link="${front_right_wheel_spinning_link}"
-                  wheel_spinning_joint="${front_right_wheel_spining_joint}"
+                  wheel_spinning_joint="${front_right_wheel_spinning_joint}"
                   wheel_origin_y="${-front_wheel_y_offset}"
                   wheel_mass="${front_wheel_mass}"
@@ -35,5 +35,5 @@
                           wheel_steering_joint="${rear_left_wheel_steering_joint}"
                           wheel_spinning_link="${rear_left_wheel_spinning_link}"
-                          wheel_spinning_joint="${rear_left_wheel_spining_joint}"
+                          wheel_spinning_joint="${rear_left_wheel_spinning_joint}"
                           wheel_origin_y="${rear_wheel_y_offset}"
                           wheel_mass="${rear_wheel_mass}"
@@ -49,5 +49,5 @@
                          wheel_steering_joint="${rear_right_wheel_steering_joint}"
                          wheel_spinning_link="${rear_right_wheel_spinning_link}"
-                         wheel_spinning_joint="${rear_right_wheel_spining_joint}"
+                         wheel_spinning_joint="${rear_right_wheel_spinning_joint}"
                          wheel_origin_y="${-rear_wheel_y_offset}"
                          wheel_mass="${rear_wheel_mass}"
