Commit message: add support of generic hardware and simulation interface for all kind of robots
Signed-off-by: jean.laneurit <jean.laneurit@inrae.fr>

File: romea_mobile_base_description/ros2_control/base1FAS4WD.ros2_control.xacro (robot description, xacro)
@@ -9,5 +9,4 @@
           <param name="front_track">${front_track}</param>
           <param name="front_wheel_radius">${front_wheel_radius}</param>
-          <param name="front_hub_carrier_offset">${front_hub_carrier_offset}</param>
           <param name="rear_wheel_radius">${rear_wheel_radius}</param>
         </hardware>
@@ -19,5 +18,4 @@
           <param name="front_track">${front_track}</param>
           <param name="front_wheel_radius">${front_wheel_radius}</param>
-          <param name="front_hub_carrier_offset">${front_hub_carrier_offset}</param>
           <param name="rear_wheel_radius">${rear_wheel_radius}</param>
         </hardware>

File: romea_mobile_base_description/ros2_control/base2AS2FWD.ros2_control.xacro (robot description, xacro)
@@ -9,6 +9,8 @@
           <param name="front_track">${front_track}</param>
           <param name="front_wheel_radius">${front_wheel_radius}</param>
+          <param name="front_hub_carrier_offset">${front_hub_carrier_offset}</param>
           <param name="rear_track">${rear_track}</param>
           <param name="rear_wheel_radius">${rear_wheel_radius}</param>
+          <param name="rear_hub_carrier_offset">${rear_hub_carrier_offset}</param>
         </hardware>
       </xacro:if>
@@ -19,6 +21,8 @@
           <param name="front_track">${front_track}</param>
           <param name="front_wheel_radius">${front_wheel_radius}</param>
+          <param name="front_hub_carrier_offset">${front_hub_carrier_offset}</param>
           <param name="rear_track">${rear_track}</param>
           <param name="rear_wheel_radius">${rear_wheel_radius}</param>
+          <param name="rear_hub_carrier_offset">${rear_hub_carrier_offset}</param>
         </hardware>
       </xacro:if>

File: romea_mobile_base_description/ros2_control/base2AS2RWD.ros2_control.xacro (robot description, xacro)
@@ -8,7 +8,9 @@
           <param name="wheelbase">${wheelbase}</param>
           <param name="front_track">${front_track}</param>
+          <param name="front_wheel_radius">${front_wheel_radius}</param>
+          <param name="front_hub_carrier_offset">${front_hub_carrier_offset}</param>
           <param name="rear_track">${rear_track}</param>
-          <param name="front_wheel_radius">${front_wheel_radius}</param>
           <param name="rear_wheel_radius">${rear_wheel_radius}</param>
+          <param name="rear_hub_carrier_offset">${rear_hub_carrier_offset}</param>
         </hardware>
       </xacro:if>
@@ -18,5 +20,9 @@
           <param name="wheelbase">${wheelbase}</param>
           <param name="front_track">${front_track}</param>
+          <param name="front_wheel_radius">${front_wheel_radius}</param>
+          <param name="front_hub_carrier_offset">${front_hub_carrier_offset}</param>
           <param name="rear_track">${rear_track}</param>
+          <param name="rear_wheel_radius">${rear_wheel_radius}</param>
+          <param name="rear_hub_carrier_offset">${rear_hub_carrier_offset}</param>
         </hardware>
       </xacro:if>

File: romea_mobile_base_description/ros2_control/base2AS4WD.ros2_control.xacro (robot description, xacro)
@@ -19,4 +19,6 @@
           <param name="front_track">${front_track}</param>
           <param name="rear_track">${rear_track}</param>
+          <param name="front_wheel_radius">${front_wheel_radius}</param>
+          <param name="rear_wheel_radius">${rear_wheel_radius}</param>
         </hardware>
       </xacro:if>

File: romea_mobile_base_description/ros2_control/base2FWS4WD.ros2_control.xacro (robot description, xacro)
@@ -9,5 +9,4 @@
           <param name="front_track">${front_track}</param>
           <param name="front_wheel_radius">${front_wheel_radius}</param>
-          <param name="front_hub_carrier_offset">${front_hub_carrier_offset}</param>
           <param name="rear_track">${rear_track}</param>
           <param name="rear_wheel_radius">${rear_wheel_radius}</param>
@@ -20,5 +19,4 @@
           <param name="front_track">${front_track}</param>
           <param name="front_wheel_radius">${front_wheel_radius}</param>
-          <param name="front_hub_carrier_offset">${front_hub_carrier_offset}</param>
           <param name="rear_track">${rear_track}</param>
           <param name="rear_wheel_radius">${rear_wheel_radius}</param>

File: romea_mobile_base_hardware/test/test_hardware_interface1FAS2FWD.xacro (robot description, xacro)
@@ -9,11 +9,17 @@
   <xacro:property name="rear_left_wheel_spinning_joint" value="joint6" />
   <xacro:property name="rear_right_wheel_spinning_joint" value="joint7" />
-  <xacro:property name="rear_right_wheel_spinning_joint" value="joint7" />
-  <xacro:property name="rear_right_wheel_spinning_joint" value="joint7" />
-  <xacro:property name="front_wheel_radius" value="0.2" />
-  <xacro:property name="maximal_axle_steering_angle" value="0.5" />
+  <xacro:property name="live_hardware_plugin" value="foo" />
+  <xacro:property name="wheelbase" value="1.4" />
+  <xacro:property name="front_track" value="1.2" />
+  <xacro:property name="front_wheel_radius" value="0.4" />
+  <xacro:property name="front_hub_carrier_offset" value="0.1" />
+  <xacro:property name="rear_track" value="1.4" />
+  <xacro:property name="rear_wheel_radius" value="0.6" />
+  <xacro:property name="rear_hub_carrier_offset" value="0.15" />
+  <xacro:property name="maximal_axle_steering_angle" value="0.50" />
+  <xacro:property name="maximal_wheel_steering_angle" value="1.00" />
   <xacro:property name="maximal_wheel_speed" value="1.0" />
   <xacro:include
     filename="$(find romea_mobile_base_description)/ros2_control/base1FAS2FWD.ros2_control.xacro" />
-  <xacro:base_control mode="test" base_name="base" />
+  <xacro:base_control mode="live" base_name="base" />
 </robot>

File: romea_mobile_base_hardware/test/test_hardware_interface1FAS2RWD.xacro (robot description, xacro)
@@ -9,9 +9,15 @@
   <xacro:property name="front_left_wheel_spinning_joint" value="joint6" />
   <xacro:property name="front_right_wheel_spinning_joint" value="joint7" />
-  <xacro:property name="rear_wheel_radius" value="0.2" />
-  <xacro:property name="maximal_axle_steering_angle" value="0.5" />
+  <xacro:property name="live_hardware_plugin" value="foo" />
+  <xacro:property name="wheelbase" value="1.3" />
+  <xacro:property name="front_track" value="0.8" />
+  <xacro:property name="front_wheel_radius" value="0.3" />
+  <xacro:property name="front_hub_carrier_offset" value="0.08" />
+  <xacro:property name="rear_wheel_radius" value="0.7" />
+  <xacro:property name="maximal_axle_steering_angle" value="0.50" />
+  <xacro:property name="maximal_wheel_steering_angle" value="1.00" />
   <xacro:property name="maximal_wheel_speed" value="1.0" />
   <xacro:include
     filename="$(find romea_mobile_base_description)/ros2_control/base1FAS2RWD.ros2_control.xacro" />
-  <xacro:base_control mode="test" base_name="base" />
+  <xacro:base_control mode="live" base_name="base" />
 </robot>

File: romea_mobile_base_hardware/test/test_hardware_interface1FAS4WD.xacro (robot description, xacro)
@@ -9,10 +9,13 @@
   <xacro:property name="front_left_wheel_steering_joint" value="joint6" />
   <xacro:property name="front_right_wheel_steering_joint" value="joint7" />
-  <xacro:property name="rear_wheel_radius" value="0.2" />
-  <xacro:property name="front_wheel_radius" value="0.2" />
+  <xacro:property name="live_hardware_plugin" value="foo" />
+  <xacro:property name="wheelbase" value="1.4" />
+  <xacro:property name="front_track" value="1.2" />
+  <xacro:property name="front_wheel_radius" value="0.4" />
+  <xacro:property name="rear_wheel_radius" value="0.6" />
   <xacro:property name="maximal_axle_steering_angle" value="0.5" />
   <xacro:property name="maximal_wheel_speed" value="1.0" />
   <xacro:include
     filename="$(find romea_mobile_base_description)/ros2_control/base1FAS4WD.ros2_control.xacro" />
-  <xacro:base_control mode="test" base_name="base" />
+  <xacro:base_control mode="live" base_name="base" />
 </robot>

File: romea_mobile_base_hardware/test/test_hardware_interface2AS2FWD.xacro (robot description, xacro)
@@ -12,9 +12,17 @@
   <xacro:property name="rear_left_wheel_spinning_joint" value="joint9" />
   <xacro:property name="rear_right_wheel_spinning_joint" value="joint10" />
-  <xacro:property name="front_wheel_radius" value="0.2" />
+  <xacro:property name="live_hardware_plugin" value="foo" />
+  <xacro:property name="wheelbase" value="1.3" />
+  <xacro:property name="front_track" value="1.2" />
+  <xacro:property name="front_wheel_radius" value="0.4" />
+  <xacro:property name="front_hub_carrier_offset" value="0.1" />
+  <xacro:property name="rear_track" value="1.2" />
+  <xacro:property name="rear_wheel_radius" value="0.6" />
+  <xacro:property name="rear_hub_carrier_offset" value="0.1" />
   <xacro:property name="maximal_axle_steering_angle" value="0.5" />
+  <xacro:property name="maximal_wheel_steering_angle" value="1.0" />
   <xacro:property name="maximal_wheel_speed" value="1.0" />
   <xacro:include
     filename="$(find romea_mobile_base_description)/ros2_control/base2AS2FWD.ros2_control.xacro" />
-  <xacro:base_control mode="test" base_name="base" />
+  <xacro:base_control mode="live" base_name="base" />
 </robot>

File: romea_mobile_base_hardware/test/test_hardware_interface2AS2RWD.xacro (robot description, xacro)
@@ -15,6 +15,17 @@
   <xacro:property name="maximal_axle_steering_angle" value="0.5" />
   <xacro:property name="maximal_wheel_speed" value="1.0" />
+  <xacro:property name="live_hardware_plugin" value="foo" />
+  <xacro:property name="wheelbase" value="1.3" />
+  <xacro:property name="front_track" value="1.2" />
+  <xacro:property name="front_wheel_radius" value="0.4" />
+  <xacro:property name="front_hub_carrier_offset" value="0.1" />
+  <xacro:property name="rear_track" value="1.2" />
+  <xacro:property name="rear_wheel_radius" value="0.6" />
+  <xacro:property name="rear_hub_carrier_offset" value="0.1" />
+  <xacro:property name="maximal_axle_steering_angle" value="0.5" />
+  <xacro:property name="maximal_wheel_steering_angle" value="1.0" />
+  <xacro:property name="maximal_wheel_speed" value="1.0" />
   <xacro:include
     filename="$(find romea_mobile_base_description)/ros2_control/base2AS2RWD.ros2_control.xacro" />
-  <xacro:base_control mode="test" base_name="base" />
+  <xacro:base_control mode="live" base_name="base" />
 </robot>

File: romea_mobile_base_hardware/test/test_hardware_interface2AS4WD.xacro (robot description, xacro)
@@ -12,10 +12,15 @@
   <xacro:property name="rear_left_wheel_steering_joint" value="joint9" />
   <xacro:property name="rear_right_wheel_steering_joint" value="joint10" />
-  <xacro:property name="rear_wheel_radius" value="0.2" />
-  <xacro:property name="front_wheel_radius" value="0.2" />
+  <xacro:property name="live_hardware_plugin" value="foo" />
+  <xacro:property name="wheelbase" value="1.3" />
+  <xacro:property name="front_track" value="1.2" />
+  <xacro:property name="front_wheel_radius" value="0.4" />
+  <xacro:property name="rear_track" value="1.2" />
+  <xacro:property name="rear_wheel_radius" value="0.6" />
   <xacro:property name="maximal_axle_steering_angle" value="0.5" />
+  <xacro:property name="maximal_wheel_steering_angle" value="1.0" />
   <xacro:property name="maximal_wheel_speed" value="1.0" />
   <xacro:include
     filename="$(find romea_mobile_base_description)/ros2_control/base2AS4WD.ros2_control.xacro" />
-  <xacro:base_control mode="test" base_name="base" />
+  <xacro:base_control mode="live" base_name="base" />
 </robot>

File: romea_mobile_base_hardware/test/test_hardware_interface2FWS2FWD.xacro (robot description, xacro)
@@ -11,6 +11,16 @@
   <xacro:property name="maximal_wheel_speed" value="1.0" />
   <xacro:property name="front_wheel_radius" value="0.2" />
+  <xacro:property name="live_hardware_plugin" value="foo" />
+  <xacro:property name="wheelbase" value="1.4" />
+  <xacro:property name="front_track" value="1.2" />
+  <xacro:property name="front_wheel_radius" value="0.4" />
+  <xacro:property name="front_hub_carrier_offset" value="0.1" />
+  <xacro:property name="rear_track" value="1.4" />
+  <xacro:property name="rear_wheel_radius" value="0.6" />
+  <xacro:property name="rear_hub_carrier_offset" value="0.15" />
+  <xacro:property name="maximal_wheel_steering_angle" value="0.50" />
+  <xacro:property name="maximal_wheel_speed" value="1.0" />
   <xacro:include
     filename="$(find romea_mobile_base_description)/ros2_control/base2FWS2FWD.ros2_control.xacro" />
-  <xacro:base_control mode="test" base_name="base" />
+  <xacro:base_control mode="live" base_name="base" />
 </robot>

File: romea_mobile_base_hardware/test/test_hardware_interface2FWS2RWD.xacro (robot description, xacro)
@@ -11,6 +11,15 @@
   <xacro:property name="maximal_wheel_speed" value="1.0" />
   <xacro:property name="rear_wheel_radius" value="0.2" />
+  <xacro:property name="live_hardware_plugin" value="foo" />
+  <xacro:property name="wheelbase" value="1.2" />
+  <xacro:property name="front_track" value="1.4" />
+  <xacro:property name="front_wheel_radius" value="0.5" />
+  <xacro:property name="front_hub_carrier_offset" value="0.1" />
+  <xacro:property name="rear_track" value="1.0" />
+  <xacro:property name="rear_wheel_radius" value="0.3" />
+  <xacro:property name="maximal_wheel_steering_angle" value="0.50" />
+  <xacro:property name="maximal_wheel_speed" value="1.0" />
   <xacro:include
     filename="$(find romea_mobile_base_description)/ros2_control/base2FWS2RWD.ros2_control.xacro" />
-  <xacro:base_control mode="test" base_name="base" />
+  <xacro:base_control mode="live" base_name="base" />
 </robot>

File: romea_mobile_base_hardware/test/test_hardware_interface2FWS4WD.xacro (robot description, xacro)
@@ -8,10 +8,14 @@
   <xacro:property name="rear_left_wheel_spinning_joint" value="joint5" />
   <xacro:property name="rear_right_wheel_spinning_joint" value="joint6" />
-  <xacro:property name="maximal_wheel_steering_angle" value="0.5" />
+  <xacro:property name="live_hardware_plugin" value="foo" />
+  <xacro:property name="wheelbase" value="1.2" />
+  <xacro:property name="front_track" value="1.4" />
+  <xacro:property name="front_wheel_radius" value="0.5" />
+  <xacro:property name="rear_track" value="1.0" />
+  <xacro:property name="rear_wheel_radius" value="0.3" />
+  <xacro:property name="maximal_wheel_steering_angle" value="0.50" />
   <xacro:property name="maximal_wheel_speed" value="1.0" />
-  <xacro:property name="front_wheel_radius" value="0.2" />
-  <xacro:property name="rear_wheel_radius" value="0.2" />
   <xacro:include
     filename="$(find romea_mobile_base_description)/ros2_control/base2FWS4WD.ros2_control.xacro" />
-  <xacro:base_control mode="test" base_name="base" />
+  <xacro:base_control mode="live" base_name="base" />
 </robot>

File: romea_mobile_base_hardware/test/test_hardware_interface2TD.xacro (robot description, xacro)
@@ -10,6 +10,11 @@
   <xacro:property name="idler_wheel_radius" value="0.15" />
   <xacro:property name="track_thickness" value="0.2" />
+  <xacro:property name="live_hardware_plugin" value="foo" />
+  <xacro:property name="sprocket_wheel_radius" value="0.8" />
+  <xacro:property name="idler_wheel_radius" value="0.3" />
+  <xacro:property name="track_thickness" value="0.1" />
+  <xacro:property name="maximal_wheel_speed" value="1.0" />
   <xacro:include
     filename="$(find romea_mobile_base_description)/ros2_control/base2TD.ros2_control.xacro" />
-  <xacro:base_control mode="test" base_name="base" />
+  <xacro:base_control mode="live" base_name="base" />
 </robot>

File: romea_mobile_base_hardware/test/test_hardware_interface2THD.xacro (robot description, xacro)
@@ -12,6 +12,11 @@
   <xacro:property name="idler_wheel_radius" value="0.15" />
   <xacro:property name="track_thickness" value="0.2" />
+  <xacro:property name="live_hardware_plugin" value="foo" />
+  <xacro:property name="sprocket_wheel_radius" value="0.8" />
+  <xacro:property name="idler_wheel_radius" value="0.3" />
+  <xacro:property name="track_thickness" value="0.1" />
+  <xacro:property name="maximal_wheel_speed" value="1.0" />
   <xacro:include
     filename="$(find romea_mobile_base_description)/ros2_control/base2THD.ros2_control.xacro" />
-  <xacro:base_control mode="test" base_name="base" />
+  <xacro:base_control mode="live" base_name="base" />
 </robot>

File: romea_mobile_base_hardware/test/test_hardware_interface2TTD.xacro (robot description, xacro)
@@ -10,10 +10,12 @@
   <xacro:property name="rear_left_roller_wheel_spinning_joint" value="joint7" />
   <xacro:property name="rear_right_roller_wheel_spinning_joint" value="joint8" />
+  <xacro:property name="live_hardware_plugin" value="foo" />
+  <xacro:property name="sprocket_wheel_radius" value="0.8" />
+  <xacro:property name="roller_wheel_radius" value="0.3" />
+  <xacro:property name="idler_wheel_radius" value="0.3" />
+  <xacro:property name="track_thickness" value="0.1" />
   <xacro:property name="maximal_wheel_speed" value="1.0" />
-  <xacro:property name="sprocket_wheel_radius" value="0.2" />
-  <xacro:property name="idler_wheel_radius" value="0.15" />
-  <xacro:property name="track_thickness" value="0.2" />
   <xacro:include
     filename="$(find romea_mobile_base_description)/ros2_control/base2TTD.ros2_control.xacro" />
-  <xacro:base_control mode="test" base_name="base" />
+  <xacro:base_control mode="live" base_name="base" />
 </robot>

File: romea_mobile_base_hardware/test/test_hardware_interface4WS4WD.xacro (robot description, xacro)
@@ -14,6 +14,14 @@
   <xacro:property name="front_wheel_radius" value="0.2" />
   <xacro:property name="rear_wheel_radius" value="0.2" />
+  <xacro:property name="live_hardware_plugin" value="foo" />
+  <xacro:property name="wheelbase" value="1.2" />
+  <xacro:property name="front_track" value="1.4" />
+  <xacro:property name="front_wheel_radius" value="0.5" />
+  <xacro:property name="rear_track" value="1.0" />
+  <xacro:property name="rear_wheel_radius" value="0.3" />
+  <xacro:property name="maximal_wheel_steering_angle" value="0.50" />
+  <xacro:property name="maximal_wheel_speed" value="1.0" />
   <xacro:include
     filename="$(find romea_mobile_base_description)/ros2_control/base4WS4WD.ros2_control.xacro" />
-  <xacro:base_control mode="test" base_name="base" />
+  <xacro:base_control mode="live" base_name="base" />
 </robot>
