Commit message: add support of generic_simulation  using joint_states I/O for all kind of robots
Signed-off-by: jean.laneurit <jean.laneurit@inrae.fr>

File: romea_mobile_base_description/ros2_control/base1FAS2FWD.ros2_control.xacro (robot description, xacro)
@@ -35,7 +35,19 @@
       </joint>
       <joint name="${prefix}${front_left_wheel_steering_joint}">
+        <xacro:if value="${'simulation' in mode}">
+          <command_interface name="position">
+            <param name="min">${-maximal_wheel_steering_angle}</param>
+            <param name="max">${maximal_wheel_steering_angle}</param>
+          </command_interface>
+        </xacro:if>
         <state_interface name="position" />
       </joint>
       <joint name="${prefix}${front_right_wheel_steering_joint}">
+        <xacro:if value="${'simulation' in mode}">
+          <command_interface name="position">
+            <param name="min">${-maximal_wheel_steering_angle}</param>
+            <param name="max">${maximal_wheel_steering_angle}</param>
+          </command_interface>
+        </xacro:if>
         <state_interface name="position" />
       </joint>
@@ -59,4 +71,10 @@
       </joint>
       <joint name="${prefix}${rear_left_wheel_spinning_joint}">
+        <xacro:if value="${'simulation' in mode}">
+          <command_interface name="velocity">
+            <param name="min">${-maximal_wheel_speed/rear_wheel_radius}</param>
+            <param name="max">${maximal_wheel_speed/rear_wheel_radius}</param>
+          </command_interface>
+        </xacro:if>
         <state_interface name="position" />
         <state_interface name="velocity" />
@@ -64,4 +82,10 @@
       </joint>
       <joint name="${prefix}${rear_right_wheel_spinning_joint}">
+        <xacro:if value="${'simulation' in mode}">
+          <command_interface name="velocity">
+            <param name="min">${-maximal_wheel_speed/rear_wheel_radius}</param>
+            <param name="max">${maximal_wheel_speed/rear_wheel_radius}</param>
+          </command_interface>
+        </xacro:if>
         <state_interface name="position" />
         <state_interface name="velocity" />

File: romea_mobile_base_description/ros2_control/base1FAS2RWD.ros2_control.xacro (robot description, xacro)
@@ -31,10 +31,28 @@
       </joint>
       <joint name="${prefix}${front_left_wheel_steering_joint}">
+        <xacro:if value="${'simulation' in mode}">
+          <command_interface name="position">
+            <param name="min">${-maximal_wheel_steering_angle}</param>
+            <param name="max">${maximal_wheel_steering_angle}</param>
+          </command_interface>
+        </xacro:if>
         <state_interface name="position" />
       </joint>
       <joint name="${prefix}${front_right_wheel_steering_joint}">
+        <xacro:if value="${'simulation' in mode}">
+          <command_interface name="position">
+            <param name="min">${-maximal_wheel_steering_angle}</param>
+            <param name="max">${maximal_wheel_steering_angle}</param>
+          </command_interface>
+        </xacro:if>
         <state_interface name="position" />
       </joint>
       <joint name="${prefix}${front_left_wheel_spinning_joint}">
+        <xacro:if value="${'simulation' in mode}">
+          <command_interface name="velocity">
+            <param name="min">${-maximal_wheel_speed/front_wheel_radius}</param>
+            <param name="max">${maximal_wheel_speed/front_wheel_radius}</param>
+          </command_interface>
+        </xacro:if>
         <state_interface name="position" />
         <state_interface name="velocity" />
@@ -42,4 +60,10 @@
       </joint>
       <joint name="${prefix}${front_right_wheel_spinning_joint}">
+        <xacro:if value="${'simulation' in mode}">
+          <command_interface name="velocity">
+            <param name="min">${-maximal_wheel_speed/front_wheel_radius}</param>
+            <param name="max">${maximal_wheel_speed/front_wheel_radius}</param>
+          </command_interface>
+        </xacro:if>
         <state_interface name="position" />
         <state_interface name="velocity" />

File: romea_mobile_base_description/ros2_control/base1FAS4WD.ros2_control.xacro (robot description, xacro)
@@ -31,7 +31,19 @@
       </joint>
       <joint name="${prefix}${front_left_wheel_steering_joint}">
+        <xacro:if value="${'simulation' in mode}">
+          <command_interface name="position">
+            <param name="min">${-maximal_wheel_steering_angle}</param>
+            <param name="max">${maximal_wheel_steering_angle}</param>
+          </command_interface>
+        </xacro:if>
         <state_interface name="position" />
       </joint>
       <joint name="${prefix}${front_right_wheel_steering_joint}">
+        <xacro:if value="${'simulation' in mode}">
+          <command_interface name="position">
+            <param name="min">${-maximal_wheel_steering_angle}</param>
+            <param name="max">${maximal_wheel_steering_angle}</param>
+          </command_interface>
+        </xacro:if>
         <state_interface name="position" />
       </joint>

File: romea_mobile_base_description/ros2_control/base2AS4WD.ros2_control.xacro (robot description, xacro)
@@ -36,13 +36,37 @@
       </joint>
       <joint name="${prefix}${front_left_wheel_steering_joint}">
+        <xacro:if value="${'simulation' in mode}">
+          <command_interface name="position">
+            <param name="min">${-maximal_wheel_steering_angle}</param>
+            <param name="max">${maximal_wheel_steering_angle}</param>
+          </command_interface>
+        </xacro:if>
         <state_interface name="position" />
       </joint>
       <joint name="${prefix}${front_right_wheel_steering_joint}">
+        <xacro:if value="${'simulation' in mode}">
+          <command_interface name="position">
+            <param name="min">${-maximal_wheel_steering_angle}</param>
+            <param name="max">${maximal_wheel_steering_angle}</param>
+          </command_interface>
+        </xacro:if>
         <state_interface name="position" />
       </joint>
       <joint name="${prefix}${rear_left_wheel_steering_joint}">
+        <xacro:if value="${'simulation' in mode}">
+          <command_interface name="position">
+            <param name="min">${-maximal_wheel_steering_angle}</param>
+            <param name="max">${maximal_wheel_steering_angle}</param>
+          </command_interface>
+        </xacro:if>
         <state_interface name="position" />
       </joint>
       <joint name="${prefix}${rear_right_wheel_steering_joint}">
+        <xacro:if value="${'simulation' in mode}">
+          <command_interface name="position">
+            <param name="min">${-maximal_wheel_steering_angle}</param>
+            <param name="max">${maximal_wheel_steering_angle}</param>
+          </command_interface>
+        </xacro:if>
         <state_interface name="position" />
       </joint>

File: romea_mobile_base_description/ros2_control/base2FWS2FWD.ros2_control.xacro (robot description, xacro)
@@ -60,4 +60,10 @@
       </joint>
       <joint name="${prefix}${rear_left_wheel_spinning_joint}">
+        <xacro:if value="${'simulation' in mode}">
+          <command_interface name="velocity">
+            <param name="min">${-maximal_wheel_speed/front_wheel_radius}</param>
+            <param name="max">${maximal_wheel_speed/front_wheel_radius}</param>
+          </command_interface>
+        </xacro:if>
         <state_interface name="position" />
         <state_interface name="velocity" />
@@ -65,4 +71,10 @@
       </joint>
       <joint name="${prefix}${rear_right_wheel_spinning_joint}">
+        <xacro:if value="${'simulation' in mode}">
+          <command_interface name="velocity">
+            <param name="min">${-maximal_wheel_speed/front_wheel_radius}</param>
+            <param name="max">${maximal_wheel_speed/front_wheel_radius}</param>
+          </command_interface>
+        </xacro:if>
         <state_interface name="position" />
         <state_interface name="velocity" />

File: romea_mobile_base_description/ros2_control/base2FWS2RWD.ros2_control.xacro (robot description, xacro)
@@ -40,4 +40,10 @@
       </joint>
       <joint name="${prefix}${front_left_wheel_spinning_joint}">
+        <xacro:if value="${'simulation' in mode}">
+          <command_interface name="velocity">
+            <param name="min">${-maximal_wheel_speed/front_wheel_radius}</param>
+            <param name="max">${maximal_wheel_speed/front_wheel_radius}</param>
+          </command_interface>
+        </xacro:if>
         <state_interface name="position" />
         <state_interface name="velocity" />
@@ -45,4 +51,10 @@
       </joint>
       <joint name="${prefix}${front_right_wheel_spinning_joint}">
+        <xacro:if value="${'simulation' in mode}">
+          <command_interface name="velocity">
+            <param name="min">${-maximal_wheel_speed/front_wheel_radius}</param>
+            <param name="max">${maximal_wheel_speed/front_wheel_radius}</param>
+          </command_interface>
+        </xacro:if>
         <state_interface name="position" />
         <state_interface name="velocity" />

File: romea_mobile_base_description/ros2_control/base2TD.ros2_control.xacro (robot description, xacro)
@@ -38,5 +38,5 @@
       </joint>
       <joint name="${prefix}${left_idler_wheel_spinning_joint}">
-        <xacro:if value="${mode == 'simulation'}">
+        <xacro:if value="${'simulation' in mode}">
           <command_interface name="velocity">
             <param name="min">${-maximal_wheel_speed/(idler_wheel_radius+track_thickness)}</param>
@@ -49,5 +49,5 @@
       </joint>
       <joint name="${prefix}${right_idler_wheel_spinning_joint}">
-        <xacro:if value="${mode == 'simulation'}">
+        <xacro:if value="${'simulation' in mode}">
           <command_interface name="velocity">
             <param name="min">${-maximal_wheel_speed/(idler_wheel_radius+track_thickness)}</param>

File: romea_mobile_base_description/ros2_control/base2THD.ros2_control.xacro (robot description, xacro)
@@ -38,5 +38,5 @@
       </joint>
       <joint name="${prefix}${front_left_idler_wheel_spinning_joint}">
-        <xacro:if value="${mode == 'simulation'}">
+        <xacro:if value="${'simulation' in mode}">
           <command_interface name="velocity">
             <param name="min">${-maximal_wheel_speed/(idler_wheel_radius+track_thickness)}</param>
@@ -49,5 +49,5 @@
       </joint>
       <joint name="${prefix}${front_right_idler_wheel_spinning_joint}">
-        <xacro:if value="${mode == 'simulation'}">
+        <xacro:if value="${'simulation' in mode}">
           <command_interface name="velocity">
             <param name="min">${-maximal_wheel_speed/(idler_wheel_radius+track_thickness)}</param>
@@ -60,5 +60,5 @@
       </joint>
       <joint name="${prefix}${rear_left_idler_wheel_spinning_joint}">
-        <xacro:if value="${mode == 'simulation'}">
+        <xacro:if value="${'simulation' in mode}">
           <command_interface name="velocity">
             <param name="min">${-maximal_wheel_speed/(idler_wheel_radius+track_thickness)}</param>
@@ -71,5 +71,5 @@
       </joint>
       <joint name="${prefix}${rear_right_idler_wheel_spinning_joint}">
-        <xacro:if value="${mode == 'simulation'}">
+        <xacro:if value="${'simulation' in mode}">
           <command_interface name="velocity">
             <param name="min">${-maximal_wheel_speed/(idler_wheel_radius+track_thickness)}</param>

File: romea_mobile_base_description/ros2_control/base2TTD.ros2_control.xacro (robot description, xacro)
@@ -40,5 +40,5 @@
       </joint>
       <joint name="${prefix}${left_idler_wheel_spinning_joint}">
-        <xacro:if value="${mode == 'simulation'}">
+        <xacro:if value="${'simulation' in mode}">
           <command_interface name="velocity">
             <param name="min">${-maximal_wheel_speed/(idler_wheel_radius+track_thickness)}</param>
@@ -51,5 +51,5 @@
       </joint>
       <joint name="${prefix}${right_idler_wheel_spinning_joint}">
-        <xacro:if value="${mode == 'simulation'}">
+        <xacro:if value="${'simulation' in mode}">
           <command_interface name="velocity">
             <param name="min">${-maximal_wheel_speed/(idler_wheel_radius+track_thickness)}</param>
@@ -62,5 +62,5 @@
       </joint>
       <joint name="${prefix}${front_left_roller_wheel_spinning_joint}">
-        <xacro:if value="${mode == 'simulation'}">
+        <xacro:if value="${'simulation' in mode}">
           <command_interface name="velocity">
             <param name="min">${-maximal_wheel_speed/(roller_wheel_radius+track_thickness)}</param>
@@ -73,5 +73,5 @@
       </joint>
       <joint name="${prefix}${front_right_roller_wheel_spinning_joint}">
-        <xacro:if value="${mode == 'simulation'}">
+        <xacro:if value="${'simulation' in mode}">
           <command_interface name="velocity">
             <param name="min">${-maximal_wheel_speed/(roller_wheel_radius+track_thickness)}</param>
@@ -84,5 +84,5 @@
       </joint>
       <joint name="${prefix}${rear_left_roller_wheel_spinning_joint}">
-        <xacro:if value="${mode == 'simulation'}">
+        <xacro:if value="${'simulation' in mode}">
           <command_interface name="velocity">
             <param name="min">${-maximal_wheel_speed/(roller_wheel_radius+track_thickness)}</param>
@@ -95,5 +95,5 @@
       </joint>
       <joint name="${prefix}${rear_right_roller_wheel_spinning_joint}">
-        <xacro:if value="${mode == 'simulation'}">
+        <xacro:if value="${'simulation' in mode}">
           <command_interface name="velocity">
             <param name="min">${-maximal_wheel_speed/(roller_wheel_radius+track_thickness)}</param>

File: romea_mobile_base_simulation/test/test_simulation_interface1FAS2FWD.xacro (robot description, xacro)
@@ -18,4 +18,5 @@
   <xacro:property name="rear_hub_carrier_offset" value="0.15" />
   <xacro:property name="maximal_axle_steering_angle" value="0.50" />
+  <xacro:property name="maximal_wheel_steering_angle" value="1.00" />
   <xacro:property name="maximal_wheel_speed" value="1.0" />
   <xacro:include

File: romea_mobile_base_simulation/test/test_simulation_interface1FAS2RWD.xacro (robot description, xacro)
@@ -3,10 +3,10 @@
   <xacro:property name="prefix" value="robot_" />
   <xacro:property name="front_axle_steering_joint" value="joint1" />
-  <xacro:property name="rear_left_wheel_spinning_joint" value="joint2" />
-  <xacro:property name="rear_right_wheel_spinning_joint" value="joint3" />
-  <xacro:property name="front_left_wheel_steering_joint" value="joint4" />
-  <xacro:property name="front_right_wheel_steering_joint" value="joint5" />
-  <xacro:property name="front_left_wheel_spinning_joint" value="joint6" />
-  <xacro:property name="front_right_wheel_spinning_joint" value="joint7" />
+  <xacro:property name="front_left_wheel_steering_joint" value="joint2" />
+  <xacro:property name="front_right_wheel_steering_joint" value="joint3" />
+  <xacro:property name="front_left_wheel_spinning_joint" value="joint4" />
+  <xacro:property name="front_right_wheel_spinning_joint" value="joint5" />
+  <xacro:property name="rear_left_wheel_spinning_joint" value="joint6" />
+  <xacro:property name="rear_right_wheel_spinning_joint" value="joint7" />
   <xacro:property name="simulation_hardware_plugin" value="foo" />
   <xacro:property name="wheelbase" value="1.3" />
@@ -16,4 +16,5 @@
   <xacro:property name="rear_wheel_radius" value="0.7" />
   <xacro:property name="maximal_axle_steering_angle" value="0.50" />
+  <xacro:property name="maximal_wheel_steering_angle" value="1.00" />
   <xacro:property name="maximal_wheel_speed" value="1.0" />
   <xacro:include

File: romea_mobile_base_simulation/test/test_simulation_interface2AS4WD.xacro (robot description, xacro)
@@ -20,6 +20,9 @@
   <xacro:property name="rear_wheel_radius" value="0.6" />
   <xacro:property name="rear_hub_carrier_offset" value="0.1" />
+  <xacro:property name="maximal_axle_steering_angle" value="0.5" />
+  <xacro:property name="maximal_wheel_steering_angle" value="1.0" />
+  <xacro:property name="maximal_wheel_speed" value="1.0" />
   <xacro:include
-    filename="$(find romea_mobile_base_description)/ros2_control/2AS_4WD.ros2_control.xacro" />
-  <xacro:base_control mode="test" base_name="base" />
+    filename="$(find romea_mobile_base_description)/ros2_control/base2AS4WD.ros2_control.xacro" />
+  <xacro:base_control mode="simulation" base_name="base" />
 </robot>
