Commit message: add hardware_options param in controler plugin

File: romea_mobile_base_description/ros2_control/base1FAS2FWD.ros2_control.xacro (robot description, xacro)
@@ -1,5 +1,5 @@
 <?xml version="1.0"?>
 <robot xmlns:xacro="http://www.ros.org/wiki/xacro">
-  <xacro:macro name="base_control" params="mode base_name">
+  <xacro:macro name="base_control" params="mode base_name has_hardware_options:=0">
     <ros2_control name="${prefix}${base_name}" type="system">
       <xacro:if value="${mode == 'live'}">
@@ -13,4 +13,7 @@
           <param name="rear_wheel_radius">${rear_wheel_radius}</param>
           <param name="rear_hub_carrier_offset">${rear_hub_carrier_offset}</param>
+          <xacro:if value="${has_hardware_options}">
+            <xacro:insert_block name="hardware_options"/>
+          </xacro:if>
         </hardware>
       </xacro:if>

File: romea_mobile_base_description/ros2_control/base1FAS2RWD.ros2_control.xacro (robot description, xacro)
@@ -1,5 +1,5 @@
 <?xml version="1.0"?>
 <robot xmlns:xacro="http://www.ros.org/wiki/xacro">
-  <xacro:macro name="base_control" params="mode base_name">
+  <xacro:macro name="base_control" params="mode base_name has_hardware_options:=0">
     <ros2_control name="${prefix}${base_name}" type="system">
       <xacro:if value="${mode == 'live'}">
@@ -11,4 +11,7 @@
           <param name="front_hub_carrier_offset">${front_hub_carrier_offset}</param>
           <param name="rear_wheel_radius">${rear_wheel_radius}</param>
+          <xacro:if value="${has_hardware_options}">
+            <xacro:insert_block name="hardware_options"/>
+          </xacro:if>
         </hardware>
       </xacro:if>

File: romea_mobile_base_description/ros2_control/base1FAS4WD.ros2_control.xacro (robot description, xacro)
@@ -1,5 +1,5 @@
 <?xml version="1.0"?>
 <robot xmlns:xacro="http://www.ros.org/wiki/xacro">
-  <xacro:macro name="base_control" params="mode base_name">
+  <xacro:macro name="base_control" params="mode base_name has_hardware_options:=0">
     <ros2_control name="${prefix}${base_name}" type="system">
       <xacro:if value="${mode == 'live'}">
@@ -10,4 +10,7 @@
           <param name="front_wheel_radius">${front_wheel_radius}</param>
           <param name="rear_wheel_radius">${rear_wheel_radius}</param>
+          <xacro:if value="${has_hardware_options}">
+            <xacro:insert_block name="hardware_options"/>
+          </xacro:if>
         </hardware>
       </xacro:if>

File: romea_mobile_base_description/ros2_control/base2AS2FWD.ros2_control.xacro (robot description, xacro)
@@ -1,5 +1,5 @@
 <?xml version="1.0"?>
 <robot xmlns:xacro="http://www.ros.org/wiki/xacro">
-  <xacro:macro name="base_control" params="mode base_name">
+  <xacro:macro name="base_control" params="mode base_name has_hardware_options:=0">
     <ros2_control name="${prefix}${base_name}" type="system">
       <xacro:if value="${mode == 'live'}">
@@ -13,4 +13,7 @@
           <param name="rear_wheel_radius">${rear_wheel_radius}</param>
           <param name="rear_hub_carrier_offset">${rear_hub_carrier_offset}</param>
+          <xacro:if value="${has_hardware_options}">
+            <xacro:insert_block name="hardware_options"/>
+          </xacro:if>
         </hardware>
       </xacro:if>

File: romea_mobile_base_description/ros2_control/base2AS2RWD.ros2_control.xacro (robot description, xacro)
@@ -1,5 +1,5 @@
 <?xml version="1.0"?>
 <robot xmlns:xacro="http://www.ros.org/wiki/xacro">
-  <xacro:macro name="base_control" params="mode base_name">
+  <xacro:macro name="base_control" params="mode base_name has_hardware_options:=0">
     <ros2_control name="${prefix}${base_name}" type="system">
       <xacro:if value="${mode == 'live'}">
@@ -13,4 +13,7 @@
           <param name="rear_wheel_radius">${rear_wheel_radius}</param>
           <param name="rear_hub_carrier_offset">${rear_hub_carrier_offset}</param>
+          <xacro:if value="${has_hardware_options}">
+            <xacro:insert_block name="hardware_options"/>
+          </xacro:if>
         </hardware>
       </xacro:if>

File: romea_mobile_base_description/ros2_control/base2AS4WD.ros2_control.xacro (robot description, xacro)
@@ -1,5 +1,5 @@
 <?xml version="1.0"?>
 <robot xmlns:xacro="http://www.ros.org/wiki/xacro">
-  <xacro:macro name="base_control" params="mode base_name">
+  <xacro:macro name="base_control" params="mode base_name has_hardware_options:=0">
     <ros2_control name="${prefix}${base_name}" type="system">
       <xacro:if value="${mode == 'live'}">
@@ -11,4 +11,7 @@
           <param name="front_wheel_radius">${front_wheel_radius}</param>
           <param name="rear_wheel_radius">${rear_wheel_radius}</param>
+          <xacro:if value="${has_hardware_options}">
+            <xacro:insert_block name="hardware_options"/>
+          </xacro:if>
         </hardware>
       </xacro:if>

File: romea_mobile_base_description/ros2_control/base2FWS2FWD.ros2_control.xacro (robot description, xacro)
@@ -1,5 +1,5 @@
 <?xml version="1.0"?>
 <robot xmlns:xacro="http://www.ros.org/wiki/xacro">
-  <xacro:macro name="base_control" params="mode base_name">
+  <xacro:macro name="base_control" params="mode base_name has_hardware_options:=0">
     <ros2_control name="${prefix}${base_name}" type="system">
       <xacro:if value="${mode == 'live'}">
@@ -13,4 +13,7 @@
           <param name="rear_wheel_radius">${rear_wheel_radius}</param>
           <param name="rear_hub_carrier_offset">${rear_hub_carrier_offset}</param>
+          <xacro:if value="${has_hardware_options}">
+            <xacro:insert_block name="hardware_options"/>
+          </xacro:if>
         </hardware>
       </xacro:if>

File: romea_mobile_base_description/ros2_control/base2FWS2RWD.ros2_control.xacro (robot description, xacro)
@@ -1,5 +1,5 @@
 <?xml version="1.0"?>
 <robot xmlns:xacro="http://www.ros.org/wiki/xacro">
-  <xacro:macro name="base_control" params="mode base_name">
+  <xacro:macro name="base_control" params="mode base_name has_hardware_options:=0">
     <ros2_control name="${prefix}${base_name}" type="system">
       <xacro:if value="${mode == 'live'}">
@@ -12,4 +12,7 @@
           <param name="rear_track">${rear_track}</param>
           <param name="rear_wheel_radius">${rear_wheel_radius}</param>
+          <xacro:if value="${has_hardware_options}">
+            <xacro:insert_block name="hardware_options"/>
+          </xacro:if>
         </hardware>
       </xacro:if>

File: romea_mobile_base_description/ros2_control/base2FWS4WD.ros2_control.xacro (robot description, xacro)
@@ -1,5 +1,5 @@
 <?xml version="1.0"?>
 <robot xmlns:xacro="http://www.ros.org/wiki/xacro">
-  <xacro:macro name="base_control" params="mode base_name">
+  <xacro:macro name="base_control" params="mode base_name has_hardware_options:=0">
     <ros2_control name="${prefix}${base_name}" type="system">
       <xacro:if value="${mode == 'live'}">
@@ -11,4 +11,7 @@
           <param name="rear_track">${rear_track}</param>
           <param name="rear_wheel_radius">${rear_wheel_radius}</param>
+          <xacro:if value="${has_hardware_options}">
+            <xacro:insert_block name="hardware_options"/>
+          </xacro:if>
         </hardware>
       </xacro:if>

File: romea_mobile_base_description/ros2_control/base2TD.ros2_control.xacro (robot description, xacro)
@@ -1,5 +1,5 @@
 <?xml version="1.0"?>
 <robot xmlns:xacro="http://www.ros.org/wiki/xacro">
-  <xacro:macro name="base_control" params="mode base_name">
+  <xacro:macro name="base_control" params="mode base_name has_hardware_options:=0">
     <ros2_control name="${prefix}${base_name}" type="system">
       <xacro:if value="${mode == 'live'}">
@@ -9,4 +9,7 @@
           <param name="idler_wheel_radius">${idler_wheel_radius}</param>
           <param name="track_thickness">${track_thickness}</param>
+          <xacro:if value="${has_hardware_options}">
+            <xacro:insert_block name="hardware_options"/>
+          </xacro:if>
         </hardware>
       </xacro:if>

File: romea_mobile_base_description/ros2_control/base2THD.ros2_control.xacro (robot description, xacro)
@@ -1,5 +1,5 @@
 <?xml version="1.0"?>
 <robot xmlns:xacro="http://www.ros.org/wiki/xacro">
-  <xacro:macro name="base_control" params="mode base_name">
+  <xacro:macro name="base_control" params="mode base_name has_hardware_options:=0">
     <ros2_control name="${prefix}${base_name}" type="system">
       <xacro:if value="${mode == 'live'}">
@@ -9,4 +9,7 @@
           <param name="idler_wheel_radius">${idler_wheel_radius}</param>
           <param name="track_thickness">${track_thickness}</param>
+          <xacro:if value="${has_hardware_options}">
+            <xacro:insert_block name="hardware_options"/>
+          </xacro:if>
         </hardware>
       </xacro:if>

File: romea_mobile_base_description/ros2_control/base2TTD.ros2_control.xacro (robot description, xacro)
@@ -1,5 +1,5 @@
 <?xml version="1.0"?>
 <robot xmlns:xacro="http://www.ros.org/wiki/xacro">
-  <xacro:macro name="base_control" params="mode base_name">
+  <xacro:macro name="base_control" params="mode base_name has_hardware_options:=0">
     <ros2_control name="${prefix}${base_name}" type="system">
       <xacro:if value="${mode == 'live'}">
@@ -10,4 +10,7 @@
           <param name="idler_wheel_radius">${idler_wheel_radius}</param>
           <param name="track_thickness">${track_thickness}</param>
+          <xacro:if value="${has_hardware_options}">
+            <xacro:insert_block name="hardware_options"/>
+          </xacro:if>
         </hardware>
       </xacro:if>

File: romea_mobile_base_description/ros2_control/base4WD.ros2_control.xacro (robot description, xacro)
@@ -1,5 +1,5 @@
 <?xml version="1.0"?>
 <robot xmlns:xacro="http://www.ros.org/wiki/xacro">
-  <xacro:macro name="base_control" params="mode base_name">
+  <xacro:macro name="base_control" params="mode base_name has_hardware_options:=0">
     <ros2_control name="${prefix}${base_name}" type="system">
       <xacro:if value="${mode == 'live'}">
@@ -11,4 +11,7 @@
           <param name="front_track">${front_track}</param>
           <param name="rear_track">${rear_track}</param>
+          <xacro:if value="${has_hardware_options}">
+            <xacro:insert_block name="hardware_options"/>
+          </xacro:if>
         </hardware>
       </xacro:if>

File: romea_mobile_base_description/ros2_control/base4WS4WD.ros2_control.xacro (robot description, xacro)
@@ -1,5 +1,5 @@
 <?xml version="1.0"?>
 <robot xmlns:xacro="http://www.ros.org/wiki/xacro">
-  <xacro:macro name="base_control" params="mode base_name">
+  <xacro:macro name="base_control" params="mode base_name has_hardware_options:=0">
     <ros2_control name="${prefix}${base_name}" type="system">
       <xacro:if value="${mode == 'live'}">
@@ -11,4 +11,7 @@
           <param name="front_wheel_radius">${front_wheel_radius}</param>
           <param name="rear_wheel_radius">${rear_wheel_radius}</param>
+          <xacro:if value="${has_hardware_options}">
+            <xacro:insert_block name="hardware_options"/>
+          </xacro:if>
         </hardware>
       </xacro:if>
