Commit message: update ros2_control xacro files in order to be indepedent of base urdf add a way get elapsed time between two get_joint_state_command
Signed-off-by: Jean Laneurit <jean.laneurit@inrae.fr>

File: romea_mobile_base_description/ros2_control/base1FAS2FWD.ros2_control.xacro (robot description, xacro)
@@ -1,4 +1,5 @@
 <?xml version="1.0"?>
 <robot xmlns:xacro="http://www.ros.org/wiki/xacro">
+  <xacro:include filename="$(find romea_mobile_base_description)/ros2_control/base1FASxxx.ros2_control.xacro" />
   <xacro:macro name="base_control_parameters" params="interface_name">
     <param name="wheelbase">${wheelbase}</param>
@@ -108,4 +109,5 @@
     name="base_control"
     params="mode base_name hardware_plugin has_hardware_options:=0">
+    <xacro:base_control_model/>
     <ros2_control name="${prefix}${base_name}" type="system">
       <xacro:base_control_hardware

File: romea_mobile_base_description/ros2_control/base1FAS2RWD.ros2_control.xacro (robot description, xacro)
@@ -1,4 +1,5 @@
 <?xml version="1.0"?>
 <robot xmlns:xacro="http://www.ros.org/wiki/xacro">
+  <xacro:include filename="$(find romea_mobile_base_description)/ros2_control/base1FASxxx.ros2_control.xacro" />
   <xacro:macro name="base_control_parameters" params="interface_name">
     <param name="wheelbase">${wheelbase}</param>
@@ -94,5 +95,5 @@
       <command_interface name="velocity">
         <param name="min">${-maximal_wheel_speed/rear_wheel_radius}</param>
-        <param name="max">${-maximal_wheel_speed/rear_wheel_radius}</param>
+        <param name="max">${maximal_wheel_speed/rear_wheel_radius}</param>
       </command_interface>
       <state_interface name="position" />
@@ -103,5 +104,7 @@
   <xacro:macro
     name="base_control"
-    params="mode base_name hardware_plugin has_hardware_options:=0">
+    params="mode base_name hardware_plugin has_hardware_options:=0
+            prefix:=^|''">
+    <xacro:base_control_model/>
     <ros2_control name="${prefix}${base_name}" type="system">
       <xacro:base_control_hardware

File: romea_mobile_base_description/ros2_control/base1FAS4WD.ros2_control.xacro (robot description, xacro)
@@ -1,4 +1,5 @@
 <?xml version="1.0"?>
 <robot xmlns:xacro="http://www.ros.org/wiki/xacro">
+  <xacro:include filename="$(find romea_mobile_base_description)/ros2_control/base1FASxxx.ros2_control.xacro" />
   <xacro:macro name="base_control_parameters" params="interface_name">
     <param name="wheelbase">${wheelbase}</param>
@@ -98,4 +99,5 @@
     name="base_control"
     params="mode base_name hardware_plugin has_hardware_options:=0">
+    <xacro:base_control_model/>
     <ros2_control name="${prefix}${base_name}" type="system">
       <xacro:base_control_hardware

File: romea_mobile_base_description/ros2_control/base2AS2FWD.ros2_control.xacro (robot description, xacro)
@@ -1,4 +1,5 @@
 <?xml version="1.0"?>
 <robot xmlns:xacro="http://www.ros.org/wiki/xacro">
+  <xacro:include filename="$(find romea_mobile_base_description)/ros2_control/base2ASxxx.ros2_control.xacro" />
   <xacro:macro name="base_control_parameters" params="interface_name">
     <param name="wheelbase">${wheelbase}</param>
@@ -100,4 +101,5 @@
     name="base_control"
     params="mode base_name hardware_plugin has_hardware_options:=0">
+    <xacro:base_control_model/>
     <ros2_control name="${prefix}${base_name}" type="system">
       <xacro:base_control_hardware

File: romea_mobile_base_description/ros2_control/base2AS2RWD.ros2_control.xacro (robot description, xacro)
@@ -1,4 +1,5 @@
 <?xml version="1.0"?>
 <robot xmlns:xacro="http://www.ros.org/wiki/xacro">
+  <xacro:include filename="$(find romea_mobile_base_description)/ros2_control/base2ASxxx.ros2_control.xacro" />
   <xacro:macro name="base_control_parameters" params="interface_name">
     <param name="wheelbase">${wheelbase}</param>
@@ -100,4 +101,5 @@
     name="base_control"
     params="mode base_name hardware_plugin has_hardware_options:=0">
+    <xacro:base_control_model/>
     <ros2_control name="${prefix}${base_name}" type="system">
       <xacro:base_control_hardware

File: romea_mobile_base_description/ros2_control/base2AS4WD.ros2_control.xacro (robot description, xacro)
@@ -1,4 +1,5 @@
 <?xml version="1.0"?>
 <robot xmlns:xacro="http://www.ros.org/wiki/xacro">
+  <xacro:include filename="$(find romea_mobile_base_description)/ros2_control/base2ASxxx.ros2_control.xacro" />
   <xacro:macro name="base_control_parameters" params="interface_name">
     <param name="wheelbase">${wheelbase}</param>
@@ -128,4 +129,5 @@
     name="base_control"
     params="mode base_name hardware_plugin has_hardware_options:=0">
+    <xacro:base_control_model/>
     <ros2_control name="${prefix}${base_name}" type="system">
       <xacro:base_control_hardware

File: romea_mobile_base_description/ros2_control/base2FWC2RWD.ros2_control.xacro (robot description, xacro)
@@ -1,4 +1,44 @@
 <?xml version="1.0"?>
 <robot xmlns:xacro="http://www.ros.org/wiki/xacro">
+  <xacro:include filename="$(find romea_mobile_base_description)/ros2_control/base_control_joints.xacro" />
+  <xacro:macro name="base_control_model">
+    <link name="${prefix}${base_link}" />
+    <link name="${prefix}${front_left_wheel_swiveling_link}" />
+    <joint name="${prefix}${front_left_wheel_swiveling_joint}" type="continuous">
+      <parent link="${prefix}${base_link}" />
+      <child link="${prefix}${front_left_wheel_swiveling_link}" />
+      <axis xyz="0 0 1" />
+    </joint>
+    <link name="${prefix}${front_right_wheel_swiveling_link}" />
+    <joint name="${prefix}${front_right_wheel_swiveling_joint}" type="continuous">
+      <parent link="${prefix}${base_link}" />
+      <child link="${prefix}${front_right_wheel_swiveling_link}" />
+      <axis xyz="0 0 1" />
+    </joint>
+    <link name="${prefix}${front_left_wheel_spinning_link}" />
+    <joint name="${prefix}${front_left_wheel_spinning_joint}" type="continuous">
+      <parent link="${prefix}${front_left_wheel_swiveling_link}" />
+      <child link="${prefix}${front_left_wheel_spinning_link}" />
+      <axis xyz="0 0 1" />
+    </joint>
+    <link name="${prefix}${front_right_wheel_spinning_link}" />
+    <joint name="${prefix}${front_right_wheel_spinning_joint}" type="continuous">
+      <parent link="${prefix}${front_right_wheel_swiveling_link}" />
+      <child link="${prefix}${front_right_wheel_spinning_link}" />
+      <axis xyz="0 0 1" />
+    </joint>
+    <xacro:base_control_continuous_joint
+      parent_link="${base_link}"
+      child_link="${rear_left_wheel_spinning_link}"
+      joint_name="${rear_left_wheel_spinning_joint}"
+      velocity="${maximal_wheel_speed/rear_wheel_radius}"
+      effort="${maximal_wheel_torque}" />
+    <xacro:base_control_continuous_joint
+      parent_link="${base_link}"
+      child_link="${rear_right_wheel_spinning_link}"
+      joint_name="${rear_right_wheel_spinning_joint}"
+      velocity="${maximal_wheel_speed/rear_wheel_radius}"
+      effort="${maximal_wheel_torque}" />
+  </xacro:macro>
   <xacro:macro name="base_control_parameters" params="interface_name">
     <param name="wheelbase">${wheelbase}</param>
@@ -74,4 +114,5 @@
     name="base_control"
     params="mode base_name hardware_plugin has_hardware_options:=0">
+    <xacro:base_control_model/>
     <ros2_control name="${prefix}${base_name}" type="system">
       <xacro:base_control_hardware

File: romea_mobile_base_description/ros2_control/base2FWS2FWD.ros2_control.xacro (robot description, xacro)
@@ -1,4 +1,5 @@
 <?xml version="1.0"?>
 <robot xmlns:xacro="http://www.ros.org/wiki/xacro">
+  <xacro:include filename="$(find romea_mobile_base_description)/ros2_control/base2FWSxxx.ros2_control.xacro" />
   <xacro:macro name="base_control_parameters" params="interface_name">
     <param name="wheelbase">${wheelbase}</param>
@@ -96,4 +97,5 @@
     name="base_control"
     params="mode base_name hardware_plugin has_hardware_options:=0">
+    <xacro:base_control_model/>
     <ros2_control name="${prefix}${base_name}" type="system">
       <xacro:base_control_hardware

File: romea_mobile_base_description/ros2_control/base2FWS2RWD.ros2_control.xacro (robot description, xacro)
@@ -1,4 +1,5 @@
 <?xml version="1.0"?>
 <robot xmlns:xacro="http://www.ros.org/wiki/xacro">
+  <xacro:include filename="$(find romea_mobile_base_description)/ros2_control/base2FWSxxx.ros2_control.xacro" />
   <xacro:macro name="base_control_parameters" params="interface_name">
     <param name="wheelbase">${wheelbase}</param>
@@ -94,4 +95,5 @@
     name="base_control"
     params="mode base_name hardware_plugin has_hardware_options:=0">
+    <xacro:base_control_model/>
     <ros2_control name="${prefix}${base_name}" type="system">
       <xacro:base_control_hardware

File: romea_mobile_base_description/ros2_control/base2FWS4WD.ros2_control.xacro (robot description, xacro)
@@ -1,4 +1,5 @@
 <?xml version="1.0"?>
 <robot xmlns:xacro="http://www.ros.org/wiki/xacro">
+  <xacro:include filename="$(find romea_mobile_base_description)/ros2_control/base2FWSxxx.ros2_control.xacro" />
   <xacro:macro name="base_control_parameters" params="interface_name">
     <param name="wheelbase">${wheelbase}</param>
@@ -88,4 +89,5 @@
     name="base_control"
     params="mode base_name hardware_plugin has_hardware_options:=0">
+    <xacro:base_control_model/>
     <ros2_control name="${prefix}${base_name}" type="system">
       <xacro:base_control_hardware

File: romea_mobile_base_description/ros2_control/base2TD.ros2_control.xacro (robot description, xacro)
@@ -1,4 +1,37 @@
 <?xml version="1.0"?>
 <robot xmlns:xacro="http://www.ros.org/wiki/xacro">
+  <xacro:include filename="$(find romea_mobile_base_description)/ros2_control/base_control_joints.xacro" />
+  <xacro:macro name="base_control_model">
+    <link name="${prefix}${base_footprint_link}" />
+    <link name="${prefix}${base_link}" />
+    <joint name="${prefix}${base_footprint_joint}" type="fixed">
+      <parent link="${prefix}${base_footprint_link}" />
+      <child link="${prefix}${base_link}" />
+    </joint>
+    <xacro:base_control_continuous_joint
+      parent_link="${base_link}"
+      child_link="${left_sprocket_wheel_spinning_link}"
+      joint_name="${left_sprocket_wheel_spinning_joint}"
+      velocity="${maximal_wheel_speed/(sprocket_wheel_radius+track_thickness)}"
+      effort="${maximal_wheel_torque}" />
+    <xacro:base_control_continuous_joint
+      parent_link="${base_link}"
+      child_link="${right_sprocket_wheel_spinning_link}"
+      joint_name="${right_sprocket_wheel_spinning_joint}"
+      velocity="${maximal_wheel_speed/(sprocket_wheel_radius+track_thickness)}"
+      effort="${maximal_wheel_torque}" />
+    <xacro:base_control_continuous_joint
+      parent_link="${base_link}"
+      child_link="${left_idler_wheel_spinning_link}"
+      joint_name="${left_idler_wheel_spinning_joint}"
+      velocity="${maximal_wheel_speed/(idler_wheel_radius+track_thickness)}"
+      effort="${maximal_wheel_torque}" />
+    <xacro:base_control_continuous_joint
+      parent_link="${base_link}"
+      child_link="${right_idler_wheel_spinning_link}"
+      joint_name="${right_idler_wheel_spinning_joint}"
+      velocity="${maximal_wheel_speed/(idler_wheel_radius+track_thickness)}"
+      effort="${maximal_wheel_torque}" />
+  </xacro:macro>
   <xacro:macro name="base_control_parameters" params="interface_name">
     <param name="sprocket_wheel_radius">${sprocket_wheel_radius}</param>
@@ -73,4 +106,5 @@
     name="base_control"
     params="mode base_name hardware_plugin has_hardware_options:=0">
+    <xacro:base_control_model/>
     <ros2_control name="${prefix}${base_name}" type="system">
       <xacro:base_control_hardware

File: romea_mobile_base_description/ros2_control/base2THD.ros2_control.xacro (robot description, xacro)
@@ -1,4 +1,49 @@
 <?xml version="1.0"?>
 <robot xmlns:xacro="http://www.ros.org/wiki/xacro">
+  <xacro:include filename="$(find romea_mobile_base_description)/ros2_control/base_control_joints.xacro" />
+  <xacro:macro name="base_control_model">
+    <link name="${prefix}${base_footprint_link}" />
+    <link name="${prefix}${base_link}" />
+    <joint name="${prefix}${base_footprint_joint}" type="fixed">
+      <parent link="${prefix}${base_footprint_link}" />
+      <child link="${prefix}${base_link}" />
+    </joint>
+    <xacro:base_control_continuous_joint
+      parent_link="${base_link}"
+      child_link="${left_sprocket_wheel_spinning_link}"
+      joint_name="${left_sprocket_wheel_spinning_joint}"
+      velocity="${maximal_wheel_speed/(sprocket_wheel_radius+track_thickness)}"
+      effort="${maximal_wheel_torque}" />
+    <xacro:base_control_continuous_joint
+      parent_link="${base_link}"
+      child_link="${right_sprocket_wheel_spinning_link}"
+      joint_name="${right_sprocket_wheel_spinning_joint}"
+      velocity="${maximal_wheel_speed/(sprocket_wheel_radius+track_thickness)}"
+      effort="${maximal_wheel_torque}" />
+    <xacro:base_control_continuous_joint
+      parent_link="${base_link}"
+      child_link="${front_left_idler_wheel_spinning_link}"
+      joint_name="${front_left_idler_wheel_spinning_joint}"
+      velocity="${maximal_wheel_speed/(idler_wheel_radius+track_thickness)}"
+      effort="${maximal_wheel_torque}" />
+    <xacro:base_control_continuous_joint
+      parent_link="${base_link}"
+      child_link="${front_right_idler_wheel_spinning_link}"
+      joint_name="${front_right_idler_wheel_spinning_joint}"
+      velocity="${maximal_wheel_speed/(idler_wheel_radius+track_thickness)}"
+      effort="${maximal_wheel_torque}" />
+    <xacro:base_control_continuous_joint
+      parent_link="${base_link}"
+      child_link="${rear_left_idler_wheel_spinning_link}"
+      joint_name="${rear_left_idler_wheel_spinning_joint}"
+      velocity="${maximal_wheel_speed/(idler_wheel_radius+track_thickness)}"
+      effort="${maximal_wheel_torque}" />
+    <xacro:base_control_continuous_joint
+      parent_link="${base_link}"
+      child_link="${rear_right_idler_wheel_spinning_link}"
+      joint_name="${rear_right_idler_wheel_spinning_joint}"
+      velocity="${maximal_wheel_speed/(idler_wheel_radius+track_thickness)}"
+      effort="${maximal_wheel_torque}" />
+  </xacro:macro>
   <xacro:macro name="base_control_joints" params="mode">
       <joint name="${prefix}${left_sprocket_wheel_spinning_joint}">
@@ -95,4 +140,5 @@
     name="base_control"
     params="mode base_name hardware_plugin has_hardware_options:=0">
+    <xacro:base_control_model/>
     <ros2_control name="${prefix}${base_name}" type="system">
       <xacro:base_control_hardware

File: romea_mobile_base_description/ros2_control/base2TTD.ros2_control.xacro (robot description, xacro)
@@ -1,4 +1,61 @@
 <?xml version="1.0"?>
 <robot xmlns:xacro="http://www.ros.org/wiki/xacro">
+  <xacro:include filename="$(find romea_mobile_base_description)/ros2_control/base_control_joints.xacro" />
+  <xacro:macro name="base_control_model">
+    <link name="${prefix}${base_footprint_link}" />
+    <link name="${prefix}${base_link}" />
+    <joint name="${prefix}${base_footprint_joint}" type="fixed">
+      <parent link="${prefix}${base_footprint_link}" />
+      <child link="${prefix}${base_link}" />
+    </joint>
+    <xacro:base_control_continuous_joint
+      parent_link="${base_link}"
+      child_link="${left_sprocket_wheel_spinning_link}"
+      joint_name="${left_sprocket_wheel_spinning_joint}"
+      velocity="${maximal_wheel_speed/(sprocket_wheel_radius+track_thickness)}"
+      effort="${maximal_wheel_torque}" />
+    <xacro:base_control_continuous_joint
+      parent_link="${base_link}"
+      child_link="${right_sprocket_wheel_spinning_link}"
+      joint_name="${right_sprocket_wheel_spinning_joint}"
+      velocity="${maximal_wheel_speed/(sprocket_wheel_radius+track_thickness)}"
+      effort="${maximal_wheel_torque}" />
+    <xacro:base_control_continuous_joint
+      parent_link="${base_link}"
+      child_link="${left_idler_wheel_spinning_link}"
+      joint_name="${left_idler_wheel_spinning_joint}"
+      velocity="${maximal_wheel_speed/(idler_wheel_radius+track_thickness)}"
+      effort="${maximal_wheel_torque}" />
+    <xacro:base_control_continuous_joint
+      parent_link="${base_link}"
+      child_link="${right_idler_wheel_spinning_link}"
+      joint_name="${right_idler_wheel_spinning_joint}"
+      velocity="${maximal_wheel_speed/(idler_wheel_radius+track_thickness)}"
+      effort="${maximal_wheel_torque}" />
+    <xacro:base_control_continuous_joint
+      parent_link="${base_link}"
+      child_link="${front_left_roller_wheel_spinning_link}"
+      joint_name="${front_left_roller_wheel_spinning_joint}"
+      velocity="${maximal_wheel_speed/(roller_wheel_radius+track_thickness)}"
+      effort="${maximal_wheel_torque}" />
+    <xacro:base_control_continuous_joint
+      parent_link="${base_link}"
+      child_link="${front_right_roller_wheel_spinning_link}"
+      joint_name="${front_right_roller_wheel_spinning_joint}"
+      velocity="${maximal_wheel_speed/(roller_wheel_radius+track_thickness)}"
+      effort="${maximal_wheel_torque}" />
+    <xacro:base_control_continuous_joint
+      parent_link="${base_link}"
+      child_link="${rear_left_roller_wheel_spinning_link}"
+      joint_name="${rear_left_roller_wheel_spinning_joint}"
+      velocity="${maximal_wheel_speed/(roller_wheel_radius+track_thickness)}"
+      effort="${maximal_wheel_torque}" />
+    <xacro:base_control_continuous_joint
+      parent_link="${base_link}"
+      child_link="${rear_right_roller_wheel_spinning_link}"
+      joint_name="${rear_right_roller_wheel_spinning_joint}"
+      velocity="${maximal_wheel_speed/(roller_wheel_radius+track_thickness)}"
+      effort="${maximal_wheel_torque}" />
+  </xacro:macro>
   <xacro:macro name="base_control_parameters" params="interface_name">
     <param name="sprocket_wheel_radius">${sprocket_wheel_radius}</param>
@@ -123,4 +180,5 @@
     name="base_control"
     params="mode base_name hardware_plugin has_hardware_options:=0">
+    <xacro:base_control_model/>
     <ros2_control name="${prefix}${base_name}" type="system">
       <xacro:base_control_hardware

File: romea_mobile_base_description/ros2_control/base4WD.ros2_control.xacro (robot description, xacro)
@@ -1,4 +1,32 @@
 <?xml version="1.0"?>
 <robot xmlns:xacro="http://www.ros.org/wiki/xacro">
+  <xacro:include filename="$(find romea_mobile_base_description)/ros2_control/base_control_joints.xacro" />
+  <xacro:macro name="base_control_model">
+    <link name="${prefix}${base_link}"/>
+    <xacro:base_control_continuous_joint
+      parent_link="${base_link}"
+      child_link="${front_left_wheel_spinning_link}"
+      joint_name="${front_left_wheel_spinning_joint}"
+      velocity="${maximal_wheel_speed/front_wheel_radius}"
+      effort="${maximal_wheel_torque}"/>
+    <xacro:base_control_continuous_joint
+      parent_link="${base_link}"
+      child_link="${front_right_wheel_spinning_link}"
+      joint_name="${front_right_wheel_spinning_joint}"
+      velocity="${maximal_wheel_speed/front_wheel_radius}"
+      effort="${maximal_wheel_torque}"/>
+    <xacro:base_control_continuous_joint
+      parent_link="${base_link}"
+      child_link="${rear_left_wheel_spinning_link}"
+      joint_name="${rear_left_wheel_spinning_joint}"
+      velocity="${maximal_wheel_speed/rear_wheel_radius}"
+      effort="${maximal_wheel_torque}"/>
+    <xacro:base_control_continuous_joint
+      parent_link="${base_link}"
+      child_link="${rear_right_wheel_spinning_link}"
+      joint_name="${rear_right_wheel_spinning_joint}"
+      velocity="${maximal_wheel_speed/rear_wheel_radius}"
+      effort="${maximal_wheel_torque}"/>
+  </xacro:macro>
   <xacro:macro name="base_control_parameters" params="interface_name">
     <param name="wheelbase">${wheelbase}</param>
@@ -72,4 +100,5 @@
     name="base_control"
     params="mode base_name hardware_plugin has_hardware_options:=0">
+    <xacro:base_control_model/>
     <ros2_control name="${prefix}${base_name}" type="system">
       <xacro:base_control_hardware
