Commit message: update ros2_control xacro files in order to be indepedent of base urdf add a way get elapsed time between two get_joint_state_command
Signed-off-by: Jean Laneurit <jean.laneurit@inrae.fr>

File: romea_mobile_base_description/ros2_control/base4WS4WD.ros2_control.xacro (robot description, xacro)
@@ -1,4 +1,64 @@
 <?xml version="1.0"?>
 <robot xmlns:xacro="http://www.ros.org/wiki/xacro">
+  <xacro:include filename="$(find romea_mobile_base_description)/ros2_control/base_control_joints.xacro" />
+  <xacro:macro name="base_control_model">
+    <link name="${prefix}${base_link}"/>
+    <xacro:base_control_revolute_joint
+      parent_link="${base_link}"
+      child_link="${front_left_wheel_steering_link}"
+      joint_name="${front_left_wheel_steering_joint}"
+      velocity="${maximal_wheel_steering_angular_speed}"
+      effort="${maximal_wheel_steering_torque}"
+      lower="${-maximal_wheel_steering_angle}"
+      upper="${maximal_wheel_steering_angle}"/>
+    <xacro:base_control_revolute_joint
+      parent_link="${base_link}"
+      child_link="${front_right_wheel_steering_link}"
+      joint_name="${front_right_wheel_steering_joint}"
+      velocity="${maximal_wheel_steering_angular_speed}"
+      effort="${maximal_wheel_steering_torque}"
+      lower="${-maximal_wheel_steering_angle}"
+      upper="${maximal_wheel_steering_angle}"/>
+    <xacro:base_control_revolute_joint
+      parent_link="${base_link}"
+      child_link="${rear_left_wheel_steering_link}"
+      joint_name="${rear_left_wheel_steering_joint}"
+      velocity="${maximal_wheel_steering_angular_speed}"
+      effort="${maximal_wheel_steering_torque}"
+      lower="${-maximal_wheel_steering_angle}"
+      upper="${maximal_wheel_steering_angle}"/>
+    <xacro:base_control_revolute_joint
+      parent_link="${base_link}"
+      child_link="${rear_right_wheel_steering_link}"
+      joint_name="${rear_right_wheel_steering_joint}"
+      velocity="${maximal_wheel_steering_angular_speed}"
+      effort="${maximal_wheel_steering_torque}"
+      lower="${-maximal_wheel_steering_angle}"
+      upper="${maximal_wheel_steering_angle}"/>
+    <xacro:base_control_continuous_joint
+      parent_link="${front_left_wheel_steering_link}"
+      child_link="${front_left_wheel_spinning_link}"
+      joint_name="${front_left_wheel_spinning_joint}"
+      velocity="${maximal_wheel_speed/front_wheel_radius}"
+      effort="${maximal_wheel_torque}"/>
+    <xacro:base_control_continuous_joint
+      parent_link="${front_right_wheel_steering_link}"
+      child_link="${front_right_wheel_spinning_link}"
+      joint_name="${front_right_wheel_spinning_joint}"
+      velocity="${maximal_wheel_speed/front_wheel_radius}"
+      effort="${maximal_wheel_torque}"/>
+    <xacro:base_control_continuous_joint
+      parent_link="${rear_left_wheel_steering_link}"
+      child_link="${rear_left_wheel_spinning_link}"
+      joint_name="${rear_left_wheel_spinning_joint}"
+      velocity="${maximal_wheel_speed/rear_wheel_radius}"
+      effort="${maximal_wheel_torque}"/>
+    <xacro:base_control_continuous_joint
+      parent_link="${rear_right_wheel_steering_link}"
+      child_link="${rear_right_wheel_spinning_link}"
+      joint_name="${rear_right_wheel_spinning_joint}"
+      velocity="${maximal_wheel_speed/rear_wheel_radius}"
+      effort="${maximal_wheel_torque}"/>
+  </xacro:macro>
   <xacro:macro name="base_control_parameters" params="interface_name">
     <param name="wheelbase">${wheelbase}</param>
@@ -104,4 +164,5 @@
     name="base_control"
     params="mode base_name hardware_plugin has_hardware_options:=0">
+    <xacro:base_control_model/>
     <ros2_control name="${prefix}${base_name}" type="system">
       <xacro:base_control_hardware

File: romea_mobile_base_description/urdf/axle_steering.xacro (robot description, xacro)
@@ -12,5 +12,9 @@
    </link>
     <joint name="${prefix}${axle_steering_joint}" type="revolute">
-      <limit lower="${minimal_axle_steering_angle}" upper="${maximal_axle_steering_angle}" effort="10000000" velocity="1000000"/>
+      <limit
+        lower="${minimal_axle_steering_angle}"
+        upper="${maximal_axle_steering_angle}"
+        effort="${maximal_axle_steering_torque}"
+        velocity="${maximal_axle_steering_angular_speed}"/>
       <parent link="${prefix}${parent_link}"/>
       <child link="${prefix}${axle_steering_link}"/>

File: romea_mobile_base_description/urdf/wheel.xacro (robot description, xacro)
@@ -6,5 +6,5 @@
       <material>Gazebo/Black</material>
     </gazebo>
-    <xacro:property name="maximal_angular_speed" value="${maximal_wheel_speed/wheel_radius}" />
+    <xacro:property name="maximal_wheel_angular_speed" value="${maximal_wheel_speed/wheel_radius}" />
     <xacro:property name="radius" value="${wheel_radius}" />
     <xacro:property name="width" value="${wheel_width}" />
@@ -57,5 +57,7 @@
     </gazebo>
     <joint name="${prefix}${wheel_spinning_joint}" type="continuous">
-      <limit effort="10000000" velocity="${maximal_angular_speed}" />
+      <limit
+        effort="${maximal_wheel_torque}"
+        velocity="${maximal_wheel_angular_speed}" />
       <parent link="${prefix}${parent_link}" />
       <child link="${prefix}${wheel_spinning_link}" />

File: romea_mobile_base_description/urdf/wheel_steered.xacro (robot description, xacro)
@@ -4,5 +4,21 @@
   <xacro:include filename="$(find romea_mobile_base_description)/urdf/wheel.xacro" />
   <xacro:macro name="wheel_steered"
-    params="parent_link wheel_steering_link wheel_steering_joint  steering_link_mass steering_link_xz steering_link_y wheel_spinning_link wheel_spinning_joint wheel_origin_x wheel_origin_y wheel_mass wheel_width wheel_radius left_right *joint_origin *visual_steering *visual_wheel">
+    params="parent_link
+            wheel_steering_link
+            wheel_steering_joint
+            steering_link_mass
+            steering_link_xz
+            steering_link_y
+            wheel_spinning_link
+            wheel_spinning_joint
+            wheel_origin_x
+            wheel_origin_y
+            wheel_mass
+            wheel_width
+            wheel_radius
+            left_right
+            *joint_origin
+            *visual_steering
+            *visual_wheel">
     <link name="${prefix}${wheel_steering_link}">
       <xacro:insert_block name="visual_steering" />
@@ -21,5 +37,6 @@
         <inertia
           ixx="${steering_link_mass/12.0 * (steering_link_y*steering_link_y + steering_link_xz*steering_link_xz)}"
-          ixy="0" ixz="0"
+          ixy="0"
+          ixz="0"
           iyy="${steering_link_mass/12.0 * (steering_link_xz*steering_link_xz + steering_link_xz*steering_link_xz)}"
           iyz="0"
@@ -28,6 +45,10 @@
     </link>
     <joint name="${prefix}${wheel_steering_joint}" type="revolute">
-      <limit lower="${minimal_wheel_steering_angle}" upper="${maximal_wheel_steering_angle}"
-        effort="10000000" velocity="1000000" />
+      <limit
+        lower="${minimal_wheel_steering_angle}"
+        upper="${maximal_wheel_steering_angle}"
+        velocity="${maximal_wheel_steering_angular_speed}"
+        effort="${maximal_wheel_steering_torque}"/>
+        <!-- effort="10000000 -->
       <axis xyz="0 0 1" />
       <parent link="${prefix}${parent_link}" />
@@ -45,5 +66,6 @@
       </joint>
     </transmission>
-    <xacro:wheel parent_link="${wheel_steering_link}"
+    <xacro:wheel
+      parent_link="${wheel_steering_link}"
       wheel_spinning_link="${wheel_spinning_link}"
       wheel_spinning_joint="${wheel_spinning_joint}"

File: romea_mobile_base_gazebo/test/test_gazebo_system_interface.xacro (robot description, xacro)
@@ -95,5 +95,7 @@
     <joint name="front_left_wheel_steering_joint">
       <command_interface name="position" />
-      <state_interface name="position" />
+      <state_interface name="position">
+        <param name="initial_value">0.25</param>
+      </state_interface>
     </joint>
     <joint name="front_right_wheel_steering_joint">

File: romea_mobile_base_gazebo/test_legacy/.xacro (robot description, xacro)
@@ -33,4 +33,5 @@
     <xacro:property name="mass_center_z" value="${props['inertia']['center'][2]}" />
     <xacro:property name="maximal_wheel_speed" value="${props['wheels_speed_control']['command']['maximal_speed']}"/>
+    <xacro:property name="maximal_wheel_torque" value="10000000" />
     <xacro:property name="body_reference_x" value="${props['control_point'][0]}" />
     <!-- Wheel Properties -->
