Commit message: fix CI errors
Signed-off-by: Jean Laneurit <jean.laneurit@inrae.fr>

File: romea_mobile_base_description/ros2_control/base2TD.ros2_control.xacro (robot description, xacro)
@@ -3,10 +3,5 @@
   <xacro:include filename="$(find romea_mobile_base_description)/ros2_control/base_control_joints.xacro" />
   <xacro:macro name="base_control_model">
-    <link name="${prefix}${base_footprint_link}" />
     <link name="${prefix}${base_link}" />
-    <joint name="${prefix}${base_footprint_joint}" type="fixed">
-      <parent link="${prefix}${base_footprint_link}" />
-      <child link="${prefix}${base_link}" />
-    </joint>
     <xacro:base_control_continuous_joint
       parent_link="${base_link}"

File: romea_mobile_base_description/ros2_control/base2THD.ros2_control.xacro (robot description, xacro)
@@ -3,10 +3,5 @@
   <xacro:include filename="$(find romea_mobile_base_description)/ros2_control/base_control_joints.xacro" />
   <xacro:macro name="base_control_model">
-    <link name="${prefix}${base_footprint_link}" />
     <link name="${prefix}${base_link}" />
-    <joint name="${prefix}${base_footprint_joint}" type="fixed">
-      <parent link="${prefix}${base_footprint_link}" />
-      <child link="${prefix}${base_link}" />
-    </joint>
     <xacro:base_control_continuous_joint
       parent_link="${base_link}"

File: romea_mobile_base_description/ros2_control/base2TTD.ros2_control.xacro (robot description, xacro)
@@ -3,10 +3,5 @@
   <xacro:include filename="$(find romea_mobile_base_description)/ros2_control/base_control_joints.xacro" />
   <xacro:macro name="base_control_model">
-    <link name="${prefix}${base_footprint_link}" />
     <link name="${prefix}${base_link}" />
-    <joint name="${prefix}${base_footprint_joint}" type="fixed">
-      <parent link="${prefix}${base_footprint_link}" />
-      <child link="${prefix}${base_link}" />
-    </joint>
     <xacro:base_control_continuous_joint
       parent_link="${base_link}"
