Commit message: mobile_base_hardware : add test for 2FWS2RD, 2FWS4WD , 2TD, 2THD, 2TTD vehicles

File: romea_mobile_base_hardware/test/test_hardware_interface1FAS2RWD.xacro (robot description, xacro)
@@ -3,11 +3,11 @@
   <xacro:property name="prefix" value="robot_"/>
   <xacro:property name="front_axle_steering_joint" value="joint1"/>
-  <xacro:property name="front_left_wheel_spinning_joint" value="joint2"/>
-  <xacro:property name="front_right_wheel_spinning_joint" value="joint3"/>
+  <xacro:property name="rear_left_wheel_spinning_joint" value="joint2"/>
+  <xacro:property name="rear_right_wheel_spinning_joint" value="joint3"/>
   <xacro:property name="front_left_wheel_steering_joint" value="joint4"/>
   <xacro:property name="front_right_wheel_steering_joint" value="joint5"/>
-  <xacro:property name="rear_left_wheel_spinning_joint" value="joint6"/>
-  <xacro:property name="rear_right_wheel_spinning_joint" value="joint7"/>
-  <xacro:include filename="$(find romea_mobile_base_description)/ros2_control/1FAS_2FWD.ros2_control.xacro" />
+  <xacro:property name="front_left_wheel_spinning_joint" value="joint6"/>
+  <xacro:property name="front_right_wheel_spinning_joint" value="joint7"/>
+  <xacro:include filename="$(find romea_mobile_base_description)/ros2_control/1FAS_2RWD.ros2_control.xacro" />
   <xacro:base_control mode="test"/>
 </robot>
