Commit message: mobile_base_hardware : update unit tests

File: romea_mobile_base_hardware/test/test_hardware_interface1FWS2RWD.xacro (robot description, xacro)
@@ -3,7 +3,7 @@
   <xacro:property name="prefix" value="robot_"/>
   <xacro:property name="front_wheel_steering_joint" value="joint1"/>
-  <xacro:property name="front_wheel_spinning_joint" value="joint2"/>
-  <xacro:property name="rear_left_wheel_spinning_joint" value="joint3"/>
-  <xacro:property name="rear_right_wheel_spinning_joint" value="joint4"/>
+  <xacro:property name="rear_left_wheel_spinning_joint" value="joint2"/>
+  <xacro:property name="rear_right_wheel_spinning_joint" value="joint3"/>
+  <xacro:property name="front_wheel_spinning_joint" value="joint4"/>
   <xacro:include filename="$(find romea_mobile_base_description)/ros2_control/1FWS_2RWD.ros2_control.xacro" />
   <xacro:base_control mode="test"/>

File: romea_mobile_base_hardware/test/test_hardware_interface2AS4WD.xacro (robot description, xacro)
@@ -4,12 +4,12 @@
   <xacro:property name="front_axle_steering_joint" value="joint1"/>
   <xacro:property name="rear_axle_steering_joint" value="joint2"/>
-  <xacro:property name="front_left_wheel_steering_joint" value="joint3"/>
-  <xacro:property name="front_right_wheel_steering_joint" value="joint4"/>
-  <xacro:property name="rear_left_wheel_steering_joint" value="joint5"/>
-  <xacro:property name="rear_right_wheel_steering_joint" value="joint6"/>
-  <xacro:property name="front_left_wheel_spinning_joint" value="joint7"/>
-  <xacro:property name="front_right_wheel_spinning_joint" value="joint8"/>
-  <xacro:property name="rear_left_wheel_spinning_joint" value="joint9"/>
-  <xacro:property name="rear_right_wheel_spinning_joint" value="joint10"/>
+  <xacro:property name="front_left_wheel_spinning_joint" value="joint3"/>
+  <xacro:property name="front_right_wheel_spinning_joint" value="joint4"/>
+  <xacro:property name="rear_left_wheel_spinning_joint" value="joint5"/>
+  <xacro:property name="rear_right_wheel_spinning_joint" value="joint6"/>
+  <xacro:property name="front_left_wheel_steering_joint" value="joint7"/>
+  <xacro:property name="front_right_wheel_steering_joint" value="joint8"/>
+  <xacro:property name="rear_left_wheel_steering_joint" value="joint9"/>
+  <xacro:property name="rear_right_wheel_steering_joint" value="joint10"/>
   <xacro:include filename="$(find romea_mobile_base_description)/ros2_control/2AS_4WD.ros2_control.xacro" />
   <xacro:base_control mode="test"/>

File: romea_mobile_base_hardware/test/test_hardware_interface2FWS2RWD.xacro (robot description, xacro)
@@ -4,8 +4,8 @@
   <xacro:property name="front_left_wheel_steering_joint" value="joint1"/>
   <xacro:property name="front_right_wheel_steering_joint" value="joint2"/>
-  <xacro:property name="front_left_wheel_spinning_joint" value="joint3"/>
-  <xacro:property name="front_right_wheel_spinning_joint" value="joint4"/>
-  <xacro:property name="rear_left_wheel_spinning_joint" value="joint5"/>
-  <xacro:property name="rear_right_wheel_spinning_joint" value="joint6"/>
+  <xacro:property name="rear_left_wheel_spinning_joint" value="joint3"/>
+  <xacro:property name="rear_right_wheel_spinning_joint" value="joint4"/>
+  <xacro:property name="front_left_wheel_spinning_joint" value="joint5"/>
+  <xacro:property name="front_right_wheel_spinning_joint" value="joint6"/>
   <xacro:include filename="$(find romea_mobile_base_description)/ros2_control/2FWS_2RWD.ros2_control.xacro" />
   <xacro:base_control mode="test"/>

File: romea_mobile_base_simulation/test/test_hardware_interface1FAS2FWD.xacro (robot description, xacro)
@@ -3,8 +3,8 @@
   <xacro:property name="prefix" value="robot_"/>
   <xacro:property name="front_axle_steering_joint" value="joint1"/>
-  <xacro:property name="front_left_wheel_spinning_joint" value="joint2"/>
-  <xacro:property name="front_right_wheel_spinning_joint" value="joint3"/>
-  <xacro:property name="front_left_wheel_steering_joint" value="joint4"/>
-  <xacro:property name="front_right_wheel_steering_joint" value="joint5"/>
+  <xacro:property name="front_left_wheel_steering_joint" value="joint2"/>
+  <xacro:property name="front_right_wheel_steering_joint" value="joint3"/>
+  <xacro:property name="front_left_wheel_spinning_joint" value="joint4"/>
+  <xacro:property name="front_right_wheel_spinning_joint" value="joint5"/>
   <xacro:property name="rear_left_wheel_spinning_joint" value="joint6"/>
   <xacro:property name="rear_right_wheel_spinning_joint" value="joint7"/>
