Commit message: harware: update xacro files used by unit tests
Signed-off-by: jean.laneurit <jean.laneurit@inrae.fr>

File: romea_mobile_base_hardware/test/test_hardware_interface1FAS2FWD.xacro (robot description, xacro)
@@ -9,4 +9,9 @@
   <xacro:property name="rear_left_wheel_spinning_joint" value="joint6" />
   <xacro:property name="rear_right_wheel_spinning_joint" value="joint7" />
+  <xacro:property name="rear_right_wheel_spinning_joint" value="joint7" />
+  <xacro:property name="rear_right_wheel_spinning_joint" value="joint7" />
+  <xacro:property name="front_wheel_radius" value="0.2" />
+  <xacro:property name="maximal_axle_steering_angle" value="0.5" />
+  <xacro:property name="maximal_wheel_speed" value="1.0" />
   <xacro:include
     filename="$(find romea_mobile_base_description)/ros2_control/base1FAS2FWD.ros2_control.xacro" />

File: romea_mobile_base_hardware/test/test_hardware_interface1FAS2RWD.xacro (robot description, xacro)
@@ -9,4 +9,7 @@
   <xacro:property name="front_left_wheel_spinning_joint" value="joint6" />
   <xacro:property name="front_right_wheel_spinning_joint" value="joint7" />
+  <xacro:property name="rear_wheel_radius" value="0.2" />
+  <xacro:property name="maximal_axle_steering_angle" value="0.5" />
+  <xacro:property name="maximal_wheel_speed" value="1.0" />
   <xacro:include
     filename="$(find romea_mobile_base_description)/ros2_control/base1FAS2RWD.ros2_control.xacro" />

File: romea_mobile_base_hardware/test/test_hardware_interface1FAS4WD.xacro (robot description, xacro)
@@ -9,4 +9,8 @@
   <xacro:property name="front_left_wheel_steering_joint" value="joint6" />
   <xacro:property name="front_right_wheel_steering_joint" value="joint7" />
+  <xacro:property name="rear_wheel_radius" value="0.2" />
+  <xacro:property name="front_wheel_radius" value="0.2" />
+  <xacro:property name="maximal_axle_steering_angle" value="0.5" />
+  <xacro:property name="maximal_wheel_speed" value="1.0" />
   <xacro:include
     filename="$(find romea_mobile_base_description)/ros2_control/base1FAS4WD.ros2_control.xacro" />

File: romea_mobile_base_hardware/test/test_hardware_interface2AS2FWD.xacro (robot description, xacro)
@@ -12,6 +12,9 @@
   <xacro:property name="rear_left_wheel_spinning_joint" value="joint9" />
   <xacro:property name="rear_right_wheel_spinning_joint" value="joint10" />
+  <xacro:property name="front_wheel_radius" value="0.2" />
+  <xacro:property name="maximal_axle_steering_angle" value="0.5" />
+  <xacro:property name="maximal_wheel_speed" value="1.0" />
   <xacro:include
-    filename="$(find romea_mobile_base_description)/ros2_control/base2AS4WD.ros2_control.xacro" />
+    filename="$(find romea_mobile_base_description)/ros2_control/base2AS2FWD.ros2_control.xacro" />
   <xacro:base_control mode="test" base_name="base" />
 </robot>

File: romea_mobile_base_hardware/test/test_hardware_interface2AS2RWD.xacro (robot description, xacro)
@@ -12,6 +12,9 @@
   <xacro:property name="front_left_wheel_spinning_joint" value="joint9" />
   <xacro:property name="front_right_wheel_spinning_joint" value="joint10" />
+  <xacro:property name="rear_wheel_radius" value="0.2" />
+  <xacro:property name="maximal_axle_steering_angle" value="0.5" />
+  <xacro:property name="maximal_wheel_speed" value="1.0" />
   <xacro:include
-    filename="$(find romea_mobile_base_description)/ros2_control/base2AS4WD.ros2_control.xacro" />
+    filename="$(find romea_mobile_base_description)/ros2_control/base2AS2RWD.ros2_control.xacro" />
   <xacro:base_control mode="test" base_name="base" />
 </robot>

File: romea_mobile_base_hardware/test/test_hardware_interface2AS4WD.xacro (robot description, xacro)
@@ -12,4 +12,8 @@
   <xacro:property name="rear_left_wheel_steering_joint" value="joint9" />
   <xacro:property name="rear_right_wheel_steering_joint" value="joint10" />
+  <xacro:property name="rear_wheel_radius" value="0.2" />
+  <xacro:property name="front_wheel_radius" value="0.2" />
+  <xacro:property name="maximal_axle_steering_angle" value="0.5" />
+  <xacro:property name="maximal_wheel_speed" value="1.0" />
   <xacro:include
     filename="$(find romea_mobile_base_description)/ros2_control/base2AS4WD.ros2_control.xacro" />

File: romea_mobile_base_hardware/test/test_hardware_interface2FWS2FWD.xacro (robot description, xacro)
@@ -8,4 +8,7 @@
   <xacro:property name="rear_left_wheel_spinning_joint" value="joint5" />
   <xacro:property name="rear_right_wheel_spinning_joint" value="joint6" />
+  <xacro:property name="maximal_wheel_steering_angle" value="0.5" />
+  <xacro:property name="maximal_wheel_speed" value="1.0" />
+  <xacro:property name="front_wheel_radius" value="0.2" />
   <xacro:include
     filename="$(find romea_mobile_base_description)/ros2_control/base2FWS2FWD.ros2_control.xacro" />

File: romea_mobile_base_hardware/test/test_hardware_interface2FWS2RWD.xacro (robot description, xacro)
@@ -8,4 +8,7 @@
   <xacro:property name="front_left_wheel_spinning_joint" value="joint5" />
   <xacro:property name="front_right_wheel_spinning_joint" value="joint6" />
+  <xacro:property name="maximal_wheel_steering_angle" value="0.5" />
+  <xacro:property name="maximal_wheel_speed" value="1.0" />
+  <xacro:property name="rear_wheel_radius" value="0.2" />
   <xacro:include
     filename="$(find romea_mobile_base_description)/ros2_control/base2FWS2RWD.ros2_control.xacro" />

File: romea_mobile_base_hardware/test/test_hardware_interface2FWS4WD.xacro (robot description, xacro)
@@ -8,4 +8,8 @@
   <xacro:property name="rear_left_wheel_spinning_joint" value="joint5" />
   <xacro:property name="rear_right_wheel_spinning_joint" value="joint6" />
+  <xacro:property name="maximal_wheel_steering_angle" value="0.5" />
+  <xacro:property name="maximal_wheel_speed" value="1.0" />
+  <xacro:property name="front_wheel_radius" value="0.2" />
+  <xacro:property name="rear_wheel_radius" value="0.2" />
   <xacro:include
     filename="$(find romea_mobile_base_description)/ros2_control/base2FWS4WD.ros2_control.xacro" />

File: romea_mobile_base_hardware/test/test_hardware_interface2TD.xacro (robot description, xacro)
@@ -6,4 +6,8 @@
   <xacro:property name="left_idler_wheel_spinning_joint" value="joint3" />
   <xacro:property name="right_idler_wheel_spinning_joint" value="joint4" />
+  <xacro:property name="maximal_wheel_speed" value="1.0" />
+  <xacro:property name="sprocket_wheel_radius" value="0.2" />
+  <xacro:property name="idler_wheel_radius" value="0.15" />
+  <xacro:property name="track_thickness" value="0.2" />
   <xacro:include
     filename="$(find romea_mobile_base_description)/ros2_control/base2TD.ros2_control.xacro" />

File: romea_mobile_base_hardware/test/test_hardware_interface2THD.xacro (robot description, xacro)
@@ -8,4 +8,8 @@
   <xacro:property name="rear_left_idler_wheel_spinning_joint" value="joint5" />
   <xacro:property name="rear_right_idler_wheel_spinning_joint" value="joint6" />
+  <xacro:property name="maximal_wheel_speed" value="1.0" />
+  <xacro:property name="sprocket_wheel_radius" value="0.2" />
+  <xacro:property name="idler_wheel_radius" value="0.15" />
+  <xacro:property name="track_thickness" value="0.2" />
   <xacro:include
     filename="$(find romea_mobile_base_description)/ros2_control/base2THD.ros2_control.xacro" />

File: romea_mobile_base_hardware/test/test_hardware_interface2TTD.xacro (robot description, xacro)
@@ -10,4 +10,8 @@
   <xacro:property name="rear_left_roller_wheel_spinning_joint" value="joint7" />
   <xacro:property name="rear_right_roller_wheel_spinning_joint" value="joint8" />
+  <xacro:property name="maximal_wheel_speed" value="1.0" />
+  <xacro:property name="sprocket_wheel_radius" value="0.2" />
+  <xacro:property name="idler_wheel_radius" value="0.15" />
+  <xacro:property name="track_thickness" value="0.2" />
   <xacro:include
     filename="$(find romea_mobile_base_description)/ros2_control/base2TTD.ros2_control.xacro" />

File: romea_mobile_base_hardware/test/test_hardware_interface2WD.xacro (robot description, xacro)
@@ -6,4 +6,6 @@
   <xacro:property name="left_idler_wheel_spinning_joint" value="joint3" />
   <xacro:property name="right_idler_wheel_spinning_joint" value="joint4" />
+  <xacro:property name="maximal_wheel_speed" value="1.0" />
+  <xacro:property name="wheel_radius" value="0.2" />
   <xacro:include
     filename="$(find romea_mobile_base_description)/ros2_control/base2TD.ros2_control.xacro" />

File: romea_mobile_base_hardware/test/test_hardware_interface4WD.xacro (robot description, xacro)
@@ -6,4 +6,7 @@
   <xacro:property name="rear_left_wheel_spinning_joint" value="joint3" />
   <xacro:property name="rear_right_wheel_spinning_joint" value="joint4" />
+  <xacro:property name="maximal_wheel_speed" value="1.0" />
+  <xacro:property name="front_wheel_radius" value="0.2" />
+  <xacro:property name="rear_wheel_radius" value="0.2" />
   <xacro:include
     filename="$(find romea_mobile_base_description)/ros2_control/base4WD.ros2_control.xacro" />

File: romea_mobile_base_hardware/test/test_hardware_interface4WS4WD.xacro (robot description, xacro)
@@ -10,4 +10,8 @@
   <xacro:property name="rear_left_wheel_spinning_joint" value="joint7" />
   <xacro:property name="rear_right_wheel_spinning_joint" value="joint8" />
+  <xacro:property name="maximal_wheel_steering_angle" value="0.5" />
+  <xacro:property name="maximal_wheel_speed" value="1.0" />
+  <xacro:property name="front_wheel_radius" value="0.2" />
+  <xacro:property name="rear_wheel_radius" value="0.2" />
   <xacro:include
     filename="$(find romea_mobile_base_description)/ros2_control/base4WS4WD.ros2_control.xacro" />
