Commit message: mobile_base_description : add 2THD and 2TTD chassis support

File: romea_mobile_base_description/urdf/base2TD.chassis.xacro (robot description, xacro)
@@ -3,5 +3,5 @@
   <xacro:include filename="$(find romea_mobile_base_description)/urdf/common.xacro" />
   <xacro:include filename="$(find romea_mobile_base_description)/urdf/wheel.xacro" />
-  <xacro:macro name="chassis" params="*visual_chassis *visual_wheel">
+  <xacro:macro name="chassis" params="*visual_chassis *visual_sprocket_wheel *visual_idler_wheel">
     <xacro:common>
       <xacro:insert_block name="visual_chassis"/>
@@ -11,9 +11,9 @@
                 wheel_spinning_joint="${left_sprocket_wheel_spinning_joint}"
                 wheel_mass="${sprocket_wheel_mass}"
-                wheel_width="${track_wheel_width}"
-                wheel_radius="${sprocket_wheel_radius}"
+                wheel_width="${track_width}"
+                wheel_radius="${sprocket_wheel_radius+track_thickness}"
                 left_right="-1">
-      <origin xyz="${sprocket_wheel_x-body_reference_x} ${track/2} ${sprocket_wheel_radius - chassis_height}" rpy="${-M_PI/2} 0 0" />
-      <xacro:insert_block name="visual_wheel"/>
+      <origin xyz="${-wheelbase/2-body_reference_x} ${track/2} ${sprocket_wheel_radius - chassis_height}" rpy="${-M_PI/2} 0 0" />
+      <xacro:insert_block name="visual_sprocket_wheel"/>
     </xacro:wheel>
     <xacro:wheel parent_link="${base_link}"
@@ -22,18 +22,18 @@
                  wheel_mass="${sprocket_wheel_mass}"
                  wheel_width="${track_width}"
-                 wheel_radius="${sprocket_wheel_radius}"
+                 wheel_radius="${sprocket_wheel_radius+track_thickness}"
                  left_right="1">
-      <origin xyz="${sprocket_wheel_x-body_reference_x} ${-track/2} ${sprocket_wheel_radius - chassis_height}" rpy="${-M_PI/2} 0 0" />
-      <xacro:insert_block name="visual_wheel"/>
+      <origin xyz="${-wheelbase/2-body_reference_x} ${-track/2} ${sprocket_wheel_radius - chassis_height}" rpy="${-M_PI/2} 0 0" />
+      <xacro:insert_block name="visual_sprocket_wheel"/>
     </xacro:wheel>
     <xacro:wheel parent_link="${base_link}"
-                 wheel_spinning_link="${left_idler_spinning_link}"
-                 wheel_spinning_joint="${left_idler_spinning_joint}"
+                 wheel_spinning_link="${left_idler_wheel_spinning_link}"
+                 wheel_spinning_joint="${left_idler_wheel_spinning_joint}"
                  wheel_mass="${idler_wheel_mass}"
                  wheel_width="${track_width}"
-                 wheel_radius="${idler_wheel_radius}"
+                 wheel_radius="${idler_wheel_radius+track_thickness}"
                  left_right="-1">
-      <origin xyz="${idler_wheel_x-body_reference_x} ${track/2} ${idler_wheel_radius - chassis_height}" rpy="${-M_PI/2} 0 0" />
-      <xacro:insert_block name="visual_wheel"/>
+      <origin xyz="${wheelbase/2-body_reference_x} ${track/2} ${idler_wheel_radius - chassis_height}" rpy="${-M_PI/2} 0 0" />
+      <xacro:insert_block name="visual_idler_wheel"/>
     </xacro:wheel>
     <xacro:wheel parent_link="${base_link}"
@@ -42,8 +42,8 @@
                  wheel_mass="${idler_wheel_mass}"
                  wheel_width="${track_width}"
-                 wheel_radius="${idler_wheel_radius}"
+                 wheel_radius="${idler_wheel_radius+track_thickness}"
                  left_right="1">
-      <origin xyz="${idler_wheel_x-body_reference_x} ${-track/2} ${idler_wheel_radius - chassis_height}" rpy="${-M_PI/2} 0 0" />
-      <xacro:insert_block name="visual_wheel"/>
+      <origin xyz="${wheelbase/2-body_reference_x} ${-track/2} ${idler_wheel_radius - chassis_height}" rpy="${-M_PI/2} 0 0" />
+      <xacro:insert_block name="visual_idler_wheel"/>
     </xacro:wheel>
   </xacro:macro>

File: romea_mobile_base_description/urdf/common.xacro (robot description, xacro)
@@ -15,5 +15,6 @@
           <box size="${aabb_length} ${aabb_width} ${aabb_height}"/>
         </geometry>
-        <origin xyz="${-body_reference_x} 0 ${ground_clearance+aabb_height/2-chassis_height}" rpy="0 0 0" />
+        <origin xyz="${aabb_center_x-body_reference_x} ${aabb_center_y} ${aabb_center_z-chassis_height}" rpy="0 0 0" />
+<!--        <origin xyz="${-body_reference_x} 0 ${ground_clearance+aabb_height/2-chassis_height}" rpy="0 0 0" />-->
       </collision>
     </link>
