Commit message: description: add rear and wheel visuas for 1FAS, 2FWS and 4WD robots
Signed-off-by: Jean Laneurit <jean.laneurit@inrae.fr>

File: romea_mobile_base_description/urdf/base1FASxxx.chassis.xacro (robot description, xacro)
@@ -5,5 +5,5 @@
   <xacro:include filename="$(find romea_mobile_base_description)/urdf/wheel_steered.xacro" />
   <xacro:include filename="$(find romea_mobile_base_description)/urdf/axle_steering.xacro" />
-  <xacro:macro name="chassis" params="*visual_chassis *visual_steering *visual_wheel">
+  <xacro:macro name="chassis" params="*visual_chassis *visual_front_steering *visual_front_wheel *visual_rear_wheel">
     <xacro:common>
       <xacro:insert_block name="visual_chassis"/>
@@ -25,6 +25,6 @@
                          left_right="-1">
        <origin xyz="${wheelbase/2-body_reference_x} ${front_track/2} ${front_wheel_radius - chassis_height}" rpy="0 0 0" />
-       <xacro:insert_block name="visual_steering"/>
-       <xacro:insert_block name="visual_wheel"/>
+       <xacro:insert_block name="visual_front_steering"/>
+       <xacro:insert_block name="visual_front_wheel"/>
      </xacro:wheel_steered>
      <xacro:wheel_steered parent_link="${base_link}"
@@ -39,6 +39,6 @@
                           left_right="1">
        <origin xyz="${wheelbase/2-body_reference_x} ${-front_track/2} ${front_wheel_radius - chassis_height}" rpy="0 0 0" />
-       <xacro:insert_block name="visual_steering"/>
-       <xacro:insert_block name="visual_wheel"/>
+       <xacro:insert_block name="visual_front_steering"/>
+       <xacro:insert_block name="visual_front_wheel"/>
      </xacro:wheel_steered>
      <xacro:wheel parent_link="${base_link}"
@@ -50,5 +50,5 @@
                   left_right="-1">
       <origin xyz="${-wheelbase/2-body_reference_x} ${rear_track/2} ${rear_wheel_radius  - chassis_height}" rpy="${-M_PI/2} 0 0" />
-      <xacro:insert_block name="visual_wheel"/>
+      <xacro:insert_block name="visual_rear_wheel"/>
     </xacro:wheel>
     <xacro:wheel parent_link="${base_link}"
@@ -60,5 +60,5 @@
                  left_right="1">
       <origin xyz="${-wheelbase/2-body_reference_x} ${-rear_track/2} ${rear_wheel_radius - chassis_height}" rpy="${-M_PI/2} 0 0" />
-      <xacro:insert_block name="visual_wheel"/>
+      <xacro:insert_block name="visual_rear_wheel"/>
     </xacro:wheel>
   </xacro:macro>

File: romea_mobile_base_description/urdf/base2FWSxxx.chassis.xacro (robot description, xacro)
@@ -4,5 +4,5 @@
   <xacro:include filename="$(find romea_mobile_base_description)/urdf/wheel.xacro" />
   <xacro:include filename="$(find romea_mobile_base_description)/urdf/wheel_steered.xacro" />
-  <xacro:macro name="chassis" params="*visual_chassis *visual_steering *visual_wheel">
+  <xacro:macro name="chassis" params="*visual_chassis *visual_front_steering *visual_front_wheel *visual_rear_wheel">
     <xacro:common>
       <xacro:insert_block name="visual_chassis"/>
@@ -19,6 +19,6 @@
                          left_right="-1">
        <origin xyz="${wheelbase/2-body_reference_x} ${front_track/2} ${front_wheel_radius - chassis_height}" rpy="0 0 0" />
-       <xacro:insert_block name="visual_steering"/>
-       <xacro:insert_block name="visual_wheel"/>
+       <xacro:insert_block name="visual_front_steering"/>
+       <xacro:insert_block name="visual_front_wheel"/>
      </xacro:wheel_steered>
      <xacro:wheel_steered parent_link="${base_link}"
@@ -33,6 +33,6 @@
                           left_right="1">
        <origin xyz="${wheelbase/2-body_reference_x} ${-front_track/2} ${front_wheel_radius - chassis_height}" rpy="0 0 0" />
-       <xacro:insert_block name="visual_steering"/>
-       <xacro:insert_block name="visual_wheel"/>
+       <xacro:insert_block name="visual_front_steering"/>
+       <xacro:insert_block name="visual_front_wheel"/>
      </xacro:wheel_steered>
      <xacro:wheel parent_link="${base_link}"
@@ -44,5 +44,5 @@
                   left_right="-1">
       <origin xyz="${-wheelbase/2-body_reference_x} ${rear_track/2} ${rear_wheel_radius  - chassis_height}" rpy="${-M_PI/2} 0 0" />
-      <xacro:insert_block name="visual_wheel"/>
+      <xacro:insert_block name="visual_rear_wheel"/>
     </xacro:wheel>
     <xacro:wheel parent_link="${base_link}"
@@ -54,5 +54,5 @@
                  left_right="1">
       <origin xyz="${-wheelbase/2-body_reference_x} ${-rear_track/2} ${rear_wheel_radius - chassis_height}" rpy="${-M_PI/2} 0 0" />
-      <xacro:insert_block name="visual_wheel"/>
+      <xacro:insert_block name="visual_rear_wheel"/>
     </xacro:wheel>
   </xacro:macro>

File: romea_mobile_base_description/urdf/base4WD.chassis.xacro (robot description, xacro)
@@ -3,5 +3,5 @@
   <xacro:include filename="$(find romea_mobile_base_description)/urdf/common.xacro" />
   <xacro:include filename="$(find romea_mobile_base_description)/urdf/wheel.xacro" />
-  <xacro:macro name="chassis" params="*visual_chassis *visual_wheel">
+  <xacro:macro name="chassis" params="*visual_chassis *visual_front_wheel *visual_rear_wheel">
     <xacro:common>
       <xacro:insert_block name="visual_chassis"/>
@@ -15,5 +15,5 @@
                 left_right="-1">
       <origin xyz="${wheelbase/2} ${front_track/2} ${front_wheel_radius - chassis_height}" rpy="${-M_PI/2} 0 0" />
-      <xacro:insert_block name="visual_wheel"/>
+      <xacro:insert_block name="visual_front_wheel"/>
     </xacro:wheel>
     <xacro:wheel parent_link="${base_link}"
@@ -25,5 +25,5 @@
                  left_right="1">
       <origin xyz="${wheelbase/2} ${-front_track/2} ${front_wheel_radius - chassis_height}" rpy="${-M_PI/2} 0 0" />
-      <xacro:insert_block name="visual_wheel"/>
+      <xacro:insert_block name="visual_front_wheel"/>
     </xacro:wheel>
     <xacro:wheel parent_link="${base_link}"
@@ -35,5 +35,5 @@
                  left_right="-1">
       <origin xyz="${-wheelbase/2} ${rear_track/2} ${rear_wheel_radius - chassis_height}" rpy="${-M_PI/2} 0 0" />
-      <xacro:insert_block name="visual_wheel"/>
+      <xacro:insert_block name="visual_rear_wheel"/>
     </xacro:wheel>
     <xacro:wheel parent_link="${base_link}"
@@ -45,5 +45,5 @@
                  left_right="1">
       <origin xyz="${-wheelbase/2} ${-rear_track/2} ${rear_wheel_radius - chassis_height}" rpy="${-M_PI/2} 0 0" />
-      <xacro:insert_block name="visual_wheel"/>
+      <xacro:insert_block name="visual_rear_wheel"/>
     </xacro:wheel>
   </xacro:macro>
