Commit message: Add the 2FWC2RWD architecture for mobile bases with front caster wheels and rear driven wheels. Update chassis xacro templates to accept multiple chassis visuals.
Signed-off-by: Jean Laneurit <jean.laneurit@inrae.fr>

File: romea_mobile_base_description/urdf/base1FASxxx.chassis.xacro (robot description, xacro)
@@ -6,5 +6,5 @@
   <xacro:include filename="$(find romea_mobile_base_description)/urdf/axle_steering.xacro" />
   <xacro:macro name="chassis"
-    params="*visual_chassis
+    params="**chassis_visuals
             *visual_front_left_steering
             *visual_front_right_steering
@@ -14,5 +14,7 @@
             *visual_rear_right_wheel">
     <xacro:common>
-      <xacro:insert_block name="visual_chassis" />
+      <chassis_visuals>
+        <xacro:insert_block name="chassis_visuals" />
+      </chassis_visuals>
     </xacro:common>
     <xacro:axle_steering parent_link="${base_link}"

File: romea_mobile_base_description/urdf/base2ASxxx.chassis.xacro (robot description, xacro)
@@ -5,5 +5,5 @@
   <xacro:include filename="$(find romea_mobile_base_description)/urdf/axle_steering.xacro" />
   <xacro:macro name="chassis"
-    params="*visual_chassis
+    params="**chassis_visuals
           *visual_front_left_steering
           *visual_front_right_steering
@@ -15,5 +15,7 @@
           *visual_rear_right_wheel">
     <xacro:common>
-      <xacro:insert_block name="visual_chassis" />
+      <chassis_visuals>
+        <xacro:insert_block name="chassis_visuals" />
+      </chassis_visuals>
     </xacro:common>
     <xacro:axle_steering parent_link="${base_link}"

File: romea_mobile_base_description/urdf/base2FWC2RWD.chassis.xacro (robot description, xacro)
@@ -5,5 +5,5 @@
   <xacro:include filename="$(find romea_mobile_base_description)/urdf/wheel_caster.xacro" />
   <xacro:macro name="chassis"
-    params="*visual_chassis
+    params="**chassis_visuals
             *visual_front_left_caster
             *visual_front_right_caster
@@ -13,5 +13,7 @@
             *visual_rear_right_wheel">
     <xacro:common>
-      <xacro:insert_block name="visual_chassis" />
+      <chassis_visuals>
+        <xacro:insert_block name="chassis_visuals" />
+      </chassis_visuals>
     </xacro:common>
     <xacro:wheel_caster parent_link="${base_link}"

File: romea_mobile_base_description/urdf/base2FWSxxx.chassis.xacro (robot description, xacro)
@@ -5,5 +5,5 @@
   <xacro:include filename="$(find romea_mobile_base_description)/urdf/wheel_steered.xacro" />
   <xacro:macro name="chassis"
-    params="*visual_chassis
+    params="**chassis_visuals
             *visual_front_left_steering
             *visual_front_right_steering
@@ -13,5 +13,7 @@
             *visual_rear_right_wheel">
     <xacro:common>
-      <xacro:insert_block name="visual_chassis" />
+      <chassis_visuals>
+        <xacro:insert_block name="chassis_visuals" />
+      </chassis_visuals>
     </xacro:common>
     <xacro:wheel_steered parent_link="${base_link}"

File: romea_mobile_base_description/urdf/base2TD.chassis.xacro (robot description, xacro)
@@ -4,5 +4,5 @@
   <xacro:include filename="$(find romea_mobile_base_description)/urdf/wheel.xacro" />
   <xacro:macro name="chassis"
-    params="*visual_chassis
+    params="**chassis_visuals
             *visual_left_sprocket_wheel
             *visual_right_sprocket_wheel
@@ -10,5 +10,7 @@
             *visual_right_idler_wheel">
     <xacro:common>
-      <xacro:insert_block name="visual_chassis" />
+      <chassis_visuals>
+        <xacro:insert_block name="chassis_visuals" />
+      </chassis_visuals>
     </xacro:common>
     <xacro:wheel parent_link="${base_link}"

File: romea_mobile_base_description/urdf/base2THD.chassis.xacro (robot description, xacro)
@@ -4,5 +4,5 @@
   <xacro:include filename="$(find romea_mobile_base_description)/urdf/wheel.xacro" />
   <xacro:macro name="chassis"
-    params="*visual_chassis
+    params="**chassis_visuals
             *visual_left_sprocket_wheel
             *visual_right_sprocket_wheel
@@ -10,5 +10,7 @@
             *visual_right_idler_wheel">
     <xacro:common>
-      <xacro:insert_block name="visual_chassis" />
+      <chassis_visuals>
+        <xacro:insert_block name="chassis_visuals" />
+      </chassis_visuals>
     </xacro:common>
     <xacro:wheel parent_link="${base_link}"

File: romea_mobile_base_description/urdf/base2TTD.chassis.xacro (robot description, xacro)
@@ -4,5 +4,5 @@
   <xacro:include filename="$(find romea_mobile_base_description)/urdf/wheel.xacro" />
   <xacro:macro name="chassis"
-    params="*visual_chassis
+    params="**chassis_visuals
             *visual_left_sprocket_wheel
             *visual_right_sprocket_wheel
@@ -12,5 +12,7 @@
             *visual_right_roller_wheel">
     <xacro:common>
-      <xacro:insert_block name="visual_chassis" />
+      <chassis_visuals>
+        <xacro:insert_block name="chassis_visuals" />
+      </chassis_visuals>
     </xacro:common>
     <xacro:wheel parent_link="${base_link}"

File: romea_mobile_base_description/urdf/base4WD.chassis.xacro (robot description, xacro)
@@ -4,5 +4,5 @@
   <xacro:include filename="$(find romea_mobile_base_description)/urdf/wheel.xacro" />
   <xacro:macro name="chassis"
-    params="*visual_chassis
+    params="**chassis_visuals
             *visual_front_left_wheel
             *visual_front_right_wheel
@@ -10,5 +10,7 @@
             *visual_rear_right_wheel">
     <xacro:common>
-      <xacro:insert_block name="visual_chassis" />
+      <chassis_visuals>
+        <xacro:insert_block name="chassis_visuals" />
+      </chassis_visuals>
     </xacro:common>
     <xacro:wheel parent_link="${base_link}"

File: romea_mobile_base_description/urdf/base4WS4WD.chassis.xacro (robot description, xacro)
@@ -4,5 +4,5 @@
   <xacro:include filename="$(find romea_mobile_base_description)/urdf/wheel_steered.xacro" />
   <xacro:macro name="chassis"
-    params="*visual_chassis
+    params="**chassis_visuals
             *visual_front_left_steering
             *visual_front_right_steering
@@ -14,5 +14,7 @@
             *visual_rear_right_wheel">
     <xacro:common>
-      <xacro:insert_block name="visual_chassis" />
+      <chassis_visuals>
+        <xacro:insert_block name="chassis_visuals" />
+      </chassis_visuals>
     </xacro:common>
     <xacro:wheel_steered parent_link="${base_link}"

File: romea_mobile_base_description/urdf/common.xacro (robot description, xacro)
@@ -3,9 +3,9 @@
 <!--  <xacro:include filename="$(find four_wheel_steering_description)/urdf/wheel_steered.xacro" />-->
   <xacro:include filename="$(find romea_mobile_base_description)/urdf/wheel_steered.xacro" />
-  <xacro:macro name="common" params="*visual_chassis">
+  <xacro:macro name="common" params="**chassis_visuals">
     <link name="${prefix}${base_footprint_link}"/>
     <!-- Base link is the center of the robot -->
     <link name="${prefix}${base_link}">
-      <xacro:insert_block name="visual_chassis"/>
+      <xacro:insert_block name="chassis_visuals"/>
       <collision>
         <geometry>
