Commit message: description: add possibility to set different visual for rear and front wheels
Signed-off-by: Jean Laneurit <jean.laneurit@inrae.fr>

File: romea_mobile_base_description/urdf/axle_steering.xacro (robot description, xacro)
@@ -1,12 +1,12 @@
 <?xml version="1.0"?>
 <robot xmlns:xacro="http://www.ros.org/wiki/xacro" name="axle_steering">
-  <xacro:macro name="axle_steering" params="parent_link axle_steering_link axle_steering_joint *joint_origin">
+  <xacro:macro name="axle_steering" params="parent_link axle_steering_link axle_steering_joint steering_link_mass steering_link_x steering_link_y steering_link_z *joint_origin">
     <link name="${prefix}${axle_steering_link}">
       <inertial>
         <mass value="${steering_link_mass}" />
         <origin xyz="0 0 0" />
-        <inertia  ixx="${steering_link_mass/12.0 * (steering_link_y*steering_link_y + steering_link_xz*steering_link_xz)}" ixy="0" ixz="0"
-                  iyy="${steering_link_mass/12.0 * (steering_link_xz*steering_link_xz + steering_link_xz*steering_link_xz)}" iyz="0"
-                  izz="${steering_link_mass/12.0 * (steering_link_y*steering_link_y + steering_link_xz*steering_link_xz)}" />
+        <inertia  ixx="${steering_link_mass/12.0 * (steering_link_y*steering_link_y + steering_link_z*steering_link_z)}" ixy="0" ixz="0"
+                  iyy="${steering_link_mass/12.0 * (steering_link_x*steering_link_x + steering_link_z*steering_link_z)}" iyz="0"
+                  izz="${steering_link_mass/12.0 * (steering_link_y*steering_link_y + steering_link_y*steering_link_y)}" />
       </inertial>
    </link>

File: romea_mobile_base_description/urdf/base1FASxxx.chassis.xacro (robot description, xacro)
@@ -11,5 +11,9 @@
     <xacro:axle_steering parent_link="${base_link}"
                          axle_steering_link="${front_axle_steering_link}"
-                         axle_steering_joint="${front_axle_steering_joint}">
+                         axle_steering_joint="${front_axle_steering_joint}"
+                         steering_link_mass="${front_axle_steering_link_mass}"
+                         steering_link_x="${front_axle_steering_link_x}"
+                         steering_link_y="${front_axle_steering_link_y}"
+                         steering_link_z="${front_axle_steering_link_z}">
        <origin xyz="${wheelbase/2-body_reference_x} 0 ${front_wheel_radius - chassis_height}" rpy="0 0 0" />
     </xacro:axle_steering>
@@ -17,7 +21,10 @@
                          wheel_steering_link="${front_left_wheel_steering_link}"
                          wheel_steering_joint="${front_left_wheel_steering_joint}"
+                         steering_link_mass="${front_wheel_steering_link_mass}"
+                         steering_link_xz="${front_wheel_steering_link_xz}"
+                         steering_link_y="${front_wheel_steering_link_y}"
                          wheel_spinning_link="${front_left_wheel_spinning_link}"
                          wheel_spinning_joint="${front_left_wheel_spinning_joint}"
-                         wheel_origin_y="${front_wheel_y_offset}"
+                         wheel_origin_y="${front_hub_carrier_offset}"
                          wheel_mass="${front_wheel_mass}"
                          wheel_width="${front_wheel_width}"
@@ -31,7 +38,10 @@
                           wheel_steering_link="${front_right_wheel_steering_link}"
                           wheel_steering_joint="${front_right_wheel_steering_joint}"
+                          steering_link_mass="${front_wheel_steering_link_mass}"
+                          steering_link_xz="${front_wheel_steering_link_xz}"
+                          steering_link_y="${front_wheel_steering_link_y}"
                           wheel_spinning_link="${front_right_wheel_spinning_link}"
                           wheel_spinning_joint="${front_right_wheel_spinning_joint}"
-                          wheel_origin_y="${-front_wheel_y_offset}"
+                          wheel_origin_y="${-front_hub_carrier_offset}"
                           wheel_mass="${front_wheel_mass}"
                           wheel_width="${front_wheel_width}"

File: romea_mobile_base_description/urdf/base2ASxxx.chassis.xacro (robot description, xacro)
@@ -4,5 +4,5 @@
   <xacro:include filename="$(find romea_mobile_base_description)/urdf/wheel_steered.xacro" />
   <xacro:include filename="$(find romea_mobile_base_description)/urdf/axle_steering.xacro" />
-  <xacro:macro name="chassis" params="*visual_chassis *visual_steering *visual_wheel">
+  <xacro:macro name="chassis" params="*visual_chassis *visual_front_steering *visual_rear_steering *visual_front_wheel *visual_rear_wheel">
     <xacro:common>
       <xacro:insert_block name="visual_chassis"/>
@@ -10,10 +10,18 @@
     <xacro:axle_steering parent_link="${base_link}"
                          axle_steering_link="${front_axle_steering_link}"
-                         axle_steering_joint="${front_axle_steering_joint}">
+                         axle_steering_joint="${front_axle_steering_joint}"
+                         steering_link_mass="${front_axle_steering_link_mass}"
+                         steering_link_x="${front_axle_steering_link_x}"
+                         steering_link_y="${front_axle_steering_link_y}"
+                         steering_link_z="${front_axle_steering_link_z}">
        <origin xyz="${wheelbase/2-body_reference_x} 0 ${front_wheel_radius - chassis_height}" rpy="0 0 0" />
     </xacro:axle_steering>
     <xacro:axle_steering parent_link="${base_link}"
                          axle_steering_link="${rear_axle_steering_link}"
-                         axle_steering_joint="${rear_axle_steering_joint}">
+                         axle_steering_joint="${rear_axle_steering_joint}"
+                         steering_link_mass="${front_axle_steering_link_mass}"
+                         steering_link_x="${front_axle_steering_link_x}"
+                         steering_link_y="${front_axle_steering_link_y}"
+                         steering_link_z="${front_axle_steering_link_z}">
        <origin xyz="${-wheelbase/2-body_reference_x} 0 ${rear_wheel_radius - chassis_height}" rpy="0 0 0" />
     </xacro:axle_steering>
@@ -21,7 +29,10 @@
                          wheel_steering_link="${front_left_wheel_steering_link}"
                          wheel_steering_joint="${front_left_wheel_steering_joint}"
+                         steering_link_mass="${front_wheel_steering_link_mass}"
+                         steering_link_xz="${front_wheel_steering_link_xz}"
+                         steering_link_y="${front_wheel_steering_link_y}"
                          wheel_spinning_link="${front_left_wheel_spinning_link}"
                          wheel_spinning_joint="${front_left_wheel_spinning_joint}"
-                         wheel_origin_y="${front_wheel_y_offset}"
+                         wheel_origin_y="${rear_hub_carrier_offset}"
                          wheel_mass="${front_wheel_mass}"
                          wheel_width="${front_wheel_width}"
@@ -29,13 +40,16 @@
                          left_right="-1">
        <origin xyz="${wheelbase/2-body_reference_x} ${front_track/2} ${front_wheel_radius - chassis_height}" rpy="0 0 0" />
-       <xacro:insert_block name="visual_steering"/>
-       <xacro:insert_block name="visual_wheel"/>
+       <xacro:insert_block name="visual_front_steering"/>
+       <xacro:insert_block name="visual_front_wheel"/>
      </xacro:wheel_steered>
      <xacro:wheel_steered parent_link="${base_link}"
                           wheel_steering_link="${front_right_wheel_steering_link}"
                           wheel_steering_joint="${front_right_wheel_steering_joint}"
+                          steering_link_mass="${front_wheel_steering_link_mass}"
+                          steering_link_xz="${front_wheel_steering_link_xz}"
+                          steering_link_y="${front_wheel_steering_link_y}"
                           wheel_spinning_link="${front_right_wheel_spinning_link}"
                           wheel_spinning_joint="${front_right_wheel_spinning_joint}"
-                          wheel_origin_y="${-front_wheel_y_offset}"
+                          wheel_origin_y="${-rear_hub_carrier_offset}"
                           wheel_mass="${front_wheel_mass}"
                           wheel_width="${front_wheel_width}"
@@ -43,13 +57,16 @@
                           left_right="1">
        <origin xyz="${wheelbase/2-body_reference_x} ${-front_track/2} ${front_wheel_radius - chassis_height}" rpy="0 0 0" />
-       <xacro:insert_block name="visual_steering"/>
-       <xacro:insert_block name="visual_wheel"/>
+       <xacro:insert_block name="visual_front_steering"/>
+       <xacro:insert_block name="visual_front_wheel"/>
      </xacro:wheel_steered>
      <xacro:wheel_steered parent_link="${base_link}"
                           wheel_steering_link="${rear_left_wheel_steering_link}"
                           wheel_steering_joint="${rear_left_wheel_steering_joint}"
+                          steering_link_mass="${rear_wheel_steering_link_mass}"
+                          steering_link_xz="${rear_wheel_steering_link_xz}"
+                          steering_link_y="${rear_wheel_steering_link_y}"
                           wheel_spinning_link="${rear_left_wheel_spinning_link}"
                           wheel_spinning_joint="${rear_left_wheel_spinning_joint}"
-                          wheel_origin_y="${rear_wheel_y_offset}"
+                          wheel_origin_y="${rear_hub_carrier_offset}"
                           wheel_mass="${rear_wheel_mass}"
                           wheel_width="${rear_wheel_width}"
@@ -57,13 +74,16 @@
                           left_right="-1">
       <origin xyz="${-wheelbase/2-body_reference_x} ${rear_track/2} ${rear_wheel_radius  - chassis_height}" rpy="0 0 0" />
-      <xacro:insert_block name="visual_steering"/>
-      <xacro:insert_block name="visual_wheel"/>
+      <xacro:insert_block name="visual_rear_steering"/>
+      <xacro:insert_block name="visual_rear_wheel"/>
     </xacro:wheel_steered>
     <xacro:wheel_steered parent_link="${base_link}"
                          wheel_steering_link="${rear_right_wheel_steering_link}"
                          wheel_steering_joint="${rear_right_wheel_steering_joint}"
+                         steering_link_mass="${rear_wheel_steering_link_mass}"
+                         steering_link_xz="${rear_wheel_steering_link_xz}"
+                         steering_link_y="${rear_wheel_steering_link_y}"
                          wheel_spinning_link="${rear_right_wheel_spinning_link}"
                          wheel_spinning_joint="${rear_right_wheel_spinning_joint}"
-                         wheel_origin_y="${-rear_wheel_y_offset}"
+                         wheel_origin_y="${-rear_hub_carrier_offset}"
                          wheel_mass="${rear_wheel_mass}"
                          wheel_width="${rear_wheel_width}"
@@ -71,6 +91,6 @@
                          left_right="1">
       <origin xyz="${-wheelbase/2-body_reference_x} ${-rear_track/2} ${rear_wheel_radius - chassis_height}" rpy="0 0 0" />
-      <xacro:insert_block name="visual_steering"/>
-      <xacro:insert_block name="visual_wheel"/>
+      <xacro:insert_block name="visual_rear_steering"/>
+      <xacro:insert_block name="visual_rear_wheel"/>
     </xacro:wheel_steered>
   </xacro:macro>

File: romea_mobile_base_description/urdf/base2FWSxxx.chassis.xacro (robot description, xacro)
@@ -11,7 +11,10 @@
                          wheel_steering_link="${front_left_wheel_steering_link}"
                          wheel_steering_joint="${front_left_wheel_steering_joint}"
+                         steering_link_mass="${front_wheel_steering_link_mass}"
+                         steering_link_xz="${front_wheel_steering_link_xz}"
+                         steering_link_y="${front_wheel_steering_link_y}"
                          wheel_spinning_link="${front_left_wheel_spinning_link}"
                          wheel_spinning_joint="${front_left_wheel_spinning_joint}"
-                         wheel_origin_y="${front_wheel_y_offset}"
+                         wheel_origin_y="${front_hub_carrier_offset}"
                          wheel_mass="${front_wheel_mass}"
                          wheel_width="${front_wheel_width}"
@@ -25,7 +28,10 @@
                           wheel_steering_link="${front_right_wheel_steering_link}"
                           wheel_steering_joint="${front_right_wheel_steering_joint}"
+                          steering_link_mass="${front_wheel_steering_link_mass}"
+                          steering_link_xz="${front_wheel_steering_link_xz}"
+                          steering_link_y="${front_wheel_steering_link_y}"
                           wheel_spinning_link="${front_right_wheel_spinning_link}"
                           wheel_spinning_joint="${front_right_wheel_spinning_joint}"
-                          wheel_origin_y="${-front_wheel_y_offset}"
+                          wheel_origin_y="${-front_hub_carrier_offset}"
                           wheel_mass="${front_wheel_mass}"
                           wheel_width="${front_wheel_width}"

File: romea_mobile_base_description/urdf/base4WS4WD.chassis.xacro (robot description, xacro)
@@ -3,5 +3,5 @@
   <xacro:include filename="$(find romea_mobile_base_description)/urdf/common.xacro" />
   <xacro:include filename="$(find romea_mobile_base_description)/urdf/wheel_steered.xacro" />
-  <xacro:macro name="chassis" params="*visual_chassis *visual_steering *visual_wheel">
+  <xacro:macro name="chassis" params="*visual_chassis *visual_front_steering *visual_rear_steering *visual_front_wheel *visual_rear_wheel">
     <xacro:common>
       <xacro:insert_block name="visual_chassis"/>
@@ -10,7 +10,10 @@
                          wheel_steering_link="${front_left_wheel_steering_link}"
                          wheel_steering_joint="${front_left_wheel_steering_joint}"
+                         steering_link_mass="${front_wheel_steering_link_mass}"
+                         steering_link_xz="${front_wheel_steering_link_xz}"
+                         steering_link_y="${front_wheel_steering_link_y}"
                          wheel_spinning_link="${front_left_wheel_spinning_link}"
                          wheel_spinning_joint="${front_left_wheel_spinning_joint}"
-                         wheel_origin_y="${front_wheel_y_offset}"
+                         wheel_origin_y="${front_hub_carrier_offset}"
                          wheel_mass="${front_wheel_mass}"
                          wheel_width="${front_wheel_width}"
@@ -18,13 +21,16 @@
                          left_right="-1">
        <origin xyz="${wheelbase/2-body_reference_x} ${front_track/2} ${front_wheel_radius - chassis_height}" rpy="0 0 0" />
-       <xacro:insert_block name="visual_steering"/>
-       <xacro:insert_block name="visual_wheel"/>
+       <xacro:insert_block name="visual_front_steering"/>
+       <xacro:insert_block name="visual_front_wheel"/>
      </xacro:wheel_steered>
      <xacro:wheel_steered parent_link="${base_link}"
                           wheel_steering_link="${front_right_wheel_steering_link}"
                           wheel_steering_joint="${front_right_wheel_steering_joint}"
+                          steering_link_mass="${front_wheel_steering_link_mass}"
+                          steering_link_xz="${front_wheel_steering_link_xz}"
+                          steering_link_y="${front_wheel_steering_link_y}"
                           wheel_spinning_link="${front_right_wheel_spinning_link}"
                           wheel_spinning_joint="${front_right_wheel_spinning_joint}"
-                          wheel_origin_y="${-front_wheel_y_offset}"
+                          wheel_origin_y="${-front_hub_carrier_offset}"
                           wheel_mass="${front_wheel_mass}"
                           wheel_width="${front_wheel_width}"
@@ -32,13 +38,16 @@
                           left_right="1">
        <origin xyz="${wheelbase/2-body_reference_x} ${-front_track/2} ${front_wheel_radius - chassis_height}" rpy="0 0 0" />
-       <xacro:insert_block name="visual_steering"/>
-       <xacro:insert_block name="visual_wheel"/>
+       <xacro:insert_block name="visual_front_steering"/>
+       <xacro:insert_block name="visual_front_wheel"/>
      </xacro:wheel_steered>
      <xacro:wheel_steered parent_link="${base_link}"
                           wheel_steering_link="${rear_left_wheel_steering_link}"
                           wheel_steering_joint="${rear_left_wheel_steering_joint}"
+                          steering_link_mass="${rear_wheel_steering_link_mass}"
+                          steering_link_xz="${rear_wheel_steering_link_xz}"
+                          steering_link_y="${rear_wheel_steering_link_y}"
                           wheel_spinning_link="${rear_left_wheel_spinning_link}"
                           wheel_spinning_joint="${rear_left_wheel_spinning_joint}"
-                          wheel_origin_y="${rear_wheel_y_offset}"
+                          wheel_origin_y="${rear_hub_carrier_offset}"
                           wheel_mass="${rear_wheel_mass}"
                           wheel_width="${rear_wheel_width}"
@@ -46,13 +55,16 @@
                           left_right="-1">
       <origin xyz="${-wheelbase/2-body_reference_x} ${rear_track/2} ${rear_wheel_radius  - chassis_height}" rpy="0 0 0" />
-      <xacro:insert_block name="visual_steering"/>
-      <xacro:insert_block name="visual_wheel"/>
+      <xacro:insert_block name="visual_rear_steering"/>
+      <xacro:insert_block name="visual_rear_wheel"/>
     </xacro:wheel_steered>
     <xacro:wheel_steered parent_link="${base_link}"
                          wheel_steering_link="${rear_right_wheel_steering_link}"
                          wheel_steering_joint="${rear_right_wheel_steering_joint}"
+                         steering_link_mass="${rear_wheel_steering_link_mass}"
+                         steering_link_xz="${rear_wheel_steering_link_xz}"
+                         steering_link_y="${rear_wheel_steering_link_y}"
                          wheel_spinning_link="${rear_right_wheel_spinning_link}"
                          wheel_spinning_joint="${rear_right_wheel_spinning_joint}"
-                         wheel_origin_y="${-rear_wheel_y_offset}"
+                         wheel_origin_y="${-rear_hub_carrier_offset}"
                          wheel_mass="${rear_wheel_mass}"
                          wheel_width="${rear_wheel_width}"
@@ -60,6 +72,6 @@
                          left_right="1">
       <origin xyz="${-wheelbase/2-body_reference_x} ${-rear_track/2} ${rear_wheel_radius - chassis_height}" rpy="0 0 0" />
-      <xacro:insert_block name="visual_steering"/>
-      <xacro:insert_block name="visual_wheel"/>
+      <xacro:insert_block name="visual_rear_steering"/>
+      <xacro:insert_block name="visual_rear_wheel"/>
     </xacro:wheel_steered>
   </xacro:macro>

File: romea_mobile_base_description/urdf/wheel_steered.xacro (robot description, xacro)
@@ -3,5 +3,5 @@
   <xacro:property name="M_PI" value="3.14159"/>
   <xacro:include filename="$(find romea_mobile_base_description)/urdf/wheel.xacro" />
-  <xacro:macro name="wheel_steered" params="parent_link wheel_steering_link wheel_steering_joint wheel_spinning_link wheel_spinning_joint wheel_origin_y wheel_mass wheel_width wheel_radius left_right *joint_origin *visual_steering *visual_wheel">
+  <xacro:macro name="wheel_steered" params="parent_link wheel_steering_link wheel_steering_joint  steering_link_mass steering_link_xz steering_link_y wheel_spinning_link wheel_spinning_joint wheel_origin_y wheel_mass wheel_width wheel_radius left_right *joint_origin *visual_steering *visual_wheel">
     <link name="${prefix}${wheel_steering_link}">
       <visual>
