Commit message: use gazebo collision bitmask in URDF

File: romea_mobile_base_description/urdf/common.xacro (robot description, xacro)
@@ -5,7 +5,4 @@
   <xacro:macro name="common" params="*visual_chassis">
     <link name="${prefix}${base_footprint_link}"/>
-    <!-- <gazebo reference="${prefix}${base_link}">
-      <material>Gazebo/Grey</material>
-    </gazebo> -->
     <!-- Base link is the center of the robot -->
     <link name="${prefix}${base_link}">
@@ -39,4 +36,14 @@
       <child link="${prefix}${inertial_link}" />
     </joint>
+    <gazebo reference="${prefix}${base_link}">
+      <collision>
+        <surface>
+          <contact>
+            <!-- bitmask: stems(4), weeds(3), crops(2), elements(1), ground(0) -->
+            <collide_bitmask>0x17</collide_bitmask>
+          </contact>
+        </surface>
+      </collision>
+    </gazebo>
   </xacro:macro>
 </robot>

File: romea_mobile_base_description/urdf/wheel.xacro (robot description, xacro)
@@ -39,10 +39,19 @@
       </collision>
     </link>
+    <!-- <gazebo reference="${prefix}${wheel_spinning_link}"> -->
+    <!--   <mu1 value="0.9" /> -->
+    <!--   <mu2 value="0.9" /> -->
+    <!--   <kp value="1e8" /> -->
+    <!--   <minDepth>0.01</minDepth> -->
+    <!-- </gazebo> -->
     <gazebo reference="${prefix}${wheel_spinning_link}">
-      <mu1 value="0.9" />
-      <mu2 value="0.9" />
-      <fdir1>0 0 1</fdir1>
-      <kp value="1e8" />
-      <minDepth>0.005</minDepth>
+      <collision>
+        <surface>
+          <contact>
+            <!-- bitmask: stems(4), weeds(3), crops(2), elements(1), ground(0) -->
+            <collide_bitmask>0x17</collide_bitmask>
+          </contact>
+        </surface>
+      </collision>
     </gazebo>
     <joint name="${prefix}${wheel_spinning_joint}" type="continuous">
