Commit message: fix: correct position of elements for base2FWC2RWD

File: romea_mobile_base_description/urdf/base2FWC2RWD.chassis.xacro (robot description, xacro)
@@ -33,5 +33,5 @@
       left_right="-1">
       <origin
-        xyz="${wheelbase/2-body_reference_x} ${front_track/2} ${front_wheel_radius - chassis_height}"
+        xyz="${wheelbase - body_reference_x} ${front_track/2} ${front_wheel_radius - chassis_height}"
         rpy="0 0 0" />
       <xacro:insert_block name="visual_front_left_caster" />
@@ -53,5 +53,5 @@
       left_right="1">
       <origin
-        xyz="${wheelbase/2-body_reference_x} ${-front_track/2} ${front_wheel_radius - chassis_height}"
+        xyz="${wheelbase - body_reference_x} ${-front_track/2} ${front_wheel_radius - chassis_height}"
         rpy="0 0 0" />
       <xacro:insert_block name="visual_front_right_caster" />
@@ -66,5 +66,5 @@
       left_right="-1">
       <origin
-        xyz="${-wheelbase/2-body_reference_x} ${rear_track/2} ${rear_wheel_radius - chassis_height}"
+        xyz="${-body_reference_x} ${rear_track/2} ${rear_wheel_radius - chassis_height}"
         rpy="${-M_PI/2} 0 0" />
       <xacro:insert_block name="visual_rear_left_wheel" />
@@ -78,5 +78,5 @@
       left_right="1">
       <origin
-        xyz="${-wheelbase/2-body_reference_x} ${-rear_track/2} ${rear_wheel_radius - chassis_height}"
+        xyz="${-body_reference_x} ${-rear_track/2} ${rear_wheel_radius - chassis_height}"
         rpy="${-M_PI/2} 0 0" />
       <xacro:insert_block name="visual_rear_right_wheel" />

File: romea_mobile_base_description/urdf/common.xacro (robot description, xacro)
@@ -13,5 +13,7 @@
           <box size="${aabb_length} ${aabb_width} ${aabb_height}"/>
         </geometry>
-        <origin xyz="${aabb_center_x-body_reference_x} ${aabb_center_y} ${aabb_center_z-chassis_height}" rpy="0 0 0" />
+        <origin
+          xyz="${aabb_center_x-body_reference_x} ${aabb_center_y} ${aabb_center_z-chassis_height}"
+          rpy="0 0 0" />
 <!--        <origin xyz="${-body_reference_x} 0 ${ground_clearance+aabb_height/2-chassis_height}" rpy="0 0 0" />-->
       </collision>
