Commit message: mobile_base_gazebo : add test for interface 2FWSxxx

File: romea_mobile_base_gazebo/test/test_gazebo_interface4WD.xacro (robot description, xacro)
@@ -1,10 +1,63 @@
-<?xml version='1.0' encoding='utf-8'?>
-<robot name="robot" xmlns:xacro="http://www.ros.org/wiki/xacro">
-  <xacro:property name="prefix" value="robot_"/>
-  <xacro:property name="front_left_wheel_spinning_joint" value="joint1"/>
-  <xacro:property name="front_right_wheel_spinning_joint" value="joint2"/>
-  <xacro:property name="rear_left_wheel_spinning_joint" value="joint3"/>
-  <xacro:property name="rear_right_wheel_spinning_joint" value="joint4"/>
-  <xacro:include filename="$(find romea_mobile_base_description)/ros2_control/4WD.ros2_control.xacro" />
-  <xacro:base_control/>
+<?xml version="1.0"?>
+<robot name="robot" xmlns:xacro="http://ros.org/wiki/xacro">
+    <xacro:property name="M_PI" value="3.14159"/>
+    <xacro:include filename="$(find romea_mobile_base_description)/urdf/base4WD.chassis.xacro" />
+    <xacro:include filename="$(find romea_mobile_base_description)/ros2_control/base4WD.ros2_control.xacro"/>
+    <xacro:property name="prefix" value=""/>
+    <!-- Link names -->
+    <xacro:property name="base_link" value="base_link" />
+    <xacro:property name="base_footprint_link" value="base_footprint_link" />
+    <xacro:property name="inertial_link" value="inertial_link_name" />
+    <xacro:property name="front_left_wheel_spinning_link" value="front_left_wheel_spinning_link" />
+    <xacro:property name="front_right_wheel_spinning_link" value="front_right_wheel_spinning_link" />
+    <xacro:property name="rear_left_wheel_spinning_link" value="rear_left_wheel_spinning_link" />
+    <xacro:property name="rear_right_wheel_spinning_link" value="rear_right_wheel_spinning_link" />
+    <!-- Joint names -->
+    <xacro:property name="base_footprint_joint" value="base_footprint_joint" />
+    <xacro:property name="inertial_joint" value="inertial_joint" />
+    <xacro:property name="front_left_wheel_spinning_joint" value="front_left_wheel_spinning_joint" />
+    <xacro:property name="front_right_wheel_spinning_joint" value="front_right_wheel_spinning_joint_name" />
+    <xacro:property name="rear_left_wheel_spinning_joint" value="rear_left_wheel_spinning_joint_name" />
+    <xacro:property name="rear_right_wheel_spinning_joint" value="rear_right_wheel_spinning_joint_name" />
+    <!-- Base Properties -->
+    <xacro:property name="aabb_length" value="0.54" />
+    <xacro:property name="aabb_width" value="0.40" />
+    <xacro:property name="aabb_height" value="0.18" />
+<!--    center: [0., 0., 0.188]-->
+    <xacro:property name="wheelbase" value="0.392"/>
+    <xacro:property name="front_track" value="0.515"/>
+    <xacro:property name="rear_track" value="0.515"/>
+    <xacro:property name="mass_base" value="17" />
+    <xacro:property name="mass_center_x" value="0.0" />
+    <xacro:property name="mass_center_y" value="0.0" />
+    <xacro:property name="mass_center_z" value="0.188" />
+    <xacro:property name="maximal_wheel_speed" value="3.0"/>
+    <xacro:property name="body_reference_x" value="0.0" />
+    <!-- Wheel Properties -->
+    <xacro:property name="front_wheel_radius" value="0.1315" />
+    <xacro:property name="rear_wheel_radius" value="0.1315" />
+    <xacro:property name="front_wheel_width" value="0.1" />
+    <xacro:property name="rear_wheel_width" value="0.1" />
+    <xacro:property name="front_wheel_mass" value="20." />
+    <xacro:property name="rear_wheel_mass" value="20." />
+    <xacro:property name="wheel_radius" value="${front_wheel_radius}" />
+    <xacro:property name="wheel_width" value="${front_wheel_width}" />
+    <!-- Wheel Mounting Positions -->
+    <xacro:property name="ground_clearance" value="0.098"/>
+    <xacro:property name="front_wheel_y_offset" value="0.0" />
+    <xacro:property name="rear_wheel_y_offset" value="0.0" />
+    <xacro:property name="chassis_height" value="${min(front_wheel_radius,rear_wheel_radius)}" />
+    <xacro:chassis>
+        <visual>
+          <geometry>
+            <box size="${aabb_length} ${aabb_width} ${aabb_height}"/>
+          </geometry>
+          <material name="grey">
+            <color rgba="0.6 0.6 0.6 1"/>
+          </material>
+        </visual>
+        <!-- visual wheel -->
+        <cylinder length="${wheel_width}" radius="${wheel_radius}"/>
+    </xacro:chassis>
+    <xacro:base_control mode="test"/>
 </robot>

Commit message: mobile_base_gazebo : add test for 2ASxxx, 2TD, 2THD, 2TTD, 4WS4WD gazebo interfaces

File: romea_mobile_base_gazebo/test/test_gazebo_interface4WD.xacro (robot description, xacro)
@@ -21,7 +21,11 @@
     <xacro:property name="rear_right_wheel_spinning_joint" value="rear_right_wheel_spinning_joint_name" />
     <!-- Base Properties -->
+    <xacro:property name="ground_clearance" value="0.098"/>
     <xacro:property name="aabb_length" value="0.54" />
     <xacro:property name="aabb_width" value="0.40" />
     <xacro:property name="aabb_height" value="0.18" />
+    <xacro:property name="aabb_center_x" value="0.0" />
+    <xacro:property name="aabb_center_y" value="0.0" />
+    <xacro:property name="aabb_center_z" value="${aabb_height/2.0+ground_clearance}" />
 <!--    center: [0., 0., 0.188]-->
     <xacro:property name="wheelbase" value="0.392"/>
@@ -44,5 +48,4 @@
     <xacro:property name="wheel_width" value="${front_wheel_width}" />
     <!-- Wheel Mounting Positions -->
-    <xacro:property name="ground_clearance" value="0.098"/>
     <xacro:property name="front_wheel_y_offset" value="0.0" />
     <xacro:property name="rear_wheel_y_offset" value="0.0" />
@@ -53,4 +56,5 @@
             <box size="${aabb_length} ${aabb_width} ${aabb_height}"/>
           </geometry>
+          <origin xyz="${aabb_center_x-body_reference_x} ${aabb_center_y}  ${aabb_center_z-chassis_height}" rpy="0 0 0" />
           <material name="grey">
             <color rgba="0.6 0.6 0.6 1"/>

File: romea_mobile_base_gazebo/test/test_gazebo_interface4WS4WD.xacro (robot description, xacro)
@@ -28,7 +28,4 @@
     <xacro:property name="aabb_width" value="1.18" />
     <xacro:property name="aabb_height" value="1.5" />
-    <xacro:property name="aabb_center_x" value="0.0" />
-    <xacro:property name="aabb_center_y" value="0.0" />
-    <xacro:property name="aabb_center_z" value="${aabb_height/2.0+ground_clearance}" />
      <xacro:property name="wheelbase" value="2.0"/>
     <xacro:property name="front_track" value="1.0"/>
@@ -36,8 +33,14 @@
     <xacro:property name="track" value="${front_track}"/>
     <xacro:property name="ground_clearance" value="0.45"/>
+<!--    <xacro:property name="mass_body" value="800." />-->
     <xacro:property name="mass_base" value="800." />
     <xacro:property name="mass_center_x" value="-0.1" />
     <xacro:property name="mass_center_y" value=" 0.0" />
     <xacro:property name="mass_center_z" value=" 0.2" />
+<!--    <xacro:property name="body_length" value="2.6" />
+    <xacro:property name="body_width" value="1.18" />
+    <xacro:property name="body_height" value="1.5" />-->
+<!--    <xacro:property name="body_offset_x" value="-1.0" />-->
+<!--    <xacro:property name="body_origin_z" value="0.0" />-->
     <xacro:property name="body_reference_x" value="-1.0" />
     <!-- Steering Properties -->
@@ -69,5 +72,5 @@
       <!-- visual chassis -->
       <visual>
-        <origin xyz="${aabb_center_x-body_reference_x} ${aabb_center_y}  ${aabb_center_z-chassis_height}" rpy="0 0 0" />
+        <origin xyz="${-body_reference_x} 0 ${ground_clearance+aabb_height/2-chassis_height}" rpy="0 0 0" />
         <geometry>
           <box size="${aabb_length} ${aabb_width} ${aabb_height}"/>
