Commit message: gazebo: remove some cout

File: romea_mobile_base_gazebo/test/test_gazebo_interface1FASxxx.xacro (robot description, xacro)
@@ -1,83 +1,87 @@
 <?xml version="1.0"?>
 <robot name="robot" xmlns:xacro="http://www.ros.org/wiki/xacro">
-    <xacro:arg name="type" default="" />
-    <xacro:include filename="$(find romea_mobile_base_description)/urdf/base1FAS4WD.chassis.xacro"/>
-    <xacro:include filename="$(find romea_mobile_base_description)/ros2_control/base$(arg type).ros2_control.xacro"/>
-    <xacro:property name="prefix" value=""/>
-    <!-- Link names -->
-    <xacro:property name="base_link" value="base_link" />
-    <xacro:property name="base_footprint_link" value="base_footprint_link"/>
-    <xacro:property name="inertial_link" value="inertial_link"/>
-    <xacro:property name="front_axle_steering_link" value="front_axle_steering_link"/>
-    <xacro:property name="front_left_wheel_steering_link" value="front_left_wheel_steering_link"/>
-    <xacro:property name="front_right_wheel_steering_link" value="front_right_wheel_steering_link"/>
-    <xacro:property name="rear_left_wheel_steering_link" value="rear_left_wheel_steering_link"/>
-    <xacro:property name="rear_right_wheel_steering_link" value="rear_right_wheel_steering_link"/>
-    <xacro:property name="front_left_wheel_spinning_link" value="front_left_wheel_spinning_link"/>
-    <xacro:property name="front_right_wheel_spinning_link" value="front_right_wheel_spinning_link"/>
-    <xacro:property name="rear_left_wheel_spinning_link" value="rear_left_wheel_spinning_link"/>
-    <xacro:property name="rear_right_wheel_spinning_link" value="rear_right_wheel_spinning_link}"/>
-    <!-- Joint names -->
-    <xacro:property name="base_footprint_joint" value="base_footprint_joint"/>
-    <xacro:property name="inertial_joint" value="inertial_joint"/>
-    <xacro:property name="front_axle_steering_joint" value="front_axle_steering_joint"/>
-    <xacro:property name="front_left_wheel_steering_joint" value="front_left_wheel_steering_joint"/>
-    <xacro:property name="front_right_wheel_steering_joint" value="front_right_wheel_steering_joint"/>
-    <xacro:property name="rear_left_wheel_steering_joint" value="rear_left_wheel_steering_joint"/>
-    <xacro:property name="rear_right_wheel_steering_joint" value="rear_right_wheel_steering_joint"/>
-    <xacro:property name="front_left_wheel_spinning_joint" value="front_left_wheel_spinning_joint"/>
-    <xacro:property name="front_right_wheel_spinning_joint" value="front_right_wheel_spinning_joint" />
-    <xacro:property name="rear_left_wheel_spinning_joint" value="rear_left_wheel_spinning_joint" />
-    <xacro:property name="rear_right_wheel_spinning_joint" value="rear_right_wheel_spinning_joint" />
-    <!-- Base Properties -->
-    <xacro:property name="ground_clearance" value="0.35"/>
-    <xacro:property name="aabb_length" value="1.66" />
-    <xacro:property name="aabb_width" value="0.6" />
-    <xacro:property name="aabb_height" value="0.6" />
-    <xacro:property name="aabb_center_x" value="0.0" />
-    <xacro:property name="aabb_center_y" value="0.0" />
-    <xacro:property name="aabb_center_z" value="${aabb_height/2.0+ground_clearance}" />
-    <xacro:property name="wheelbase" value="2.5"/>
-    <xacro:property name="front_track" value="1.2"/>
-    <xacro:property name="rear_track" value="1.2"/>
-    <xacro:property name="mass_base" value="400.0" />
-    <xacro:property name="mass_center_x" value="0.0" />
-    <xacro:property name="mass_center_y" value="0.0" />
-    <xacro:property name="mass_center_z" value="0.5" />
-    <xacro:property name="maximal_axle_steering_angle" value="1.0"/>
-    <xacro:property name="maximal_wheel_steering_angle" value="${atan(tan(maximal_axle_steering_angle)/(1-tan(maximal_axle_steering_angle)*front_track/(2*wheelbase)))}"/>
-    <xacro:property name="minimal_axle_steering_angle" value="${-maximal_axle_steering_angle}"/>
-    <xacro:property name="minimal_wheel_steering_angle" value="${-maximal_wheel_steering_angle} "/>
-    <xacro:property name="maximal_wheel_speed" value="2.0"/>
-    <xacro:property name="body_reference_x" value="-1.25" />
-     <!-- Wheel Properties -->
-     <xacro:property name="steering_link_mass" value="30" />
-     <xacro:property name="steering_link_y" value="0.05" />
-     <xacro:property name="steering_link_xz" value="0.1" />
-     <xacro:property name="front_wheel_radius" value="0.2" />
-     <xacro:property name="rear_wheel_radius" value="0.2" />
-     <xacro:property name="front_wheel_width" value="0.12" />
-     <xacro:property name="rear_wheel_width" value="0.012" />
-     <xacro:property name="front_wheel_mass" value="10" />
-     <xacro:property name="rear_wheel_mass" value="10" />
-     <xacro:property name="wheel_radius" value="${front_wheel_radius}" />
-     <xacro:property name="wheel_width" value="${front_wheel_width}" />
-     <!-- Wheel Mounting Positions -->
-     <xacro:property name="front_wheel_y_offset" value="0.1" />
-     <xacro:property name="rear_wheel_y_offset" value="0.1" />
-     <xacro:property name="chassis_height" value="${min(front_wheel_radius,rear_wheel_radius)}" />
-     <xacro:chassis>
-       <!-- visual chassis -->
-       <visual>
-        <origin xyz="${aabb_center_x-body_reference_x} ${aabb_center_y}  ${aabb_center_z-chassis_height}" rpy="0 0 0" />
-         <geometry>
-           <box size="${aabb_length} ${aabb_width} ${aabb_height}"/>
-         </geometry>
-       </visual>
-       <!-- visual front steering -->
-       <box size="${steering_link_xz} ${steering_link_y} ${steering_link_xz}"/>
-       <!-- visual wheel -->
-       <cylinder length="${wheel_width}" radius="${wheel_radius}"/>
-     </xacro:chassis>
-     <xacro:base_control mode="test"/>
+  <xacro:arg name="type" default="" />
+  <xacro:include filename="$(find romea_mobile_base_description)/urdf/base1FASxxx.chassis.xacro" />
+  <xacro:include
+    filename="$(find romea_mobile_base_description)/ros2_control/base$(arg type).ros2_control.xacro" />
+  <xacro:property name="prefix" value="" />
+  <!-- Link names -->
+  <xacro:property name="base_link" value="base_link" />
+  <xacro:property name="base_footprint_link" value="base_footprint_link" />
+  <xacro:property name="inertial_link" value="inertial_link" />
+  <xacro:property name="front_axle_steering_link" value="front_axle_steering_link" />
+  <xacro:property name="front_left_wheel_steering_link" value="front_left_wheel_steering_link" />
+  <xacro:property name="front_right_wheel_steering_link" value="front_right_wheel_steering_link" />
+  <xacro:property name="rear_left_wheel_steering_link" value="rear_left_wheel_steering_link" />
+  <xacro:property name="rear_right_wheel_steering_link" value="rear_right_wheel_steering_link" />
+  <xacro:property name="front_left_wheel_spinning_link" value="front_left_wheel_spinning_link" />
+  <xacro:property name="front_right_wheel_spinning_link" value="front_right_wheel_spinning_link" />
+  <xacro:property name="rear_left_wheel_spinning_link" value="rear_left_wheel_spinning_link" />
+  <xacro:property name="rear_right_wheel_spinning_link" value="rear_right_wheel_spinning_link}" />
+  <!-- Joint names -->
+  <xacro:property name="base_footprint_joint" value="base_footprint_joint" />
+  <xacro:property name="inertial_joint" value="inertial_joint" />
+  <xacro:property name="front_axle_steering_joint" value="front_axle_steering_joint" />
+  <xacro:property name="front_left_wheel_steering_joint" value="front_left_wheel_steering_joint" />
+  <xacro:property name="front_right_wheel_steering_joint" value="front_right_wheel_steering_joint" />
+  <xacro:property name="rear_left_wheel_steering_joint" value="rear_left_wheel_steering_joint" />
+  <xacro:property name="rear_right_wheel_steering_joint" value="rear_right_wheel_steering_joint" />
+  <xacro:property name="front_left_wheel_spinning_joint" value="front_left_wheel_spinning_joint" />
+  <xacro:property name="front_right_wheel_spinning_joint" value="front_right_wheel_spinning_joint" />
+  <xacro:property name="rear_left_wheel_spinning_joint" value="rear_left_wheel_spinning_joint" />
+  <xacro:property name="rear_right_wheel_spinning_joint" value="rear_right_wheel_spinning_joint" />
+  <!-- Base Properties -->
+  <xacro:property name="ground_clearance" value="0.35" />
+  <xacro:property name="aabb_length" value="1.66" />
+  <xacro:property name="aabb_width" value="0.6" />
+  <xacro:property name="aabb_height" value="0.6" />
+  <xacro:property name="aabb_center_x" value="0.0" />
+  <xacro:property name="aabb_center_y" value="0.0" />
+  <xacro:property name="aabb_center_z" value="${aabb_height/2.0+ground_clearance}" />
+  <xacro:property name="wheelbase" value="2.5" />
+  <xacro:property name="front_track" value="1.2" />
+  <xacro:property name="rear_track" value="1.2" />
+  <xacro:property name="mass_base" value="400.0" />
+  <xacro:property name="mass_center_x" value="0.0" />
+  <xacro:property name="mass_center_y" value="0.0" />
+  <xacro:property name="mass_center_z" value="0.5" />
+  <xacro:property name="maximal_axle_steering_angle" value="1.0" />
+  <xacro:property name="maximal_wheel_steering_angle"
+    value="${atan(tan(maximal_axle_steering_angle)/(1-tan(maximal_axle_steering_angle)*front_track/(2*wheelbase)))}" />
+  <xacro:property name="minimal_axle_steering_angle" value="${-maximal_axle_steering_angle}" />
+  <xacro:property name="minimal_wheel_steering_angle" value="${-maximal_wheel_steering_angle} " />
+  <xacro:property name="maximal_wheel_speed" value="2.0" />
+  <xacro:property name="body_reference_x" value="-1.25" />
+  <!-- Wheel Properties -->
+  <xacro:property name="steering_link_mass" value="30" />
+  <xacro:property name="steering_link_y" value="0.05" />
+  <xacro:property name="steering_link_xz" value="0.1" />
+  <xacro:property name="front_wheel_radius" value="0.2" />
+  <xacro:property name="rear_wheel_radius" value="0.2" />
+  <xacro:property name="front_wheel_width" value="0.12" />
+  <xacro:property name="rear_wheel_width" value="0.012" />
+  <xacro:property name="front_wheel_mass" value="10" />
+  <xacro:property name="rear_wheel_mass" value="10" />
+  <xacro:property name="wheel_radius" value="${front_wheel_radius}" />
+  <xacro:property name="wheel_width" value="${front_wheel_width}" />
+  <!-- Wheel Mounting Positions -->
+  <xacro:property name="front_wheel_y_offset" value="0.1" />
+  <xacro:property name="rear_wheel_y_offset" value="0.1" />
+  <xacro:property name="chassis_height" value="${min(front_wheel_radius,rear_wheel_radius)}" />
+  <xacro:chassis>
+    <!-- visual chassis -->
+    <visual>
+      <origin
+        xyz="${aabb_center_x-body_reference_x} ${aabb_center_y}  ${aabb_center_z-chassis_height}"
+        rpy="0 0 0" />
+      <geometry>
+        <box size="${aabb_length} ${aabb_width} ${aabb_height}" />
+      </geometry>
+    </visual>
+    <!-- visual front steering -->
+    <box size="${steering_link_xz} ${steering_link_y} ${steering_link_xz}" />
+    <!-- visual wheel -->
+    <cylinder length="${wheel_width}" radius="${wheel_radius}" />
+  </xacro:chassis>
+  <xacro:base_control mode="test" />
 </robot>

File: romea_mobile_base_gazebo/test/test_gazebo_interface2ASxxx.xacro (robot description, xacro)
@@ -1,85 +1,89 @@
 <?xml version="1.0"?>
 <robot name="robot" xmlns:xacro="http://www.ros.org/wiki/xacro">
-    <xacro:arg name="type" default="" />
-    <xacro:include filename="$(find romea_mobile_base_description)/urdf/base2AS4WD.chassis.xacro"/>
-    <xacro:include filename="$(find romea_mobile_base_description)/ros2_control/base$(arg type).ros2_control.xacro"/>
-    <xacro:property name="prefix" value=""/>
-    <!-- Link names -->
-    <xacro:property name="base_link" value="base_link" />
-    <xacro:property name="base_footprint_link" value="base_footprint_link"/>
-    <xacro:property name="inertial_link" value="inertial_link"/>
-    <xacro:property name="front_axle_steering_link" value="front_axle_steering_link"/>
-    <xacro:property name="rear_axle_steering_link" value="rear_axle_steering_link"/>
-    <xacro:property name="front_left_wheel_steering_link" value="front_left_wheel_steering_link"/>
-    <xacro:property name="front_right_wheel_steering_link" value="front_right_wheel_steering_link"/>
-    <xacro:property name="rear_left_wheel_steering_link" value="rear_left_wheel_steering_link"/>
-    <xacro:property name="rear_right_wheel_steering_link" value="rear_right_wheel_steering_link"/>
-    <xacro:property name="front_left_wheel_spinning_link" value="front_left_wheel_spinning_link"/>
-    <xacro:property name="front_right_wheel_spinning_link" value="front_right_wheel_spinning_link"/>
-    <xacro:property name="rear_left_wheel_spinning_link" value="rear_left_wheel_spinning_link"/>
-    <xacro:property name="rear_right_wheel_spinning_link" value="rear_right_wheel_spinning_link}"/>
-    <!-- Joint names -->
-    <xacro:property name="base_footprint_joint" value="base_footprint_joint"/>
-    <xacro:property name="inertial_joint" value="inertial_joint"/>
-    <xacro:property name="front_axle_steering_joint" value="front_axle_steering_joint"/>
-    <xacro:property name="rear_axle_steering_joint" value="rear_axle_steering_joint"/>
-    <xacro:property name="front_left_wheel_steering_joint" value="front_left_wheel_steering_joint"/>
-    <xacro:property name="front_right_wheel_steering_joint" value="front_right_wheel_steering_joint"/>
-    <xacro:property name="rear_left_wheel_steering_joint" value="rear_left_wheel_steering_joint"/>
-    <xacro:property name="rear_right_wheel_steering_joint" value="rear_right_wheel_steering_joint"/>
-    <xacro:property name="front_left_wheel_spinning_joint" value="front_left_wheel_spinning_joint"/>
-    <xacro:property name="front_right_wheel_spinning_joint" value="front_right_wheel_spinning_joint" />
-    <xacro:property name="rear_left_wheel_spinning_joint" value="rear_left_wheel_spinning_joint" />
-    <xacro:property name="rear_right_wheel_spinning_joint" value="rear_right_wheel_spinning_joint" />
-    <!-- Base Properties -->
-    <xacro:property name="ground_clearance" value="0.35"/>
-    <xacro:property name="aabb_length" value="1.66" />
-    <xacro:property name="aabb_width" value="0.6" />
-    <xacro:property name="aabb_height" value="0.6" />
-    <xacro:property name="aabb_center_x" value="0.0" />
-    <xacro:property name="aabb_center_y" value="0.0" />
-    <xacro:property name="aabb_center_z" value="${aabb_height/2.0+ground_clearance}" />
-    <xacro:property name="wheelbase" value="2.0"/>
-    <xacro:property name="front_track" value="0.9"/>
-    <xacro:property name="rear_track" value="0.9"/>
-    <xacro:property name="mass_base" value="500.0" />
-    <xacro:property name="mass_center_x" value="0.0" />
-    <xacro:property name="mass_center_y" value="0.0" />
-    <xacro:property name="mass_center_z" value="0.68" />
-    <xacro:property name="maximal_axle_steering_angle" value="0.2"/>
-    <xacro:property name="maximal_wheel_steering_angle" value="${atan(tan(maximal_axle_steering_angle)/(1-tan(maximal_axle_steering_angle)*front_track/(2*wheelbase)))}"/>
-    <xacro:property name="minimal_axle_steering_angle" value="${-maximal_axle_steering_angle}"/>
-    <xacro:property name="minimal_wheel_steering_angle" value="${-maximal_wheel_steering_angle} "/>
-    <xacro:property name="maximal_wheel_speed" value="2.0"/>
-    <xacro:property name="body_reference_x" value="-0.6" />
-     <!-- Wheel Properties -->
-     <xacro:property name="steering_link_mass" value="30" />
-     <xacro:property name="steering_link_y" value="0.05" />
-     <xacro:property name="steering_link_xz" value="0.1" />
-     <xacro:property name="front_wheel_radius" value="0.398" />
-     <xacro:property name="rear_wheel_radius" value="0.398" />
-     <xacro:property name="front_wheel_width" value="0.2" />
-     <xacro:property name="rear_wheel_width" value="0.2" />
-     <xacro:property name="front_wheel_mass" value="10" />
-     <xacro:property name="rear_wheel_mass" value="10" />
-     <xacro:property name="wheel_radius" value="${front_wheel_radius}" />
-     <xacro:property name="wheel_width" value="${front_wheel_width}" />
-     <!-- Wheel Mounting Positions -->
-     <xacro:property name="front_wheel_y_offset" value="0.1" />
-     <xacro:property name="rear_wheel_y_offset" value="0.1" />
-     <xacro:property name="chassis_height" value="${min(front_wheel_radius,rear_wheel_radius)}" />
-     <xacro:chassis>
-       <!-- visual chassis -->
-       <visual>
-        <origin xyz="${aabb_center_x-body_reference_x} ${aabb_center_y}  ${aabb_center_z-chassis_height}" rpy="0 0 0" />
-         <geometry>
-           <box size="${aabb_length} ${aabb_width} ${aabb_height}"/>
-         </geometry>
-       </visual>
-       <!-- visual front steering -->
-       <box size="${steering_link_xz} ${steering_link_y} ${steering_link_xz}"/>
-       <!-- visual wheel -->
-       <cylinder length="${wheel_width}" radius="${wheel_radius}"/>
-     </xacro:chassis>
-     <xacro:base_control mode="test"/>
+  <xacro:arg name="type" default="" />
+  <xacro:include filename="$(find romea_mobile_base_description)/urdf/base2ASxxx.chassis.xacro" />
+  <xacro:include
+    filename="$(find romea_mobile_base_description)/ros2_control/base$(arg type).ros2_control.xacro" />
+  <xacro:property name="prefix" value="" />
+  <!-- Link names -->
+  <xacro:property name="base_link" value="base_link" />
+  <xacro:property name="base_footprint_link" value="base_footprint_link" />
+  <xacro:property name="inertial_link" value="inertial_link" />
+  <xacro:property name="front_axle_steering_link" value="front_axle_steering_link" />
+  <xacro:property name="rear_axle_steering_link" value="rear_axle_steering_link" />
+  <xacro:property name="front_left_wheel_steering_link" value="front_left_wheel_steering_link" />
+  <xacro:property name="front_right_wheel_steering_link" value="front_right_wheel_steering_link" />
+  <xacro:property name="rear_left_wheel_steering_link" value="rear_left_wheel_steering_link" />
+  <xacro:property name="rear_right_wheel_steering_link" value="rear_right_wheel_steering_link" />
+  <xacro:property name="front_left_wheel_spinning_link" value="front_left_wheel_spinning_link" />
+  <xacro:property name="front_right_wheel_spinning_link" value="front_right_wheel_spinning_link" />
+  <xacro:property name="rear_left_wheel_spinning_link" value="rear_left_wheel_spinning_link" />
+  <xacro:property name="rear_right_wheel_spinning_link" value="rear_right_wheel_spinning_link}" />
+  <!-- Joint names -->
+  <xacro:property name="base_footprint_joint" value="base_footprint_joint" />
+  <xacro:property name="inertial_joint" value="inertial_joint" />
+  <xacro:property name="front_axle_steering_joint" value="front_axle_steering_joint" />
+  <xacro:property name="rear_axle_steering_joint" value="rear_axle_steering_joint" />
+  <xacro:property name="front_left_wheel_steering_joint" value="front_left_wheel_steering_joint" />
+  <xacro:property name="front_right_wheel_steering_joint" value="front_right_wheel_steering_joint" />
+  <xacro:property name="rear_left_wheel_steering_joint" value="rear_left_wheel_steering_joint" />
+  <xacro:property name="rear_right_wheel_steering_joint" value="rear_right_wheel_steering_joint" />
+  <xacro:property name="front_left_wheel_spinning_joint" value="front_left_wheel_spinning_joint" />
+  <xacro:property name="front_right_wheel_spinning_joint" value="front_right_wheel_spinning_joint" />
+  <xacro:property name="rear_left_wheel_spinning_joint" value="rear_left_wheel_spinning_joint" />
+  <xacro:property name="rear_right_wheel_spinning_joint" value="rear_right_wheel_spinning_joint" />
+  <!-- Base Properties -->
+  <xacro:property name="ground_clearance" value="0.35" />
+  <xacro:property name="aabb_length" value="1.66" />
+  <xacro:property name="aabb_width" value="0.6" />
+  <xacro:property name="aabb_height" value="0.6" />
+  <xacro:property name="aabb_center_x" value="0.0" />
+  <xacro:property name="aabb_center_y" value="0.0" />
+  <xacro:property name="aabb_center_z" value="${aabb_height/2.0+ground_clearance}" />
+  <xacro:property name="wheelbase" value="2.0" />
+  <xacro:property name="front_track" value="0.9" />
+  <xacro:property name="rear_track" value="0.9" />
+  <xacro:property name="mass_base" value="500.0" />
+  <xacro:property name="mass_center_x" value="0.0" />
+  <xacro:property name="mass_center_y" value="0.0" />
+  <xacro:property name="mass_center_z" value="0.68" />
+  <xacro:property name="maximal_axle_steering_angle" value="0.2" />
+  <xacro:property name="maximal_wheel_steering_angle"
+    value="${atan(tan(maximal_axle_steering_angle)/(1-tan(maximal_axle_steering_angle)*front_track/(2*wheelbase)))}" />
+  <xacro:property name="minimal_axle_steering_angle" value="${-maximal_axle_steering_angle}" />
+  <xacro:property name="minimal_wheel_steering_angle" value="${-maximal_wheel_steering_angle} " />
+  <xacro:property name="maximal_wheel_speed" value="2.0" />
+  <xacro:property name="body_reference_x" value="-0.6" />
+  <!-- Wheel Properties -->
+  <xacro:property name="steering_link_mass" value="30" />
+  <xacro:property name="steering_link_y" value="0.05" />
+  <xacro:property name="steering_link_xz" value="0.1" />
+  <xacro:property name="front_wheel_radius" value="0.398" />
+  <xacro:property name="rear_wheel_radius" value="0.398" />
+  <xacro:property name="front_wheel_width" value="0.2" />
+  <xacro:property name="rear_wheel_width" value="0.2" />
+  <xacro:property name="front_wheel_mass" value="10" />
+  <xacro:property name="rear_wheel_mass" value="10" />
+  <xacro:property name="wheel_radius" value="${front_wheel_radius}" />
+  <xacro:property name="wheel_width" value="${front_wheel_width}" />
+  <!-- Wheel Mounting Positions -->
+  <xacro:property name="front_wheel_y_offset" value="0.1" />
+  <xacro:property name="rear_wheel_y_offset" value="0.1" />
+  <xacro:property name="chassis_height" value="${min(front_wheel_radius,rear_wheel_radius)}" />
+  <xacro:chassis>
+    <!-- visual chassis -->
+    <visual>
+      <origin
+        xyz="${aabb_center_x-body_reference_x} ${aabb_center_y}  ${aabb_center_z-chassis_height}"
+        rpy="0 0 0" />
+      <geometry>
+        <box size="${aabb_length} ${aabb_width} ${aabb_height}" />
+      </geometry>
+    </visual>
+    <!-- visual front steering -->
+    <box size="${steering_link_xz} ${steering_link_y} ${steering_link_xz}" />
+    <!-- visual wheel -->
+    <cylinder length="${wheel_width}" radius="${wheel_radius}" />
+  </xacro:chassis>
+  <xacro:base_control mode="test" />
 </robot>
