Commit message: gazebo: update xacro test files
Signed-off-by: jean.laneurit <jean.laneurit@inrae.fr>

File: romea_mobile_base_gazebo/test/test_gazebo_interface1FASxxx.xacro (robot description, xacro)
@@ -32,5 +32,4 @@
   <xacro:property name="rear_right_wheel_spinning_joint" value="rear_right_wheel_spinning_joint" />
   <!-- Base Properties -->
-  <xacro:property name="ground_clearance" value="0.35" />
   <xacro:property name="aabb_length" value="1.66" />
   <xacro:property name="aabb_width" value="0.6" />
@@ -46,15 +45,9 @@
   <xacro:property name="mass_center_y" value="0.0" />
   <xacro:property name="mass_center_z" value="0.5" />
-  <xacro:property name="maximal_axle_steering_angle" value="1.0" />
-  <xacro:property name="maximal_wheel_steering_angle"
-    value="${atan(tan(maximal_axle_steering_angle)/(1-tan(maximal_axle_steering_angle)*front_track/(2*wheelbase)))}" />
-  <xacro:property name="minimal_axle_steering_angle" value="${-maximal_axle_steering_angle}" />
-  <xacro:property name="minimal_wheel_steering_angle" value="${-maximal_wheel_steering_angle} " />
-  <xacro:property name="maximal_wheel_speed" value="2.0" />
+  <xacro:property name="ground_clearance" value="0.35" />
   <xacro:property name="body_reference_x" value="-1.25" />
   <!-- Wheel Properties -->
-  <xacro:property name="steering_link_mass" value="30" />
-  <xacro:property name="steering_link_y" value="0.05" />
-  <xacro:property name="steering_link_xz" value="0.1" />
+  <xacro:property name="front_wheel_x_offset" value="0" />
+  <xacro:property name="front_hub_carrier_offset" value="0" />
   <xacro:property name="front_wheel_radius" value="0.2" />
   <xacro:property name="rear_wheel_radius" value="0.2" />
@@ -63,24 +56,34 @@
   <xacro:property name="front_wheel_mass" value="10" />
   <xacro:property name="rear_wheel_mass" value="10" />
-  <xacro:property name="wheel_radius" value="${front_wheel_radius}" />
-  <xacro:property name="wheel_width" value="${front_wheel_width}" />
-  <!-- Wheel Mounting Positions -->
-  <xacro:property name="front_wheel_y_offset" value="0.1" />
-  <xacro:property name="rear_wheel_y_offset" value="0.1" />
-  <xacro:property name="chassis_height" value="${min(front_wheel_radius,rear_wheel_radius)}" />
+  <xacro:property name="wheel_mass" value="5" />
+  <xacro:property name="front_wheel_mass" value="5" />
+  <xacro:property name="rear_wheel_mass" value="5" />
+  <xacro:property name="chassis_height" value="0.2" />
+  <xacro:property name="maximal_wheel_speed" value="2.0" />
+  <!-- Steering Properties -->
+  <xacro:property name="maximal_axle_steering_angle" value="1.0" />
+  <xacro:property name="maximal_wheel_steering_angle"
+    value="${atan(tan(maximal_axle_steering_angle)/(1-tan(maximal_axle_steering_angle)*front_track/(2*wheelbase)))}" />
+  <xacro:property name="minimal_axle_steering_angle" value="${-maximal_axle_steering_angle}" />
+  <xacro:property name="minimal_wheel_steering_angle" value="${-maximal_wheel_steering_angle} " />
+  <xacro:property name="minimal_axle_steering_angle"
+    value="${-maximal_axle_steering_angle}" />
+  <xacro:property name="minimal_wheel_steering_angle"
+    value="${-maximal_wheel_steering_angle} " />
+  <xacro:property name="front_axle_steering_link_mass" value="1" />
+  <xacro:property name="front_axle_steering_link_x" value="0.05" />
+  <xacro:property name="front_axle_steering_link_y" value="0.05" />
+  <xacro:property name="front_axle_steering_link_z" value="0.05" />
+  <xacro:property name="front_wheel_steering_link_mass" value="1" />
+  <xacro:property name="front_wheel_steering_link_y" value="${front_hub_carrier_offset}" />
+  <xacro:property name="front_wheel_steering_link_xz" value="0.1" />
   <xacro:chassis>
-    <!-- visual chassis -->
-    <visual>
-      <origin
-        xyz="${aabb_center_x-body_reference_x} ${aabb_center_y}  ${aabb_center_z-chassis_height}"
-        rpy="0 0 0" />
-      <geometry>
-        <box size="${aabb_length} ${aabb_width} ${aabb_height}" />
-      </geometry>
-    </visual>
-    <!-- visual front steering -->
-    <box size="${steering_link_xz} ${steering_link_y} ${steering_link_xz}" />
-    <!-- visual wheel -->
-    <cylinder length="${wheel_width}" radius="${wheel_radius}" />
+    <visual />
+    <visual />
+    <visual />
+    <visual />
+    <visual />
+    <visual />
+    <visual />
   </xacro:chassis>
   <xacro:base_control mode="test" base_name="base" />

File: romea_mobile_base_gazebo/test/test_gazebo_interface2ASxxx.xacro (robot description, xacro)
@@ -48,15 +48,10 @@
   <xacro:property name="mass_center_y" value="0.0" />
   <xacro:property name="mass_center_z" value="0.68" />
-  <xacro:property name="maximal_axle_steering_angle" value="0.2" />
-  <xacro:property name="maximal_wheel_steering_angle"
-    value="${atan(tan(maximal_axle_steering_angle)/(1-tan(maximal_axle_steering_angle)*front_track/(2*wheelbase)))}" />
-  <xacro:property name="minimal_axle_steering_angle" value="${-maximal_axle_steering_angle}" />
-  <xacro:property name="minimal_wheel_steering_angle" value="${-maximal_wheel_steering_angle} " />
-  <xacro:property name="maximal_wheel_speed" value="2.0" />
   <xacro:property name="body_reference_x" value="-0.6" />
   <!-- Wheel Properties -->
-  <xacro:property name="steering_link_mass" value="30" />
-  <xacro:property name="steering_link_y" value="0.05" />
-  <xacro:property name="steering_link_xz" value="0.1" />
+  <xacro:property name="front_wheel_x_offset" value="0.0" />
+  <xacro:property name="rear_wheel_x_offset" value="0.0" />
+  <xacro:property name="front_hub_carrier_offset" value="0.1" />
+  <xacro:property name="rear_hub_carrier_offset" value="0.1" />
   <xacro:property name="front_wheel_radius" value="0.398" />
   <xacro:property name="rear_wheel_radius" value="0.398" />
@@ -65,24 +60,34 @@
   <xacro:property name="front_wheel_mass" value="10" />
   <xacro:property name="rear_wheel_mass" value="10" />
-  <xacro:property name="wheel_radius" value="${front_wheel_radius}" />
-  <xacro:property name="wheel_width" value="${front_wheel_width}" />
-  <!-- Wheel Mounting Positions -->
-  <xacro:property name="front_wheel_y_offset" value="0.1" />
-  <xacro:property name="rear_wheel_y_offset" value="0.1" />
-  <xacro:property name="chassis_height" value="${min(front_wheel_radius,rear_wheel_radius)}" />
+  <xacro:property name="maximal_wheel_speed" value="2.0" />
+  <xacro:property name="chassis_height" value="0.398" />
+  <!-- Steering Properties -->
+  <xacro:property name="maximal_axle_steering_angle" value="0.2" />
+  <xacro:property name="maximal_wheel_steering_angle"
+    value="${atan(tan(maximal_axle_steering_angle)/(1-tan(maximal_axle_steering_angle)*front_track/(2*wheelbase)))}" />
+  <xacro:property name="minimal_axle_steering_angle"
+    value="${-maximal_axle_steering_angle}" />
+  <xacro:property name="minimal_wheel_steering_angle"
+    value="${-maximal_wheel_steering_angle} " />
+  <xacro:property name="front_axle_steering_link_mass" value="1" />
+  <xacro:property name="front_axle_steering_link_x" value="0.05" />
+  <xacro:property name="front_axle_steering_link_y" value="0.05" />
+  <xacro:property name="front_axle_steering_link_z" value="0.05" />
+  <xacro:property name="front_wheel_steering_link_mass" value="30" />
+  <xacro:property name="front_wheel_steering_link_y" value="${front_hub_carrier_offset}" />
+  <xacro:property name="front_wheel_steering_link_xz" value="0.05" />
+  <xacro:property name="rear_wheel_steering_link_mass" value="30" />
+  <xacro:property name="rear_wheel_steering_link_y" value="${rear_hub_carrier_offset}" />
+  <xacro:property name="rear_wheel_steering_link_xz" value="0.05" />
   <xacro:chassis>
-    <!-- visual chassis -->
-    <visual>
-      <origin
-        xyz="${aabb_center_x-body_reference_x} ${aabb_center_y}  ${aabb_center_z-chassis_height}"
-        rpy="0 0 0" />
-      <geometry>
-        <box size="${aabb_length} ${aabb_width} ${aabb_height}" />
-      </geometry>
-    </visual>
-    <!-- visual front steering -->
-    <box size="${steering_link_xz} ${steering_link_y} ${steering_link_xz}" />
-    <!-- visual wheel -->
-    <cylinder length="${wheel_width}" radius="${wheel_radius}" />
+    <visual />
+    <visual />
+    <visual />
+    <visual />
+    <visual />
+    <visual />
+    <visual />
+    <visual />
+    <visual />
   </xacro:chassis>
   <xacro:base_control mode="test" base_name="base" />

File: romea_mobile_base_gazebo/test/test_gazebo_interface2FWSxxx.xacro (robot description, xacro)
@@ -36,5 +36,4 @@
   <xacro:property name="rear_track" value="1.0" />
   <xacro:property name="track" value="${front_track}" />
-  <xacro:property name="ground_clearance" value="0.45" />
   <xacro:property name="mass_base" value="800." />
   <xacro:property name="mass_center_x" value="-0.1" />
@@ -42,46 +41,31 @@
   <xacro:property name="mass_center_z" value=" 0.2" />
   <xacro:property name="body_reference_x" value="-1.0" />
-  <!-- Steering Properties -->
-  <xacro:property name="steering_angle_max_in" value="1.04" />
-  <xacro:property name="steering_angle_max_out" value="0.59" />
-  <xacro:property name="front_wheel_y_offset" value="0.02" />
-  <xacro:property name="rear_wheel_y_offset" value="0.02" />
-  <xacro:property name="wheel_y_offset" value="${front_wheel_y_offset}" />
-  <xacro:property name="steering_link_mass" value="1" />
-  <xacro:property name="steering_link_y_size" value="${wheel_y_offset}" />
-  <xacro:property name="steering_link_xz_size" value="0.1" />
-  <xacro:property name="steering_link_y" value="${wheel_y_offset}" />
-  <xacro:property name="steering_link_xz" value="0.1" />
+  <xacro:property name="ground_clearance" value="0.45" />
   <!-- Wheel Properties -->
+  <xacro:property name="front_wheel_x_offset" value="0.0" />
+  <xacro:property name="front_hub_carrier_offset" value="0.02" />
+  <xacro:property name="rear_hub_carrier_offset" value="0.02" />
   <xacro:property name="front_wheel_radius" value="0.32" />
   <xacro:property name="rear_wheel_radius" value="0.32" />
   <xacro:property name="front_wheel_width" value="0.2" />
   <xacro:property name="rear_wheel_width" value="0.2" />
-  <xacro:property name="wheel_radius" value="${front_wheel_radius}" />
-  <xacro:property name="wheel_width" value="${front_wheel_width}" />
-  <xacro:property name="chassis_height" value="${min(front_wheel_radius,rear_wheel_radius)}" />
+  <xacro:property name="front_wheel_mass" value="5" />
+  <xacro:property name="rear_wheel_mass" value="5" />
+  <xacro:property name="maximal_wheel_speed" value="3.0" />
+  <xacro:property name="chassis_height" value="0.32" />
+  <!-- Steering Properties -->
   <xacro:property name="minimal_wheel_steering_angle" value="-1.04" />
   <xacro:property name="maximal_wheel_steering_angle" value="1.04" />
-  <xacro:property name="maximal_wheel_speed" value="3.0" />
-  <xacro:property name="wheel_mass" value="5" />
-  <xacro:property name="front_wheel_mass" value="5" />
-  <xacro:property name="rear_wheel_mass" value="5" />
+  <xacro:property name="front_wheel_steering_link_mass" value="1" />
+  <xacro:property name="front_wheel_steering_link_y" value="${front_hub_carrier_offset}" />
+  <xacro:property name="front_wheel_steering_link_xz" value="0.05" />
   <xacro:chassis>
-    <!-- visual chassis -->
-    <visual>
-      <origin
-        xyz="${aabb_center_x-body_reference_x} ${aabb_center_y}  ${aabb_center_z-chassis_height}"
-        rpy="0 0 0" />
-      <geometry>
-        <box size="${aabb_length} ${aabb_width} ${aabb_height}" />
-      </geometry>
-      <material name="grey">
-        <color rgba="0.6 0.6 0.6 1" />
-      </material>
-    </visual>
-    <!-- visual front steering -->
-    <box size="${steering_link_xz_size} ${steering_link_y_size} ${steering_link_xz_size}" />
-    <!-- visual wheel -->
-    <cylinder length="${wheel_width}" radius="${wheel_radius}" />
+    <visual />
+    <visual />
+    <visual />
+    <visual />
+    <visual />
+    <visual />
+    <visual />
   </xacro:chassis>
   <xacro:base_control mode="test" base_name="base" />

File: romea_mobile_base_gazebo/test/test_gazebo_interface2TD.xacro (robot description, xacro)
@@ -2,96 +2,71 @@
 <robot name="robot" xmlns:xacro="http://ros.org/wiki/xacro">
   <xacro:property name="M_PI" value="3.14159" />
-    <xacro:include
+  <xacro:include
     filename="$(find romea_mobile_base_description)/urdf/base2TD.chassis.xacro" />
-    <xacro:include
+  <xacro:include
     filename="$(find romea_mobile_base_description)/ros2_control/base2TD.ros2_control.xacro" />
-    <xacro:property
+  <xacro:property
     name="prefix" value="" />
   <!-- Link names -->
-     <xacro:property name="base_link" value="base_link" />
-     <xacro:property
-    name="base_footprint_link" value="base_footprint_link" />
-     <xacro:property name="inertial_link"
+  <xacro:property name="base_link"
+    value="base_link" />
+  <xacro:property name="base_footprint_link"
+    value="base_footprint_link" />
+  <xacro:property name="inertial_link"
     value="inertial_link" />
-     <xacro:property name="left_sprocket_wheel_spinning_link"
+  <xacro:property name="left_sprocket_wheel_spinning_link"
     value="left_sprocket_wheel_spinning_link" />
-     <xacro:property
-    name="right_sprocket_wheel_spinning_link" value="right_sprocket_wheel_spinning_link" />
-     <xacro:property
-    name="left_idler_wheel_spinning_link" value="left_idler_wheel_spinning_link" />
-     <xacro:property
-    name="right_idler_wheel_spinning_link" value="right_idler_wheel_spinning_link" />
+  <xacro:property name="right_sprocket_wheel_spinning_link"
+    value="right_sprocket_wheel_spinning_link" />
+  <xacro:property name="left_idler_wheel_spinning_link"
+    value="left_idler_wheel_spinning_link" />
+  <xacro:property name="right_idler_wheel_spinning_link"
+    value="right_idler_wheel_spinning_link" />
   <!-- Joint names -->
-     <xacro:property
-    name="base_footprint_joint" value="base_footprint_joint" />
-     <xacro:property name="inertial_joint"
+  <xacro:property name="base_footprint_joint"
+    value="base_footprint_joint" />
+  <xacro:property name="inertial_joint"
     value="inertial_joint" />
-     <xacro:property name="left_sprocket_wheel_spinning_joint"
+  <xacro:property name="left_sprocket_wheel_spinning_joint"
     value="left_sprocket_wheel_spinning_joint" />
-     <xacro:property
-    name="right_sprocket_wheel_spinning_joint" value="right_sprocket_wheel_spinning_joint" />
-     <xacro:property
-    name="left_idler_wheel_spinning_joint" value="left_idler_wheel_spinning_joint" />
-     <xacro:property
-    name="right_idler_wheel_spinning_joint" value="right_idler_wheel_spinning_joint" />
+  <xacro:property name="right_sprocket_wheel_spinning_joint"
+    value="right_sprocket_wheel_spinning_joint" />
+  <xacro:property name="left_idler_wheel_spinning_joint"
+    value="left_idler_wheel_spinning_joint" />
+  <xacro:property name="right_idler_wheel_spinning_joint"
+    value="right_idler_wheel_spinning_joint" />
   <!-- Base Properties -->
-      <xacro:property
-    name="track_width" value="0.2" />
-      <xacro:property name="track_thickness" value="0.08" />
-      <xacro:property
-    name="sprocket_wheel_radius" value="0.15" />
-      <xacro:property name="sprocket_wheel_mass"
-    value="30" />
-      <xacro:property name="idler_wheel_radius" value="0.15" />
-      <xacro:property
-    name="idler_wheel_mass" value="30" />
-      <xacro:property name="ground_clearance"
-    value="${sprocket_wheel_radius}" />
-      <xacro:property name="aabb_length" value="2.0" />
-      <xacro:property
-    name="aabb_width" value="1.0" />
-      <xacro:property name="aabb_height" value="2.3" />
-      <xacro:property
-    name="aabb_center_x" value="0" />
-      <xacro:property name="aabb_center_y" value="0" />
-      <xacro:property
-    name="aabb_center_z" value="${aabb_height/2+ground_clearance}" />
-      <xacro:property
-    name="wheelbase" value="1.6" />
-      <xacro:property name="front_track" value="1.2" />
-      <xacro:property
-    name="rear_track" value="1.2" />
-      <xacro:property name="track" value="${front_track}" />
-      <xacro:property
-    name="mass_base" value="1000." />
-      <xacro:property name="mass_center_x" value=" 0.0" />
-      <xacro:property
-    name="mass_center_y" value=" 0.0" />
-      <xacro:property name="mass_center_z" value=" 0.2" />
-      <xacro:property
-    name="body_reference_x" value="0.0" />
-      <xacro:property name="maximal_track_speed" value="3.0" />
-      <xacro:property
-    name="maximal_wheel_speed" value="${maximal_track_speed}" />
-      <xacro:property
-    name="chassis_height" value="${min(sprocket_wheel_radius,idler_wheel_radius)}" />
-  ${ground_clearance+aabb_height/2-chassis_height} <xacro:chassis>
-    <visual>
-      <geometry>
-        <box size="${aabb_length} ${aabb_width} ${aabb_height}" />
-      </geometry>
-      <origin
-        xyz="${aabb_center_x-body_reference_x} ${aabb_center_y}  ${aabb_center_z-chassis_height}"
-        rpy="0 0 0" />
-      <material name="grey">
-        <color rgba="0.6 0.6 0.6 1" />
-      </material>
-    </visual>
-    <!-- visual sprocket wheel -->
-    <cylinder length="${track_width}" radius="${sprocket_wheel_radius+track_thickness}" />
-    <!-- visual idler wheel -->
-    <cylinder length="${track_width}" radius="${idler_wheel_radius+track_thickness}" />
+  <xacro:property name="track_width" value="0.2" />
+  <xacro:property name="track_thickness" value="0.08" />
+  <xacro:property name="sprocket_wheel_radius" value="0.15" />
+  <xacro:property name="sprocket_wheel_mass" value="30" />
+  <xacro:property name="idler_wheel_radius" value="0.15" />
+  <xacro:property name="idler_wheel_mass" value="30" />
+  <xacro:property name="ground_clearance" value="${sprocket_wheel_radius}" />
+  <xacro:property name="aabb_length" value="2.0" />
+  <xacro:property name="aabb_width" value="1.0" />
+  <xacro:property name="aabb_height" value="2.3" />
+  <xacro:property name="aabb_center_x" value="0" />
+  <xacro:property name="aabb_center_y" value="0" />
+  <xacro:property name="aabb_center_z" value="${aabb_height/2+ground_clearance}" />
+  <xacro:property name="wheelbase" value="1.6" />
+  <xacro:property name="front_track" value="1.2" />
+  <xacro:property name="rear_track" value="1.2" />
+  <xacro:property name="track" value="${front_track}" />
+  <xacro:property name="mass_base" value="1000." />
+  <xacro:property name="mass_center_x" value=" 0.0" />
+  <xacro:property name="mass_center_y" value=" 0.0" />
+  <xacro:property name="mass_center_z" value=" 0.2" />
+  <xacro:property name="body_reference_x" value="0.0" />
+  <xacro:property name="maximal_track_speed" value="3.0" />
+  <xacro:property name="maximal_wheel_speed" value="${maximal_track_speed}" />
+  <xacro:property name="chassis_height" value="${min(sprocket_wheel_radius,idler_wheel_radius)}" />
+  <xacro:chassis>
+    <visual />
+    <visual />
+    <visual />
+    <visual />
+    <visual />
   </xacro:chassis>
-  <xacro:base_control
-    mode="test" base_name="base" />
+  <xacro:base_control mode="test" base_name="base" />
 </robot>

File: romea_mobile_base_gazebo/test/test_gazebo_interface2THD.xacro (robot description, xacro)
@@ -7,8 +7,11 @@
   <xacro:property name="prefix" value="" />
   <!-- Link names -->
-  <xacro:property name="base_link" value="base_link" />
-  <xacro:property name="base_footprint_link" value="base_footprint_link" />
+  <xacro:property name="base_link"
+    value="base_link" />
+  <xacro:property name="base_footprint_link"
+    value="base_footprint_link" />
   <xacro:property name="inertial_link" value="inertial_link" />
-  <xacro:property name="left_sprocket_wheel_spinning_link" value="left_sprocket_wheel_spinning_link" />
+  <xacro:property name="left_sprocket_wheel_spinning_link"
+    value="left_sprocket_wheel_spinning_link" />
   <xacro:property name="right_sprocket_wheel_spinning_link"
     value="right_sprocket_wheel_spinning_link" />
@@ -22,6 +25,8 @@
     value="rear_right_idler_wheel_spinning_link" />
   <!-- Joint names -->
-  <xacro:property name="base_footprint_joint" value="base_footprint_joint" />
-  <xacro:property name="inertial_joint" value="inertial_joint" />
+  <xacro:property name="base_footprint_joint"
+    value="base_footprint_joint" />
+  <xacro:property name="inertial_joint"
+    value="inertial_joint" />
   <xacro:property name="left_sprocket_wheel_spinning_joint"
     value="left_sprocket_wheel_spinning_joint" />
@@ -65,19 +70,9 @@
   <xacro:property name="chassis_height" value="${idler_wheel_radius}" />
   <xacro:chassis>
-    <visual>
-      <geometry>
-        <box size="${aabb_length} ${aabb_width} ${aabb_height}" />
-      </geometry>
-      <origin
-        xyz="${aabb_center_x-body_reference_x} ${aabb_center_y}  ${aabb_center_z-chassis_height}"
-        rpy="0 0 0" />
-      <material name="grey">
-        <color rgba="0.6 0.6 0.6 1" />
-      </material>
-    </visual>
-    <!-- visual sprocket wheel -->
-    <cylinder length="${track_width}" radius="${sprocket_wheel_radius+track_thickness}" />
-    <!-- visual idler wheel -->
-    <cylinder length="${track_width}" radius="${idler_wheel_radius+track_thickness}" />
+    <visual />
+    <visual />
+    <visual />
+    <visual />
+    <visual />
   </xacro:chassis>
   <xacro:base_control mode="test" base_name="base" />
