Commit message: gazebo: update xacro test files
Signed-off-by: jean.laneurit <jean.laneurit@inrae.fr>

File: romea_mobile_base_gazebo/test/test_gazebo_interface2TTD.xacro (robot description, xacro)
@@ -7,12 +7,18 @@
   <xacro:property name="prefix" value="" />
   <!-- Link names -->
-  <xacro:property name="base_link" value="base_link" />
-  <xacro:property name="base_footprint_link" value="base_footprint_link" />
-  <xacro:property name="inertial_link" value="inertial_link" />
-  <xacro:property name="left_sprocket_wheel_spinning_link" value="left_sprocket_wheel_spinning_link" />
+  <xacro:property name="base_link"
+    value="base_link" />
+  <xacro:property name="base_footprint_link"
+    value="base_footprint_link" />
+  <xacro:property name="inertial_link"
+    value="inertial_link" />
+  <xacro:property name="left_sprocket_wheel_spinning_link"
+    value="left_sprocket_wheel_spinning_link" />
   <xacro:property name="right_sprocket_wheel_spinning_link"
     value="right_sprocket_wheel_spinning_link" />
-  <xacro:property name="left_idler_wheel_spinning_link" value="left_idler_wheel_spinning_link" />
-  <xacro:property name="right_idler_wheel_spinning_link" value="right_idler_wheel_spinning_link" />
+  <xacro:property name="left_idler_wheel_spinning_link"
+    value="left_idler_wheel_spinning_link" />
+  <xacro:property name="right_idler_wheel_spinning_link"
+    value="right_idler_wheel_spinning_link" />
   <xacro:property name="front_left_roller_wheel_spinning_link"
     value="front_left_roller_wheel_spinning_link" />
@@ -24,12 +30,16 @@
     value="rear_right_roller_wheel_spinning_link" />
   <!-- Joint names -->
-  <xacro:property name="base_footprint_joint" value="base_footprint_joint" />
-  <xacro:property name="inertial_joint" value="inertial_joint" />
+  <xacro:property name="base_footprint_joint"
+    value="base_footprint_joint" />
+  <xacro:property name="inertial_joint"
+    value="inertial_joint" />
   <xacro:property name="left_sprocket_wheel_spinning_joint"
     value="left_sprocket_wheel_spinning_joint" />
   <xacro:property name="right_sprocket_wheel_spinning_joint"
     value="right_sprocket_wheel_spinning_joint" />
-  <xacro:property name="left_idler_wheel_spinning_joint" value="left_idler_wheel_spinning_joint" />
-  <xacro:property name="right_idler_wheel_spinning_joint" value="right_idler_wheel_spinning_joint" />
+  <xacro:property name="left_idler_wheel_spinning_joint"
+    value="left_idler_wheel_spinning_joint" />
+  <xacro:property name="right_idler_wheel_spinning_joint"
+    value="right_idler_wheel_spinning_joint" />
   <xacro:property name="front_left_roller_wheel_spinning_joint"
     value="front_left_roller_wheel_spinning_joint" />
@@ -73,21 +83,11 @@
   <xacro:property name="chassis_height" value="${idler_wheel_radius}" />
   <xacro:chassis>
-    <visual>
-      <geometry>
-        <box size="${aabb_length} ${aabb_width} ${aabb_height}" />
-      </geometry>
-      <origin
-        xyz="${aabb_center_x-body_reference_x} ${aabb_center_y}  ${aabb_center_z-chassis_height}"
-        rpy="0 0 0" />
-      <material name="grey">
-        <color rgba="0.6 0.6 0.6 1" />
-      </material>
-    </visual>
-    <!-- visual sprocket wheel -->
-    <cylinder length="${track_width}" radius="${sprocket_wheel_radius+track_thickness}" />
-    <!-- visual idler wheel -->
-    <cylinder length="${track_width}" radius="${idler_wheel_radius+track_thickness}" />
-    <!-- visual roller wheel -->
-    <cylinder length="${track_width}" radius="${roller_wheel_radius+track_thickness}" />
+    <visual />
+    <visual />
+    <visual />
+    <visual />
+    <visual />
+    <visual />
+    <visual />
   </xacro:chassis>
   <xacro:base_control mode="test" base_name="base" />

File: romea_mobile_base_gazebo/test/test_gazebo_interface4WD.xacro (robot description, xacro)
@@ -7,18 +7,29 @@
   <xacro:property name="prefix" value="" />
   <!-- Link names -->
-  <xacro:property name="base_link" value="base_link" />
-  <xacro:property name="base_footprint_link" value="base_footprint_link" />
-  <xacro:property name="inertial_link" value="inertial_link_name" />
-  <xacro:property name="front_left_wheel_spinning_link" value="front_left_wheel_spinning_link" />
-  <xacro:property name="front_right_wheel_spinning_link" value="front_right_wheel_spinning_link" />
-  <xacro:property name="rear_left_wheel_spinning_link" value="rear_left_wheel_spinning_link" />
-  <xacro:property name="rear_right_wheel_spinning_link" value="rear_right_wheel_spinning_link" />
+  <xacro:property name="base_link"
+    value="base_link" />
+  <xacro:property name="base_footprint_link"
+    value="base_footprint_link" />
+  <xacro:property name="inertial_link"
+    value="inertial_link_name" />
+  <xacro:property name="front_left_wheel_spinning_link"
+    value="front_left_wheel_spinning_link" />
+  <xacro:property name="front_right_wheel_spinning_link"
+    value="front_right_wheel_spinning_link" />
+  <xacro:property name="rear_left_wheel_spinning_link"
+    value="rear_left_wheel_spinning_link" />
+  <xacro:property name="rear_right_wheel_spinning_link"
+    value="rear_right_wheel_spinning_link" />
   <!-- Joint names -->
-  <xacro:property name="base_footprint_joint" value="base_footprint_joint" />
-  <xacro:property name="inertial_joint" value="inertial_joint" />
-  <xacro:property name="front_left_wheel_spinning_joint" value="front_left_wheel_spinning_joint" />
+  <xacro:property name="base_footprint_joint"
+    value="base_footprint_joint" />
+  <xacro:property name="inertial_joint"
+    value="inertial_joint" />
+  <xacro:property name="front_left_wheel_spinning_joint"
+    value="front_left_wheel_spinning_joint" />
   <xacro:property name="front_right_wheel_spinning_joint"
     value="front_right_wheel_spinning_joint_name" />
-  <xacro:property name="rear_left_wheel_spinning_joint" value="rear_left_wheel_spinning_joint_name" />
+  <xacro:property name="rear_left_wheel_spinning_joint"
+    value="rear_left_wheel_spinning_joint_name" />
   <xacro:property name="rear_right_wheel_spinning_joint"
     value="rear_right_wheel_spinning_joint_name" />
@@ -55,17 +66,9 @@
   <xacro:property name="chassis_height" value="${min(front_wheel_radius,rear_wheel_radius)}" />
   <xacro:chassis>
-    <visual>
-      <geometry>
-        <box size="${aabb_length} ${aabb_width} ${aabb_height}" />
-      </geometry>
-      <origin
-        xyz="${aabb_center_x-body_reference_x} ${aabb_center_y}  ${aabb_center_z-chassis_height}"
-        rpy="0 0 0" />
-      <material name="grey">
-        <color rgba="0.6 0.6 0.6 1" />
-      </material>
-    </visual>
-    <!-- visual wheel -->
-    <cylinder length="${wheel_width}" radius="${wheel_radius}" />
+    <visual />
+    <visual />
+    <visual />
+    <visual />
+    <visual />
   </xacro:chassis>
   <xacro:base_control mode="test" base_name="base" />

File: romea_mobile_base_gazebo/test/test_gazebo_interface4WS4WD.xacro (robot description, xacro)
@@ -2,7 +2,7 @@
 <robot name="robot" xmlns:xacro="http://www.ros.org/wiki/xacro">
   <xacro:arg name="type" default="" />
-  <xacro:include filename="$(find romea_mobile_base_description)/urdf/base2FWS4WD.chassis.xacro" />
+  <xacro:include filename="$(find romea_mobile_base_description)/urdf/base4WS4WD.chassis.xacro" />
   <xacro:include
-    filename="$(find romea_mobile_base_description)/ros2_control/base$(arg type).ros2_control.xacro" />
+    filename="$(find romea_mobile_base_description)/ros2_control/base4WS4WD.ros2_control.xacro" />
   <xacro:property name="prefix" value="" />
   <!-- Link names -->
@@ -12,4 +12,6 @@
   <xacro:property name="front_left_wheel_steering_link" value="front_left_wheel_steering_link" />
   <xacro:property name="front_right_wheel_steering_link" value="front_right_wheel_steering_link" />
+  <xacro:property name="rear_left_wheel_steering_link" value="rear_left_wheel_steering_link" />
+  <xacro:property name="rear_right_wheel_steering_link" value="rear_right_wheel_steering_link" />
   <xacro:property name="front_left_wheel_spinning_link" value="front_left_wheel_spinning_link" />
   <xacro:property name="front_right_wheel_spinning_link" value="front_right_wheel_spinning_link" />
@@ -21,4 +23,6 @@
   <xacro:property name="front_left_wheel_steering_joint" value="front_left_wheel_steering_joint" />
   <xacro:property name="front_right_wheel_steering_joint" value="front_right_wheel_steering_joint" />
+  <xacro:property name="rear_left_wheel_steering_joint" value="rear_left_wheel_steering_joint" />
+  <xacro:property name="rear_right_wheel_steering_joint" value="rear_right_wheel_steering_joint" />
   <xacro:property name="front_left_wheel_spinning_joint" value="front_left_wheel_spinning_joint" />
   <xacro:property name="front_right_wheel_spinning_joint" value="front_right_wheel_spinning_joint" />
@@ -29,9 +33,11 @@
   <xacro:property name="aabb_width" value="1.18" />
   <xacro:property name="aabb_height" value="1.5" />
+  <xacro:property name="aabb_center_x" value="0" />
+  <xacro:property name="aabb_center_y" value="0" />
+  <xacro:property name="aabb_center_z" value="1" />
   <xacro:property name="wheelbase" value="2.0" />
   <xacro:property name="front_track" value="1.0" />
   <xacro:property name="rear_track" value="1.0" />
   <xacro:property name="track" value="${front_track}" />
-  <xacro:property name="ground_clearance" value="0.45" />
   <!--    <xacro:property name="mass_body" value="800." />-->
   <xacro:property name="mass_base" value="800." />
@@ -39,4 +45,6 @@
   <xacro:property name="mass_center_y" value=" 0.0" />
   <xacro:property name="mass_center_z" value=" 0.2" />
+  <xacro:property name="body_reference_x" value="-1.0" />
+  <xacro:property name="ground_clearance" value="0.45" />
   <!--    <xacro:property name="body_length" value="2.6" />
     <xacro:property name="body_width" value="1.18" />
@@ -44,5 +52,4 @@
   <!--    <xacro:property name="body_offset_x" value="-1.0" />-->
   <!--    <xacro:property name="body_origin_z" value="0.0" />-->
-  <xacro:property name="body_reference_x" value="-1.0" />
   <!-- Steering Properties -->
   <xacro:property name="steering_angle_max_in" value="1.04" />
@@ -57,33 +64,35 @@
   <xacro:property name="steering_link_xz" value="0.1" />
   <!-- Wheel Properties -->
+  <xacro:property name="front_wheel_x_offset" value="0.0" />
+  <xacro:property name="rear_wheel_x_offset" value="0.0" />
+  <xacro:property name="front_hub_carrier_offset" value="0.1" />
+  <xacro:property name="rear_hub_carrier_offset" value="0.1" />
   <xacro:property name="front_wheel_radius" value="0.32" />
   <xacro:property name="rear_wheel_radius" value="0.32" />
   <xacro:property name="front_wheel_width" value="0.2" />
   <xacro:property name="rear_wheel_width" value="0.2" />
-  <xacro:property name="wheel_radius" value="${front_wheel_radius}" />
-  <xacro:property name="wheel_width" value="${front_wheel_width}" />
-  <xacro:property name="chassis_height" value="${min(front_wheel_radius,rear_wheel_radius)}" />
+  <xacro:property name="front_wheel_mass" value="5" />
+  <xacro:property name="rear_wheel_mass" value="5" />
+  <xacro:property name="chassis_height" value="0.32" />
+  <xacro:property name="maximal_wheel_speed" value="3.0" />
+  <!-- Steering Properties -->
   <xacro:property name="minimal_wheel_steering_angle" value="-1.04" />
   <xacro:property name="maximal_wheel_steering_angle" value="1.04" />
-  <xacro:property name="maximal_wheel_speed" value="3.0" />
-  <xacro:property name="wheel_mass" value="5" />
-  <xacro:property name="front_wheel_mass" value="5" />
-  <xacro:property name="rear_wheel_mass" value="5" />
+  <xacro:property name="front_wheel_steering_link_mass" value="3" />
+  <xacro:property name="front_wheel_steering_link_y" value="${front_hub_carrier_offset}" />
+  <xacro:property name="front_wheel_steering_link_xz" value="0.05" />
+  <xacro:property name="rear_wheel_steering_link_mass" value="3" />
+  <xacro:property name="rear_wheel_steering_link_y" value="${rear_hub_carrier_offset}" />
+  <xacro:property name="rear_wheel_steering_link_xz" value="0.05" />
   <xacro:chassis>
-    <!-- visual chassis -->
-    <visual>
-      <origin xyz="${-body_reference_x} 0 ${ground_clearance+aabb_height/2-chassis_height}"
-        rpy="0 0 0" />
-      <geometry>
-        <box size="${aabb_length} ${aabb_width} ${aabb_height}" />
-      </geometry>
-      <material name="grey">
-        <color rgba="0.6 0.6 0.6 1" />
-      </material>
-    </visual>
-    <!-- visual front steering -->
-    <box size="${steering_link_xz_size} ${steering_link_y_size} ${steering_link_xz_size}" />
-    <!-- visual wheel -->
-    <cylinder length="${wheel_width}" radius="${wheel_radius}" />
+    <visual />
+    <visual />
+    <visual />
+    <visual />
+    <visual />
+    <visual />
+    <visual />
+    <visual />
+    <visual />
   </xacro:chassis>
   <xacro:base_control mode="test" base_name="base" />
