Commit message: simulation: update xacro tests file
Signed-off-by: jean.laneurit <jean.laneurit@inrae.fr>

File: romea_mobile_base_simulation/test/test_simulation_interface1FAS2FWD.xacro (robot description, xacro)
@@ -17,4 +17,6 @@
   <xacro:property name="rear_wheel_radius" value="0.6" />
   <xacro:property name="rear_hub_carrier_offset" value="0.15" />
+  <xacro:property name="maximal_axle_steering_angle" value="0.50" />
+  <xacro:property name="maximal_wheel_speed" value="1.0" />
   <xacro:include
     filename="$(find romea_mobile_base_description)/ros2_control/base1FAS2FWD.ros2_control.xacro" />

File: romea_mobile_base_simulation/test/test_simulation_interface1FAS2RWD.xacro (robot description, xacro)
@@ -15,4 +15,6 @@
   <xacro:property name="front_hub_carrier_offset" value="0.08" />
   <xacro:property name="rear_wheel_radius" value="0.7" />
+  <xacro:property name="maximal_axle_steering_angle" value="0.50" />
+  <xacro:property name="maximal_wheel_speed" value="1.0" />
   <xacro:include
     filename="$(find romea_mobile_base_description)/ros2_control/base1FAS2RWD.ros2_control.xacro" />

File: romea_mobile_base_simulation/test/test_simulation_interface2FWS2FWD.xacro (robot description, xacro)
@@ -16,4 +16,6 @@
   <xacro:property name="rear_wheel_radius" value="0.6" />
   <xacro:property name="rear_hub_carrier_offset" value="0.15" />
+  <xacro:property name="maximal_wheel_steering_angle" value="0.50" />
+  <xacro:property name="maximal_wheel_speed" value="1.0" />
   <xacro:include
     filename="$(find romea_mobile_base_description)/ros2_control/base2FWS2FWD.ros2_control.xacro" />

File: romea_mobile_base_simulation/test/test_simulation_interface2FWS2RWD.xacro (robot description, xacro)
@@ -15,4 +15,6 @@
   <xacro:property name="rear_track" value="1.0" />
   <xacro:property name="rear_wheel_radius" value="0.3" />
+  <xacro:property name="maximal_wheel_steering_angle" value="0.50" />
+  <xacro:property name="maximal_wheel_speed" value="1.0" />
   <xacro:include
     filename="$(find romea_mobile_base_description)/ros2_control/base2FWS2RWD.ros2_control.xacro" />

File: romea_mobile_base_simulation/test/test_simulation_interface2TD.xacro (robot description, xacro)
@@ -10,4 +10,5 @@
   <xacro:property name="idler_wheel_radius" value="0.3" />
   <xacro:property name="track_thickness" value="0.1" />
+  <xacro:property name="maximal_wheel_speed" value="1.0" />
   <xacro:include
     filename="$(find romea_mobile_base_description)/ros2_control/base2TD.ros2_control.xacro" />

File: romea_mobile_base_simulation/test/test_simulation_interface2THD.xacro (robot description, xacro)
@@ -12,4 +12,5 @@
   <xacro:property name="idler_wheel_radius" value="0.3" />
   <xacro:property name="track_thickness" value="0.1" />
+  <xacro:property name="maximal_wheel_speed" value="1.0" />
   <xacro:include
     filename="$(find romea_mobile_base_description)/ros2_control/base2THD.ros2_control.xacro" />

File: romea_mobile_base_simulation/test/test_simulation_interface2TTD.xacro (robot description, xacro)
@@ -15,4 +15,5 @@
   <xacro:property name="idler_wheel_radius" value="0.3" />
   <xacro:property name="track_thickness" value="0.1" />
+  <xacro:property name="maximal_wheel_speed" value="1.0" />
   <xacro:include
     filename="$(find romea_mobile_base_description)/ros2_control/base2TTD.ros2_control.xacro" />
