Commit message: fix steering link mass for simulation

File: romea_mobile_base_gazebo_classic/test/test_gazebo_interface1FASxxx.xacro (robot description, xacro)
@@ -75,5 +75,5 @@
   <xacro:property name="front_axle_steering_link_y" value="0.05" />
   <xacro:property name="front_axle_steering_link_z" value="0.05" />
-  <xacro:property name="front_wheel_steering_link_mass" value="1" />
+  <xacro:property name="front_wheel_steering_link_mass" value="10" />
   <xacro:property name="front_wheel_steering_link_y" value="${front_hub_carrier_offset}" />
   <xacro:property name="front_wheel_steering_link_xz" value="0.1" />

File: romea_mobile_base_gazebo_classic/test/test_gazebo_interface2FWSxxx.xacro (robot description, xacro)
@@ -57,5 +57,5 @@
   <xacro:property name="minimal_wheel_steering_angle" value="-1.04" />
   <xacro:property name="maximal_wheel_steering_angle" value="1.04" />
-  <xacro:property name="front_wheel_steering_link_mass" value="1" />
+  <xacro:property name="front_wheel_steering_link_mass" value="15" />
   <xacro:property name="front_wheel_steering_link_y" value="${front_hub_carrier_offset}" />
   <xacro:property name="front_wheel_steering_link_xz" value="0.05" />

File: romea_mobile_base_gazebo_classic/test/test_gazebo_interface4WS4WD.xacro (robot description, xacro)
@@ -79,8 +79,8 @@
   <xacro:property name="minimal_wheel_steering_angle" value="-1.04" />
   <xacro:property name="maximal_wheel_steering_angle" value="1.04" />
-  <xacro:property name="front_wheel_steering_link_mass" value="3" />
+  <xacro:property name="front_wheel_steering_link_mass" value="15" />
   <xacro:property name="front_wheel_steering_link_y" value="${front_hub_carrier_offset}" />
   <xacro:property name="front_wheel_steering_link_xz" value="0.05" />
-  <xacro:property name="rear_wheel_steering_link_mass" value="3" />
+  <xacro:property name="rear_wheel_steering_link_mass" value="15" />
   <xacro:property name="rear_wheel_steering_link_y" value="${rear_hub_carrier_offset}" />
   <xacro:property name="rear_wheel_steering_link_xz" value="0.05" />
