Commit message: add GazeboSystemInterface plugin add GenericGazeboSystemInterface plugin add GenericHardwareSystemInterface plugin add support of 2FWC2RWD robot
Signed-off-by: Jean Laneurit <jean.laneurit@inrae.fr>

File: romea_mobile_base_utils/test/test_hardware_info1FASxxx.xacro (robot description, xacro)
@@ -1,4 +1,25 @@
 <?xml version='1.0' encoding='utf-8'?>
 <robot name="robot" xmlns:xacro="http://www.ros.org/wiki/xacro">
+  <link name="robot_base_link" />
+  <link name="robot_link1" />
+  <link name="robot_link2" />
+  <link name="robot_link3" />
+  <link name="robot_link4" />
+  <link name="robot_link5" />
+  <link name="robot_link6" />
+  <link name="robot_link7" />
+  <link name="robot_link8" />
+  <link name="robot_link9" />
+  <link name="robot_link10" />
+  <joint name="robot_joint1" type="continuous"><parent link="robot_base_link"/><child link="robot_link1"/></joint>
+  <joint name="robot_joint2" type="continuous"><parent link="robot_base_link"/><child link="robot_link2"/></joint>
+  <joint name="robot_joint3" type="continuous"><parent link="robot_base_link"/><child link="robot_link3"/></joint>
+  <joint name="robot_joint4" type="continuous"><parent link="robot_base_link"/><child link="robot_link4"/></joint>
+  <joint name="robot_joint5" type="continuous"><parent link="robot_base_link"/><child link="robot_link5"/></joint>
+  <joint name="robot_joint6" type="continuous"><parent link="robot_base_link"/><child link="robot_link6"/></joint>
+  <joint name="robot_joint7" type="continuous"><parent link="robot_base_link"/><child link="robot_link7"/></joint>
+  <joint name="robot_joint8" type="continuous"><parent link="robot_base_link"/><child link="robot_link8"/></joint>
+  <joint name="robot_joint9" type="continuous"><parent link="robot_base_link"/><child link="robot_link9"/></joint>
+  <joint name="robot_joint10" type="continuous"><parent link="robot_base_link"/><child link="robot_link10"/></joint>
   <xacro:property name="prefix" value="robot_" />
   <xacro:property name="front_axle_steering_joint" value="joint1" />
@@ -22,4 +43,4 @@
   <xacro:include
     filename="$(find romea_mobile_base_description)/ros2_control/base1FAS2FWD.ros2_control.xacro" />
-  <xacro:base_control mode="simulation" base_name="base" />
+  <xacro:base_control mode="simulation" base_name="base" hardware_plugin="${simulation_hardware_plugin}" />
 </robot>

File: romea_mobile_base_utils/test/test_hardware_info2ASxxx.xacro (robot description, xacro)
@@ -1,4 +1,25 @@
 <?xml version='1.0' encoding='utf-8'?>
 <robot name="robot" xmlns:xacro="http://www.ros.org/wiki/xacro">
+  <link name="robot_base_link" />
+  <link name="robot_link1" />
+  <link name="robot_link2" />
+  <link name="robot_link3" />
+  <link name="robot_link4" />
+  <link name="robot_link5" />
+  <link name="robot_link6" />
+  <link name="robot_link7" />
+  <link name="robot_link8" />
+  <link name="robot_link9" />
+  <link name="robot_link10" />
+  <joint name="robot_joint1" type="continuous"><parent link="robot_base_link"/><child link="robot_link1"/></joint>
+  <joint name="robot_joint2" type="continuous"><parent link="robot_base_link"/><child link="robot_link2"/></joint>
+  <joint name="robot_joint3" type="continuous"><parent link="robot_base_link"/><child link="robot_link3"/></joint>
+  <joint name="robot_joint4" type="continuous"><parent link="robot_base_link"/><child link="robot_link4"/></joint>
+  <joint name="robot_joint5" type="continuous"><parent link="robot_base_link"/><child link="robot_link5"/></joint>
+  <joint name="robot_joint6" type="continuous"><parent link="robot_base_link"/><child link="robot_link6"/></joint>
+  <joint name="robot_joint7" type="continuous"><parent link="robot_base_link"/><child link="robot_link7"/></joint>
+  <joint name="robot_joint8" type="continuous"><parent link="robot_base_link"/><child link="robot_link8"/></joint>
+  <joint name="robot_joint9" type="continuous"><parent link="robot_base_link"/><child link="robot_link9"/></joint>
+  <joint name="robot_joint10" type="continuous"><parent link="robot_base_link"/><child link="robot_link10"/></joint>
   <xacro:property name="prefix" value="robot_" />
   <xacro:property name="front_axle_steering_joint" value="joint1" />
@@ -25,4 +46,4 @@
   <xacro:include
     filename="$(find romea_mobile_base_description)/ros2_control/base2AS2RWD.ros2_control.xacro" />
-  <xacro:base_control mode="simulation" base_name="base" />
+  <xacro:base_control mode="simulation" base_name="base" hardware_plugin="${simulation_hardware_plugin}" />
 </robot>

File: romea_mobile_base_utils/test/test_hardware_info2FWSxxx.xacro (robot description, xacro)
@@ -1,4 +1,25 @@
 <?xml version='1.0' encoding='utf-8'?>
 <robot name="robot" xmlns:xacro="http://www.ros.org/wiki/xacro">
+  <link name="robot_base_link" />
+  <link name="robot_link1" />
+  <link name="robot_link2" />
+  <link name="robot_link3" />
+  <link name="robot_link4" />
+  <link name="robot_link5" />
+  <link name="robot_link6" />
+  <link name="robot_link7" />
+  <link name="robot_link8" />
+  <link name="robot_link9" />
+  <link name="robot_link10" />
+  <joint name="robot_joint1" type="continuous"><parent link="robot_base_link"/><child link="robot_link1"/></joint>
+  <joint name="robot_joint2" type="continuous"><parent link="robot_base_link"/><child link="robot_link2"/></joint>
+  <joint name="robot_joint3" type="continuous"><parent link="robot_base_link"/><child link="robot_link3"/></joint>
+  <joint name="robot_joint4" type="continuous"><parent link="robot_base_link"/><child link="robot_link4"/></joint>
+  <joint name="robot_joint5" type="continuous"><parent link="robot_base_link"/><child link="robot_link5"/></joint>
+  <joint name="robot_joint6" type="continuous"><parent link="robot_base_link"/><child link="robot_link6"/></joint>
+  <joint name="robot_joint7" type="continuous"><parent link="robot_base_link"/><child link="robot_link7"/></joint>
+  <joint name="robot_joint8" type="continuous"><parent link="robot_base_link"/><child link="robot_link8"/></joint>
+  <joint name="robot_joint9" type="continuous"><parent link="robot_base_link"/><child link="robot_link9"/></joint>
+  <joint name="robot_joint10" type="continuous"><parent link="robot_base_link"/><child link="robot_link10"/></joint>
   <xacro:property name="prefix" value="robot_" />
   <xacro:property name="front_left_wheel_steering_joint" value="joint1" />
@@ -20,4 +41,4 @@
   <xacro:include
     filename="$(find romea_mobile_base_description)/ros2_control/base2FWS2FWD.ros2_control.xacro" />
-  <xacro:base_control mode="simulation" base_name="base" />
+  <xacro:base_control mode="simulation" base_name="base" hardware_plugin="${simulation_hardware_plugin}" />
 </robot>

File: romea_mobile_base_utils/test/test_hardware_info2TD.xacro (robot description, xacro)
@@ -1,4 +1,25 @@
 <?xml version='1.0' encoding='utf-8'?>
 <robot name="robot" xmlns:xacro="http://www.ros.org/wiki/xacro">
+  <link name="robot_base_link" />
+  <link name="robot_link1" />
+  <link name="robot_link2" />
+  <link name="robot_link3" />
+  <link name="robot_link4" />
+  <link name="robot_link5" />
+  <link name="robot_link6" />
+  <link name="robot_link7" />
+  <link name="robot_link8" />
+  <link name="robot_link9" />
+  <link name="robot_link10" />
+  <joint name="robot_joint1" type="continuous"><parent link="robot_base_link"/><child link="robot_link1"/></joint>
+  <joint name="robot_joint2" type="continuous"><parent link="robot_base_link"/><child link="robot_link2"/></joint>
+  <joint name="robot_joint3" type="continuous"><parent link="robot_base_link"/><child link="robot_link3"/></joint>
+  <joint name="robot_joint4" type="continuous"><parent link="robot_base_link"/><child link="robot_link4"/></joint>
+  <joint name="robot_joint5" type="continuous"><parent link="robot_base_link"/><child link="robot_link5"/></joint>
+  <joint name="robot_joint6" type="continuous"><parent link="robot_base_link"/><child link="robot_link6"/></joint>
+  <joint name="robot_joint7" type="continuous"><parent link="robot_base_link"/><child link="robot_link7"/></joint>
+  <joint name="robot_joint8" type="continuous"><parent link="robot_base_link"/><child link="robot_link8"/></joint>
+  <joint name="robot_joint9" type="continuous"><parent link="robot_base_link"/><child link="robot_link9"/></joint>
+  <joint name="robot_joint10" type="continuous"><parent link="robot_base_link"/><child link="robot_link10"/></joint>
   <xacro:property name="prefix" value="robot_" />
   <xacro:property name="left_sprocket_wheel_spinning_joint" value="joint1" />
@@ -13,4 +34,4 @@
   <xacro:include
     filename="$(find romea_mobile_base_description)/ros2_control/base2TD.ros2_control.xacro" />
-  <xacro:base_control mode="simulation" base_name="base" />
+  <xacro:base_control mode="simulation" base_name="base" hardware_plugin="${simulation_hardware_plugin}" />
 </robot>

File: romea_mobile_base_utils/test/test_hardware_info2THD.xacro (robot description, xacro)
@@ -1,4 +1,25 @@
 <?xml version='1.0' encoding='utf-8'?>
 <robot name="robot" xmlns:xacro="http://www.ros.org/wiki/xacro">
+  <link name="robot_base_link" />
+  <link name="robot_link1" />
+  <link name="robot_link2" />
+  <link name="robot_link3" />
+  <link name="robot_link4" />
+  <link name="robot_link5" />
+  <link name="robot_link6" />
+  <link name="robot_link7" />
+  <link name="robot_link8" />
+  <link name="robot_link9" />
+  <link name="robot_link10" />
+  <joint name="robot_joint1" type="continuous"><parent link="robot_base_link"/><child link="robot_link1"/></joint>
+  <joint name="robot_joint2" type="continuous"><parent link="robot_base_link"/><child link="robot_link2"/></joint>
+  <joint name="robot_joint3" type="continuous"><parent link="robot_base_link"/><child link="robot_link3"/></joint>
+  <joint name="robot_joint4" type="continuous"><parent link="robot_base_link"/><child link="robot_link4"/></joint>
+  <joint name="robot_joint5" type="continuous"><parent link="robot_base_link"/><child link="robot_link5"/></joint>
+  <joint name="robot_joint6" type="continuous"><parent link="robot_base_link"/><child link="robot_link6"/></joint>
+  <joint name="robot_joint7" type="continuous"><parent link="robot_base_link"/><child link="robot_link7"/></joint>
+  <joint name="robot_joint8" type="continuous"><parent link="robot_base_link"/><child link="robot_link8"/></joint>
+  <joint name="robot_joint9" type="continuous"><parent link="robot_base_link"/><child link="robot_link9"/></joint>
+  <joint name="robot_joint10" type="continuous"><parent link="robot_base_link"/><child link="robot_link10"/></joint>
   <xacro:property name="prefix" value="robot_" />
   <xacro:property name="left_sprocket_wheel_spinning_joint" value="joint1" />
@@ -15,4 +36,4 @@
   <xacro:include
     filename="$(find romea_mobile_base_description)/ros2_control/base2THD.ros2_control.xacro" />
-  <xacro:base_control mode="simulation" base_name="base" />
+  <xacro:base_control mode="simulation" base_name="base" hardware_plugin="${simulation_hardware_plugin}" />
 </robot>

File: romea_mobile_base_utils/test/test_hardware_info2TTD.xacro (robot description, xacro)
@@ -1,4 +1,25 @@
 <?xml version='1.0' encoding='utf-8'?>
 <robot name="robot" xmlns:xacro="http://www.ros.org/wiki/xacro">
+  <link name="robot_base_link" />
+  <link name="robot_link1" />
+  <link name="robot_link2" />
+  <link name="robot_link3" />
+  <link name="robot_link4" />
+  <link name="robot_link5" />
+  <link name="robot_link6" />
+  <link name="robot_link7" />
+  <link name="robot_link8" />
+  <link name="robot_link9" />
+  <link name="robot_link10" />
+  <joint name="robot_joint1" type="continuous"><parent link="robot_base_link"/><child link="robot_link1"/></joint>
+  <joint name="robot_joint2" type="continuous"><parent link="robot_base_link"/><child link="robot_link2"/></joint>
+  <joint name="robot_joint3" type="continuous"><parent link="robot_base_link"/><child link="robot_link3"/></joint>
+  <joint name="robot_joint4" type="continuous"><parent link="robot_base_link"/><child link="robot_link4"/></joint>
+  <joint name="robot_joint5" type="continuous"><parent link="robot_base_link"/><child link="robot_link5"/></joint>
+  <joint name="robot_joint6" type="continuous"><parent link="robot_base_link"/><child link="robot_link6"/></joint>
+  <joint name="robot_joint7" type="continuous"><parent link="robot_base_link"/><child link="robot_link7"/></joint>
+  <joint name="robot_joint8" type="continuous"><parent link="robot_base_link"/><child link="robot_link8"/></joint>
+  <joint name="robot_joint9" type="continuous"><parent link="robot_base_link"/><child link="robot_link9"/></joint>
+  <joint name="robot_joint10" type="continuous"><parent link="robot_base_link"/><child link="robot_link10"/></joint>
   <xacro:property name="prefix" value="robot_" />
   <xacro:property name="left_sprocket_wheel_spinning_joint" value="joint1" />
@@ -18,4 +39,4 @@
   <xacro:include
     filename="$(find romea_mobile_base_description)/ros2_control/base2TTD.ros2_control.xacro" />
-  <xacro:base_control mode="simulation" base_name="base" />
+  <xacro:base_control mode="simulation" base_name="base" hardware_plugin="${simulation_hardware_plugin}" />
 </robot>

File: romea_mobile_base_utils/test/test_hardware_info4WD.xacro (robot description, xacro)
@@ -1,4 +1,25 @@
 <?xml version='1.0' encoding='utf-8'?>
 <robot name="robot" xmlns:xacro="http://www.ros.org/wiki/xacro">
+  <link name="robot_base_link" />
+  <link name="robot_link1" />
+  <link name="robot_link2" />
+  <link name="robot_link3" />
+  <link name="robot_link4" />
+  <link name="robot_link5" />
+  <link name="robot_link6" />
+  <link name="robot_link7" />
+  <link name="robot_link8" />
+  <link name="robot_link9" />
+  <link name="robot_link10" />
+  <joint name="robot_joint1" type="continuous"><parent link="robot_base_link"/><child link="robot_link1"/></joint>
+  <joint name="robot_joint2" type="continuous"><parent link="robot_base_link"/><child link="robot_link2"/></joint>
+  <joint name="robot_joint3" type="continuous"><parent link="robot_base_link"/><child link="robot_link3"/></joint>
+  <joint name="robot_joint4" type="continuous"><parent link="robot_base_link"/><child link="robot_link4"/></joint>
+  <joint name="robot_joint5" type="continuous"><parent link="robot_base_link"/><child link="robot_link5"/></joint>
+  <joint name="robot_joint6" type="continuous"><parent link="robot_base_link"/><child link="robot_link6"/></joint>
+  <joint name="robot_joint7" type="continuous"><parent link="robot_base_link"/><child link="robot_link7"/></joint>
+  <joint name="robot_joint8" type="continuous"><parent link="robot_base_link"/><child link="robot_link8"/></joint>
+  <joint name="robot_joint9" type="continuous"><parent link="robot_base_link"/><child link="robot_link9"/></joint>
+  <joint name="robot_joint10" type="continuous"><parent link="robot_base_link"/><child link="robot_link10"/></joint>
   <xacro:property name="prefix" value="robot_" />
   <xacro:property name="front_left_wheel_spinning_joint" value="joint1" />
@@ -18,4 +39,4 @@
   <xacro:include
     filename="$(find romea_mobile_base_description)/ros2_control/base4WD.ros2_control.xacro" />
-  <xacro:base_control mode="live" base_name="base" />
+  <xacro:base_control mode="live" base_name="base" hardware_plugin="${live_hardware_plugin}" />
 </robot>

File: romea_mobile_base_utils/test/test_hardware_info4WS4WD.xacro (robot description, xacro)
@@ -1,4 +1,25 @@
 <?xml version='1.0' encoding='utf-8'?>
 <robot name="robot" xmlns:xacro="http://www.ros.org/wiki/xacro">
+  <link name="robot_base_link" />
+  <link name="robot_link1" />
+  <link name="robot_link2" />
+  <link name="robot_link3" />
+  <link name="robot_link4" />
+  <link name="robot_link5" />
+  <link name="robot_link6" />
+  <link name="robot_link7" />
+  <link name="robot_link8" />
+  <link name="robot_link9" />
+  <link name="robot_link10" />
+  <joint name="robot_joint1" type="continuous"><parent link="robot_base_link"/><child link="robot_link1"/></joint>
+  <joint name="robot_joint2" type="continuous"><parent link="robot_base_link"/><child link="robot_link2"/></joint>
+  <joint name="robot_joint3" type="continuous"><parent link="robot_base_link"/><child link="robot_link3"/></joint>
+  <joint name="robot_joint4" type="continuous"><parent link="robot_base_link"/><child link="robot_link4"/></joint>
+  <joint name="robot_joint5" type="continuous"><parent link="robot_base_link"/><child link="robot_link5"/></joint>
+  <joint name="robot_joint6" type="continuous"><parent link="robot_base_link"/><child link="robot_link6"/></joint>
+  <joint name="robot_joint7" type="continuous"><parent link="robot_base_link"/><child link="robot_link7"/></joint>
+  <joint name="robot_joint8" type="continuous"><parent link="robot_base_link"/><child link="robot_link8"/></joint>
+  <joint name="robot_joint9" type="continuous"><parent link="robot_base_link"/><child link="robot_link9"/></joint>
+  <joint name="robot_joint10" type="continuous"><parent link="robot_base_link"/><child link="robot_link10"/></joint>
   <xacro:property name="prefix" value="robot_" />
   <xacro:property name="front_left_wheel_steering_joint" value="joint1" />
@@ -22,4 +43,4 @@
   <xacro:include
     filename="$(find romea_mobile_base_description)/ros2_control/base4WS4WD.ros2_control.xacro" />
-  <xacro:base_control mode="live" base_name="base" />
+  <xacro:base_control mode="live" base_name="base" hardware_plugin="${live_hardware_plugin}" />
 </robot>
