Commit message: fix unit tests
Signed-off-by: Jean Laneurit <jean.laneurit@inrae.fr>

File: romea_mobile_base_hardware/test_legacy/test_hardware_interface2FWC2RWD.xacro (robot description, xacro)
@@ -16,35 +16,12 @@
   <xacro:property name="rear_wheel_radius" value="0.3" />
   <xacro:property name="maximal_wheel_speed" value="1.0" />
-  <link name="${prefix}base_link" />
-  <link name="${prefix}front_left_wheel_swiveling_link" />
-  <link name="${prefix}front_right_wheel_swiveling_link" />
-  <link name="${prefix}front_left_wheel_spinning_link" />
-  <link name="${prefix}front_right_wheel_spinning_link" />
-  <link name="${prefix}rear_left_wheel_spinning_link" />
-  <link name="${prefix}rear_right_wheel_spinning_link" />
-  <joint name="${prefix}${front_left_wheel_swiveling_joint}" type="continuous">
-    <parent link="${prefix}base_link" />
-    <child link="${prefix}front_left_wheel_swiveling_link" />
-  </joint>
-  <joint name="${prefix}${front_right_wheel_swiveling_joint}" type="continuous">
-    <parent link="${prefix}base_link" />
-    <child link="${prefix}front_right_wheel_swiveling_link" />
-  </joint>
-  <joint name="${prefix}${front_left_wheel_spinning_joint}" type="continuous">
-    <parent link="${prefix}front_left_wheel_swiveling_link" />
-    <child link="${prefix}front_left_wheel_spinning_link" />
-  </joint>
-  <joint name="${prefix}${front_right_wheel_spinning_joint}" type="continuous">
-    <parent link="${prefix}front_right_wheel_swiveling_link" />
-    <child link="${prefix}front_right_wheel_spinning_link" />
-  </joint>
-  <joint name="${prefix}${rear_left_wheel_spinning_joint}" type="continuous">
-    <parent link="${prefix}base_link" />
-    <child link="${prefix}rear_left_wheel_spinning_link" />
-  </joint>
-  <joint name="${prefix}${rear_right_wheel_spinning_joint}" type="continuous">
-    <parent link="${prefix}base_link" />
-    <child link="${prefix}rear_right_wheel_spinning_link" />
-  </joint>
+  <xacro:property name="base_link" value="base_link" />
+  <xacro:property name="front_left_wheel_swiveling_link" value="front_left_wheel_swiveling_link" />
+  <xacro:property name="front_right_wheel_swiveling_link" value="front_right_wheel_swiveling_link" />
+  <xacro:property name="front_left_wheel_spinning_link" value="front_left_wheel_spinning_link" />
+  <xacro:property name="front_right_wheel_spinning_link" value="front_right_wheel_spinning_link" />
+  <xacro:property name="rear_left_wheel_spinning_link" value="rear_left_wheel_spinning_link" />
+  <xacro:property name="rear_right_wheel_spinning_link" value="rear_right_wheel_spinning_link" />
+  <xacro:property name="maximal_wheel_torque" value="10000000" />
   <xacro:include
     filename="$(find romea_mobile_base_description)/ros2_control/base2FWC2RWD.ros2_control.xacro" />

File: romea_mobile_base_hardware/test_legacy/test_hardware_interface2TD.xacro (robot description, xacro)
@@ -2,5 +2,4 @@
 <robot name="robot" xmlns:xacro="http://www.ros.org/wiki/xacro">
   <xacro:property name="prefix" value="robot_" />
-  <xacro:property name="base_footprint_link" value="base_footprint" />
   <xacro:property name="base_link" value="base_link" />
   <xacro:property name="left_sprocket_wheel_spinning_link" value="left_sprocket_wheel_spinning_link" />
@@ -8,5 +7,4 @@
   <xacro:property name="left_idler_wheel_spinning_link" value="left_idler_wheel_spinning_link" />
   <xacro:property name="right_idler_wheel_spinning_link" value="right_idler_wheel_spinning_link" />
-  <xacro:property name="base_footprint_joint" value="base_footprint_joint" />
   <xacro:property name="left_sprocket_wheel_spinning_joint" value="joint1" />
   <xacro:property name="right_sprocket_wheel_spinning_joint" value="joint2" />
@@ -20,5 +18,4 @@
   <xacro:property name="maximal_wheel_torque" value="10000000" />
   <xacro:include filename="$(find romea_mobile_base_description)/ros2_control/base2TD.ros2_control.xacro" />
-  <xacro:base_control_model />
   <xacro:base_control mode="live" base_name="base" hardware_plugin="${live_hardware_plugin}" />
 </robot>

File: romea_mobile_base_hardware/test_legacy/test_hardware_interface2THD.xacro (robot description, xacro)
@@ -8,8 +8,12 @@
   <xacro:property name="rear_left_idler_wheel_spinning_joint" value="joint5" />
   <xacro:property name="rear_right_idler_wheel_spinning_joint" value="joint6" />
-  <xacro:property name="maximal_wheel_speed" value="1.0" />
-  <xacro:property name="sprocket_wheel_radius" value="0.2" />
-  <xacro:property name="idler_wheel_radius" value="0.15" />
-  <xacro:property name="track_thickness" value="0.2" />
+  <xacro:property name="base_link" value="base_link" />
+  <xacro:property name="left_sprocket_wheel_spinning_link" value="left_sprocket_wheel_spinning_link" />
+  <xacro:property name="right_sprocket_wheel_spinning_link" value="right_sprocket_wheel_spinning_link" />
+  <xacro:property name="front_left_idler_wheel_spinning_link" value="front_left_idler_wheel_spinning_link" />
+  <xacro:property name="front_right_idler_wheel_spinning_link" value="front_right_idler_wheel_spinning_link" />
+  <xacro:property name="rear_left_idler_wheel_spinning_link" value="rear_left_idler_wheel_spinning_link" />
+  <xacro:property name="rear_right_idler_wheel_spinning_link" value="rear_right_idler_wheel_spinning_link" />
+  <xacro:property name="maximal_wheel_torque" value="10000000" />
   <xacro:property name="live_hardware_plugin" value="foo" />
   <xacro:property name="sprocket_wheel_radius" value="0.8" />
@@ -17,35 +21,4 @@
   <xacro:property name="track_thickness" value="0.1" />
   <xacro:property name="maximal_wheel_speed" value="1.0" />
-  <link name="${prefix}base_link" />
-  <link name="${prefix}left_sprocket_wheel_spinning_link" />
-  <link name="${prefix}right_sprocket_wheel_spinning_link" />
-  <link name="${prefix}front_left_idler_wheel_spinning_link" />
-  <link name="${prefix}front_right_idler_wheel_spinning_link" />
-  <link name="${prefix}rear_left_idler_wheel_spinning_link" />
-  <link name="${prefix}rear_right_idler_wheel_spinning_link" />
-  <joint name="${prefix}${left_sprocket_wheel_spinning_joint}" type="continuous">
-    <parent link="${prefix}base_link" />
-    <child link="${prefix}left_sprocket_wheel_spinning_link" />
-  </joint>
-  <joint name="${prefix}${right_sprocket_wheel_spinning_joint}" type="continuous">
-    <parent link="${prefix}base_link" />
-    <child link="${prefix}right_sprocket_wheel_spinning_link" />
-  </joint>
-  <joint name="${prefix}${front_left_idler_wheel_spinning_joint}" type="continuous">
-    <parent link="${prefix}base_link" />
-    <child link="${prefix}front_left_idler_wheel_spinning_link" />
-  </joint>
-  <joint name="${prefix}${front_right_idler_wheel_spinning_joint}" type="continuous">
-    <parent link="${prefix}base_link" />
-    <child link="${prefix}front_right_idler_wheel_spinning_link" />
-  </joint>
-  <joint name="${prefix}${rear_left_idler_wheel_spinning_joint}" type="continuous">
-    <parent link="${prefix}base_link" />
-    <child link="${prefix}rear_left_idler_wheel_spinning_link" />
-  </joint>
-  <joint name="${prefix}${rear_right_idler_wheel_spinning_joint}" type="continuous">
-    <parent link="${prefix}base_link" />
-    <child link="${prefix}rear_right_idler_wheel_spinning_link" />
-  </joint>
   <xacro:include
     filename="$(find romea_mobile_base_description)/ros2_control/base2THD.ros2_control.xacro" />

File: romea_mobile_base_hardware/test_legacy/test_hardware_interface2TTD.xacro (robot description, xacro)
@@ -2,5 +2,4 @@
 <robot name="robot" xmlns:xacro="http://www.ros.org/wiki/xacro">
   <xacro:property name="prefix" value="robot_" />
-  <xacro:property name="base_footprint_link" value="base_footprint" />
   <xacro:property name="base_link" value="base_link" />
   <xacro:property name="left_sprocket_wheel_spinning_link" value="left_sprocket_wheel_spinning_link" />
@@ -12,5 +11,4 @@
   <xacro:property name="rear_left_roller_wheel_spinning_link" value="rear_left_roller_wheel_spinning_link" />
   <xacro:property name="rear_right_roller_wheel_spinning_link" value="rear_right_roller_wheel_spinning_link" />
-  <xacro:property name="base_footprint_joint" value="base_footprint_joint" />
   <xacro:property name="left_sprocket_wheel_spinning_joint" value="joint1" />
   <xacro:property name="right_sprocket_wheel_spinning_joint" value="joint2" />
@@ -29,5 +27,4 @@
   <xacro:property name="maximal_wheel_torque" value="10000000" />
   <xacro:include filename="$(find romea_mobile_base_description)/ros2_control/base2TTD.ros2_control.xacro" />
-  <xacro:base_control_model />
   <xacro:base_control mode="live" base_name="base" hardware_plugin="${live_hardware_plugin}" />
 </robot>

File: romea_mobile_base_hardware/test_legacy/test_hardware_interface4WD.xacro (robot description, xacro)
@@ -24,5 +24,4 @@
   <xacro:include
     filename="$(find romea_mobile_base_description)/ros2_control/base4WD.ros2_control.xacro" />
-  <xacro:base_control_model/>
     <xacro:base_control mode="live" base_name="base" hardware_plugin="${live_hardware_plugin}" />
 </robot>

File: romea_mobile_base_hardware/test_legacy/test_hardware_interface4WS4WD.xacro (robot description, xacro)
@@ -36,5 +36,4 @@
   <xacro:include
     filename="$(find romea_mobile_base_description)/ros2_control/base4WS4WD.ros2_control.xacro" />
-  <xacro:base_control_model/>
     <xacro:base_control mode="live" base_name="base" hardware_plugin="${live_hardware_plugin}" />
 </robot>

File: romea_mobile_base_simulation/test_legacy/test_simulation_interface2FWC2RWD.xacro (robot description, xacro)
@@ -16,41 +16,12 @@
   <xacro:property name="rear_wheel_radius" value="0.6" />
   <xacro:property name="maximal_wheel_speed" value="1.0" />
-  <link name="robot_base_link" />
-  <link name="robot_link1" />
-  <link name="robot_link2" />
-  <link name="robot_link3" />
-  <link name="robot_link4" />
-  <link name="robot_link5" />
-  <link name="robot_link6" />
-  <joint name="robot_joint1" type="continuous">
-    <parent link="robot_base_link" />
-    <child link="robot_link1" />
-    <axis xyz="0 0 1" />
-  </joint>
-  <joint name="robot_joint2" type="continuous">
-    <parent link="robot_base_link" />
-    <child link="robot_link2" />
-    <axis xyz="0 0 1" />
-  </joint>
-  <joint name="robot_joint3" type="continuous">
-    <parent link="robot_link1" />
-    <child link="robot_link3" />
-    <axis xyz="0 1 0" />
-  </joint>
-  <joint name="robot_joint4" type="continuous">
-    <parent link="robot_link2" />
-    <child link="robot_link4" />
-    <axis xyz="0 1 0" />
-  </joint>
-  <joint name="robot_joint5" type="continuous">
-    <parent link="robot_base_link" />
-    <child link="robot_link5" />
-    <axis xyz="0 1 0" />
-  </joint>
-  <joint name="robot_joint6" type="continuous">
-    <parent link="robot_base_link" />
-    <child link="robot_link6" />
-    <axis xyz="0 1 0" />
-  </joint>
+  <xacro:property name="base_link" value="base_link" />
+  <xacro:property name="front_left_wheel_swiveling_link" value="front_left_wheel_swiveling_link" />
+  <xacro:property name="front_right_wheel_swiveling_link" value="front_right_wheel_swiveling_link" />
+  <xacro:property name="front_left_wheel_spinning_link" value="front_left_wheel_spinning_link" />
+  <xacro:property name="front_right_wheel_spinning_link" value="front_right_wheel_spinning_link" />
+  <xacro:property name="rear_left_wheel_spinning_link" value="rear_left_wheel_spinning_link" />
+  <xacro:property name="rear_right_wheel_spinning_link" value="rear_right_wheel_spinning_link" />
+  <xacro:property name="maximal_wheel_torque" value="10000000" />
   <xacro:include
     filename="$(find romea_mobile_base_description)/ros2_control/base2FWC2RWD.ros2_control.xacro" />

File: romea_mobile_base_simulation/test_legacy/test_simulation_interface2TD.xacro (robot description, xacro)
@@ -2,5 +2,4 @@
 <robot name="robot" xmlns:xacro="http://www.ros.org/wiki/xacro">
   <xacro:property name="prefix" value="robot_" />
-  <xacro:property name="base_footprint_link" value="base_footprint" />
   <xacro:property name="base_link" value="base_link" />
   <xacro:property name="left_sprocket_wheel_spinning_link" value="left_sprocket_wheel_spinning_link" />
@@ -8,5 +7,4 @@
   <xacro:property name="left_idler_wheel_spinning_link" value="left_idler_wheel_spinning_link" />
   <xacro:property name="right_idler_wheel_spinning_link" value="right_idler_wheel_spinning_link" />
-  <xacro:property name="base_footprint_joint" value="base_footprint_joint" />
   <xacro:property name="left_sprocket_wheel_spinning_joint" value="joint1" />
   <xacro:property name="right_sprocket_wheel_spinning_joint" value="joint2" />
@@ -20,5 +18,4 @@
   <xacro:property name="maximal_wheel_torque" value="10000000" />
   <xacro:include filename="$(find romea_mobile_base_description)/ros2_control/base2TD.ros2_control.xacro" />
-  <xacro:base_control_model />
   <xacro:base_control mode="simulation" base_name="base" hardware_plugin="${simulation_hardware_plugin}" />
 </robot>

File: romea_mobile_base_simulation/test_legacy/test_simulation_interface2THD.xacro (robot description, xacro)
@@ -8,4 +8,12 @@
   <xacro:property name="rear_left_idler_wheel_spinning_joint" value="joint5" />
   <xacro:property name="rear_right_idler_wheel_spinning_joint" value="joint6" />
+  <xacro:property name="base_link" value="base_link" />
+  <xacro:property name="left_sprocket_wheel_spinning_link" value="left_sprocket_wheel_spinning_link" />
+  <xacro:property name="right_sprocket_wheel_spinning_link" value="right_sprocket_wheel_spinning_link" />
+  <xacro:property name="front_left_idler_wheel_spinning_link" value="front_left_idler_wheel_spinning_link" />
+  <xacro:property name="front_right_idler_wheel_spinning_link" value="front_right_idler_wheel_spinning_link" />
+  <xacro:property name="rear_left_idler_wheel_spinning_link" value="rear_left_idler_wheel_spinning_link" />
+  <xacro:property name="rear_right_idler_wheel_spinning_link" value="rear_right_idler_wheel_spinning_link" />
+  <xacro:property name="maximal_wheel_torque" value="10000000" />
   <xacro:property name="simulation_hardware_plugin" value="foo" />
   <xacro:property name="sprocket_wheel_radius" value="0.8" />

File: romea_mobile_base_simulation/test_legacy/test_simulation_interface2TTD.xacro (robot description, xacro)
@@ -2,5 +2,4 @@
 <robot name="robot" xmlns:xacro="http://www.ros.org/wiki/xacro">
   <xacro:property name="prefix" value="robot_" />
-  <xacro:property name="base_footprint_link" value="base_footprint" />
   <xacro:property name="base_link" value="base_link" />
   <xacro:property name="left_sprocket_wheel_spinning_link" value="left_sprocket_wheel_spinning_link" />
@@ -12,5 +11,4 @@
   <xacro:property name="rear_left_roller_wheel_spinning_link" value="rear_left_roller_wheel_spinning_link" />
   <xacro:property name="rear_right_roller_wheel_spinning_link" value="rear_right_roller_wheel_spinning_link" />
-  <xacro:property name="base_footprint_joint" value="base_footprint_joint" />
   <xacro:property name="left_sprocket_wheel_spinning_joint" value="joint1" />
   <xacro:property name="right_sprocket_wheel_spinning_joint" value="joint2" />
@@ -29,5 +27,4 @@
   <xacro:property name="maximal_wheel_torque" value="10000000" />
   <xacro:include filename="$(find romea_mobile_base_description)/ros2_control/base2TTD.ros2_control.xacro" />
-  <xacro:base_control_model />
   <xacro:base_control mode="simulation" base_name="base" hardware_plugin="${simulation_hardware_plugin}" />
 </robot>

File: romea_mobile_base_utils/test/test_hardware_info2THD.xacro (robot description, xacro)
@@ -1,25 +1,4 @@
 <?xml version='1.0' encoding='utf-8'?>
 <robot name="robot" xmlns:xacro="http://www.ros.org/wiki/xacro">
-  <link name="robot_base_link" />
-  <link name="robot_link1" />
-  <link name="robot_link2" />
-  <link name="robot_link3" />
-  <link name="robot_link4" />
-  <link name="robot_link5" />
-  <link name="robot_link6" />
-  <link name="robot_link7" />
-  <link name="robot_link8" />
-  <link name="robot_link9" />
-  <link name="robot_link10" />
-  <joint name="robot_joint1" type="continuous"><parent link="robot_base_link"/><child link="robot_link1"/></joint>
-  <joint name="robot_joint2" type="continuous"><parent link="robot_base_link"/><child link="robot_link2"/></joint>
-  <joint name="robot_joint3" type="continuous"><parent link="robot_base_link"/><child link="robot_link3"/></joint>
-  <joint name="robot_joint4" type="continuous"><parent link="robot_base_link"/><child link="robot_link4"/></joint>
-  <joint name="robot_joint5" type="continuous"><parent link="robot_base_link"/><child link="robot_link5"/></joint>
-  <joint name="robot_joint6" type="continuous"><parent link="robot_base_link"/><child link="robot_link6"/></joint>
-  <joint name="robot_joint7" type="continuous"><parent link="robot_base_link"/><child link="robot_link7"/></joint>
-  <joint name="robot_joint8" type="continuous"><parent link="robot_base_link"/><child link="robot_link8"/></joint>
-  <joint name="robot_joint9" type="continuous"><parent link="robot_base_link"/><child link="robot_link9"/></joint>
-  <joint name="robot_joint10" type="continuous"><parent link="robot_base_link"/><child link="robot_link10"/></joint>
   <xacro:property name="prefix" value="robot_" />
   <xacro:property name="left_sprocket_wheel_spinning_joint" value="joint1" />
@@ -29,4 +8,12 @@
   <xacro:property name="rear_left_idler_wheel_spinning_joint" value="joint5" />
   <xacro:property name="rear_right_idler_wheel_spinning_joint" value="joint6" />
+  <xacro:property name="base_link" value="base_link" />
+  <xacro:property name="left_sprocket_wheel_spinning_link" value="left_sprocket_wheel_spinning_link" />
+  <xacro:property name="right_sprocket_wheel_spinning_link" value="right_sprocket_wheel_spinning_link" />
+  <xacro:property name="front_left_idler_wheel_spinning_link" value="front_left_idler_wheel_spinning_link" />
+  <xacro:property name="front_right_idler_wheel_spinning_link" value="front_right_idler_wheel_spinning_link" />
+  <xacro:property name="rear_left_idler_wheel_spinning_link" value="rear_left_idler_wheel_spinning_link" />
+  <xacro:property name="rear_right_idler_wheel_spinning_link" value="rear_right_idler_wheel_spinning_link" />
+  <xacro:property name="maximal_wheel_torque" value="10000000" />
   <xacro:property name="simulation_hardware_plugin" value="foo" />
   <xacro:property name="sprocket_wheel_radius" value="0.8" />

File: romea_mobile_base_utils/test/test_hardware_info2TTD.xacro (robot description, xacro)
@@ -2,5 +2,4 @@
 <robot name="robot" xmlns:xacro="http://www.ros.org/wiki/xacro">
   <xacro:property name="prefix" value="robot_" />
-  <xacro:property name="base_footprint_link" value="base_footprint" />
   <xacro:property name="base_link" value="base_link" />
   <xacro:property name="left_sprocket_wheel_spinning_link" value="left_sprocket_wheel_spinning_link" />
@@ -12,5 +11,4 @@
   <xacro:property name="rear_left_roller_wheel_spinning_link" value="rear_left_roller_wheel_spinning_link" />
   <xacro:property name="rear_right_roller_wheel_spinning_link" value="rear_right_roller_wheel_spinning_link" />
-  <xacro:property name="base_footprint_joint" value="base_footprint_joint" />
   <xacro:property name="left_sprocket_wheel_spinning_joint" value="joint1" />
   <xacro:property name="right_sprocket_wheel_spinning_joint" value="joint2" />
@@ -29,5 +27,4 @@
   <xacro:property name="maximal_wheel_torque" value="10000000" />
   <xacro:include filename="$(find romea_mobile_base_description)/ros2_control/base2TTD.ros2_control.xacro" />
-  <xacro:base_control_model />
   <xacro:base_control mode="simulation" base_name="base" hardware_plugin="${simulation_hardware_plugin}" />
 </robot>

File: romea_mobile_base_utils/test/test_hardware_info4WD.xacro (robot description, xacro)
@@ -24,5 +24,4 @@
   <xacro:include
     filename="$(find romea_mobile_base_description)/ros2_control/base4WD.ros2_control.xacro" />
-  <xacro:base_control_model/>
     <xacro:base_control mode="live" base_name="base" hardware_plugin="${live_hardware_plugin}" />
 </robot>

File: romea_mobile_base_utils/test/test_hardware_info4WS4WD.xacro (robot description, xacro)
@@ -34,5 +34,4 @@
   <xacro:include
     filename="$(find romea_mobile_base_description)/ros2_control/base4WS4WD.ros2_control.xacro" />
-  <xacro:base_control_model/>
     <xacro:base_control mode="live" base_name="base" hardware_plugin="${live_hardware_plugin}" />
 </robot>
